File: boards/control-2011-c/control-fpga-config.sch (EAGLE design)
At the start: 285 parts, among them J1 0528520870, J10 2MM-6H, J11 JST_VH_2, J12 2MM-4V, J13 2MM-4H, J14 2MM-4H, J15 2MM-4H, J16 2MM-4H, J17 2MM-8H, J19 JST_VH_2, J2 MINI-USB, J20 2MM-5V, J3 2MM-2H, J4 Molex 0522711179, J5 Molex 0522711179, J6 Molex 0522711179, J7 Molex 0522711179, J8 MMCX_RA, J9 2MM-3H, Q1 IRF9310TRPBF, Q10 IRF8734TRPBF, Q11 IRF9310TRPBF, Q12 IRF8734TRPBF, Q13 IRF9310TRPBF, Q14 IRF8734TRPBF, Q15 IRF9310TRPBF, Q16 IRF8734TRPBF, Q17 IRF9310TRPBF, Q18 IRF8734TRPBF, Q19 IRF9310TRPBF, Q2 IRF8734TRPBF, Q20 IRF8734TRPBF, Q21 IRF9310TRPBF, Q22 IRF8734TRPBF, Q23 IRF9310TRPBF, Q24 IRF8734TRPBF, Q25 IRF9310TRPBF, Q26 IRF8734TRPBF, Q27 IRF9310TRPBF, Q28 IRF8734TRPBF, Q29 IRF9310TRPBF, Q3 IRF9310TRPBF, Q30 IRF8734TRPBF, Q33 FDV304P, Q4 IRF8734TRPBF, Q5 IRF9310TRPBF, Q6 IRF8734TRPBF, Q7 IRF9310TRPBF, Q8 IRF8734TRPBF, Q9 IRF9310TRPBF, U1 XC3S100E, U10 CC1101, U12 TC4428, U13 0896BM15A0001, U15 TC4428, U18 TC4428, U19 IMU3000, U2 M25P10, U20 KXTF9-2050, U21 TC4428, U24 TC4428, U27 TC4428, U3 LM2734, U30 TC4428, U33 TC4428, U36 TC4428, U39 TC4428, U4 MCP1824T-1202E/OT, U42 TC4428, U45 TC4428, U48 TC4428, U5 MCP1824T-2502E/OT, U6 TC4428, U7 AT91SAM7S256, U8 MCP1824ST-3302E/DB, U9 TC4428, X1 18.432MHz, X2 644-1055-1-ND

Commit message: control-2011-c
Other:
- note added: "CCLK"
- note added: "CSO_B"
- note added: "DIN/D0"
- note added: "DOUT/BUSY"
- note added: "INIT_B"
- note added: "M0"
- note added: "M1"
- note added: "M2"
- note added: "MOSI/CSI_B"
- note added: "VS0/A17"
- note added: "VS1/A18"
- note added: "VS2/A19"
Changed lines of the file:
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@@
 <?xml version="1.0" encoding="utf-8"?>
 <!DOCTYPE eagle SYSTEM "eagle.dtd">
-<eagle version="6.1">
+<eagle version="6.5.0">
 <drawing>
 <settings>
@@
 <setting verticaltext="up"/>
 </settings>
-<grid distance="0.1" unitdist="inch" unit="inch" style="lines" multiple="1" display="no" altdistance="0.01" altunitdist="inch" altunit="inch"/>
+<grid distance="0.025" unitdist="inch" unit="inch" style="lines" multiple="1" display="yes" altdistance="0.01" altunitdist="inch" altunit="inch"/>
 <layers>
 <layer number="1" name="Top" color="4" fill="1" visible="no" active="no"/>
@@
 <layer number="95" name="Names" color="7" fill="1" visible="yes" active="yes"/>
 <layer number="96" name="Values" color="7" fill="1" visible="yes" active="yes"/>
-<layer number="97" name="Info" color="7" fill="1" visible="yes" active="yes"/>
-<layer number="98" name="Guide" color="7" fill="1" visible="yes" active="yes"/>
+<layer number="97" name="Info" color="1" fill="1" visible="yes" active="yes"/>
+<layer number="98" name="Guide" color="9" fill="1" visible="yes" active="yes"/>
 <layer number="100" name="Muster" color="7" fill="1" visible="yes" active="yes"/>
 <layer number="101" name="Patch_Top" color="7" fill="1" visible="yes" active="yes"/>
@@
 <text x="12.7" y="175.26" size="1.778" layer="91" rot="R90">SPARE FPGA I/O</text>
 <text x="5.08" y="22.86" size="1.778" layer="91">Cable: Parlex 100R08-51B</text>
+<text x="268.605" y="50.8" size="2.032" layer="97" font="vector" ratio="12" align="center-right">INIT_B</text>
+<text x="268.605" y="129.54" size="2.032" layer="97" font="vector" ratio="12" align="center-right">CCLK</text>
+<text x="268.605" y="106.68" size="2.032" layer="98" font="vector" ratio="12" align="center-right">M0</text>
+<text x="268.605" y="48.26" size="2.032" layer="97" font="vector" ratio="12" align="center-right">CSO_B</text>
+<text x="268.605" y="60.96" size="2.032" layer="97" font="vector" ratio="12" align="center-right">MOSI/CSI_B</text>
+<text x="268.605" y="58.42" size="2.032" layer="97" font="vector" ratio="12" align="center-right">DOUT/BUSY</text>
+<text x="268.605" y="109.22" size="2.032" layer="97" font="vector" ratio="12" align="center-right">DIN/D0</text>
+<text x="268.605" y="121.92" size="2.032" layer="97" font="vector" ratio="12" align="center-right">VS1/A18</text>
+<text x="268.605" y="119.38" size="2.032" layer="97" font="vector" ratio="12" align="center-right">VS2/A19</text>
+<text x="268.605" y="127" size="2.032" layer="97" font="vector" ratio="12" align="center-right">VS0/A17</text>
+<text x="268.605" y="93.98" size="2.032" layer="98" font="vector" ratio="12" align="center-right">M2</text>
+<text x="268.605" y="101.6" size="2.032" layer="98" font="vector" ratio="12" align="center-right">M1</text>
 </plain>
 <instances>
