File: boards/base-station-v2.0/base-station.sch (EAGLE design)
At the start: 3 parts, among them J1 UX60A-MB-5ST, U1 609-3706-1-ND-MALE

Commit message: New base station
Parts:
- removed U1: 609-3706-1-ND-MALE, RoboJackets-Connectors:609-3706-1-ND-MALE
- added J2: SBH11-PBPC-D05-RA, RoboJackets-Connectors:SBH11-PBPC-D05-RA
- added LED1, LED2: (no value), led:LED3MM
- added R1, R2: (no value), resistor:R-US_R0603
Connections:
- net N$1 renamed D-
- net N$2 renamed D+
- removed net !CS: KIT1.P29, U1.2
- removed net GPIO0: U1.4
- removed net GPIO3: U1.7
- removed net IRQ: KIT1.P10, U1.5
- removed net VCC: KIT1.VO, U1.10, U1.9
- new net !CS!-RADIO: J2.10, KIT1.P29
- new net !RST!-RADIO: J2.5, KIT1.P23
- new net +3.3V: J2.6, KIT1.VO, LED1.A, LED2.A
- new net INT-RADIO: J2.3, KIT1.P10
- new net LED1: KIT1.P25, R1.1
- new net LED2: KIT1.P24, R2.1
- new net N$1: LED1.C, R1.2
- new net N$2: LED2.C, R2.2
- net GND: now also J2.7; no longer U1.8
- net MISO: now also J2.8; no longer U1.6
- net MOSI: now also J2.2; no longer U1.3
- net SCK: now also J2.1; no longer U1.1
Other:
- note added: "Enclosure used: Serpac A21,BK (Digikey: SRA21B-ND)"
- moved on the sheet: J1, KIT1
