File: boards/kicker-3.2/kicker.sch (EAGLE design)
At the start: 144 parts, among them J1 B2PS-VH(LF)(SN), J2 B2PS-VH(LF)(SN), J3 B2PS-VH(LF)(SN), J4 HFW8R-1ST, J5 2-PIN_2MM-H, J6 3-PIN_2MM-H, J7 !BTN_KCK_PRE_EXT, J8 !BTN_CHP_PRE_EXT, J9 !BTN_CHG_PRE_EXT, Q1 ATP302ATPAK, Q10 BSS806NSOT-23-3, Q2 IRFS4227, Q3 IXGK400N30A3, Q4 IXGK400N30A3, Q5 BSS127, Q6 AOD1N60, Q7 BSS127, Q8 BSS127, Q9 BSS127, T1 DA203X-ALDA2034, U1 MPM3620GQV-P, U2 15V, U3 LT3751FE, U4 IX4427N, U5 AT32ATQFP44, U6 ADUM744XARQZ-RL7, U7 ADUM744XCRQZ-RL7

Commit message: passing core fixes
Parts:
- R2, R3, R4: device rcl:R-US_R0402 -> rcl:R-US_R0603
- R47: value 50 -> 51
- U6: value ADUM744XARQZ-RL7 -> ADUM7441ARQZ-RL7
- U7: value ADUM744XCRQZ-RL7 -> ADUM7441CRQZ-RL7
Connections:
- removed net N$2: U7.V_IA
- net CHARGE: no longer C25.1
- net CHARGE_RAW: now also C25.1
- net GND: now also U7.V_IA
Other:
- moved on the sheet: C25, R24
Changed lines of the file:
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@@
 <?xml version="1.0" encoding="utf-8"?>
 <!DOCTYPE eagle SYSTEM "eagle.dtd">
-<eagle version="9.3.2">
+<eagle version="9.4.2">
 <drawing>
 <settings>
@@
 <attribute name="REV" value="3.1"/>
 </part>
-<part name="R47" library="rcl" deviceset="R-US_" device="R0603" value="50"/>
+<part name="R47" library="rcl" deviceset="R-US_" device="R0603" value="51"/>
 <part name="R48" library="rcl" deviceset="R-US_" device="R0603" value="10k"/>
 <part name="SUPPLY95" library="supply2" deviceset="GND" device=""/>
@@
 <part name="D19" library="RoboJackets-LEDs" deviceset="LED-SMD" device="" technology="-RED" value="RED"/>
 <part name="Q9" library="RoboJackets-Discrete" deviceset="BSS127" device=""/>
-<part name="R44" library="rcl" library_urn="urn:adsk.eagle:library:334" deviceset="R-US_" device="R0603" package3d_urn="urn:adsk.eagle:package:23555/2" value="330"/>
+<part name="R44" library="rcl" library_urn="urn:adsk.eagle:library:334" deviceset="R-US_" device="R0603" package3d_urn="urn:adsk.eagle:package:23555/3" value="330"/>
 <part name="SUPPLY89" library="supply2" library_urn="urn:adsk.eagle:library:372" deviceset="+5V" device=""/>
 <part name="Q8" library="RoboJackets-Discrete" deviceset="BSS127" device=""/>
-<part name="R43" library="rcl" library_urn="urn:adsk.eagle:library:334" deviceset="R-US_" device="R0603" package3d_urn="urn:adsk.eagle:package:23555/2" value="1k"/>
+<part name="R43" library="rcl" library_urn="urn:adsk.eagle:library:334" deviceset="R-US_" device="R0603" package3d_urn="urn:adsk.eagle:package:23555/3" value="1k"/>
 <part name="D20" library="RoboJackets-LEDs" deviceset="LED-SMD" device="" technology="-YELLOW" value="YELLOW"/>
 <part name="SUPPLY91" library="supply2" deviceset="V+" device=""/>
@@
 <part name="U1" library="RoboJackets-PowerICs" deviceset="MPM3620GQV-P" device=""/>
 <part name="C1" library="rcl" library_urn="urn:adsk.eagle:library:334" deviceset="C-US" device="C1206" package3d_urn="urn:adsk.eagle:package:23618/2" value="10uF 50V"/>
-<part name="R2" library="rcl" library_urn="urn:adsk.eagle:library:334" deviceset="R-US_" device="R0402" package3d_urn="urn:adsk.eagle:package:23547/2" value="100k"/>
+<part name="R2" library="rcl" library_urn="urn:adsk.eagle:library:334" deviceset="R-US_" device="R0603" package3d_urn="urn:adsk.eagle:package:23555/3" value="100k"/>
 <part name="SUPPLY4" library="supply2" deviceset="GND" device=""/>
-<part name="R1" library="rcl" library_urn="urn:adsk.eagle:library:334" deviceset="R-US_" device="R0603" package3d_urn="urn:adsk.eagle:package:23555/2" value="43.2k 1%"/>
-<part name="R3" library="rcl" library_urn="urn:adsk.eagle:library:334" deviceset="R-US_" device="R0402" package3d_urn="urn:adsk.eagle:package:23547/2" value="160k 1%"/>
-<part name="R4" library="rcl" library_urn="urn:adsk.eagle:library:334" deviceset="R-US_" device="R0402" package3d_urn="urn:adsk.eagle:package:23547/2" value="30.1k 1%"/>
+<part name="R1" library="rcl" library_urn="urn:adsk.eagle:library:334" deviceset="R-US_" device="R0603" package3d_urn="urn:adsk.eagle:package:23555/3" value="43.2k 1%"/>
+<part name="R3" library="rcl" library_urn="urn:adsk.eagle:library:334" deviceset="R-US_" device="R0603" package3d_urn="urn:adsk.eagle:package:23555/3" value="160k 1%"/>
+<part name="R4" library="rcl" library_urn="urn:adsk.eagle:library:334" deviceset="R-US_" device="R0603" package3d_urn="urn:adsk.eagle:package:23555/3" value="30.1k 1%"/>
 <part name="C2" library="rcl" library_urn="urn:adsk.eagle:library:334" deviceset="C-US" device="C0603" package3d_urn="urn:adsk.eagle:package:23616/2" value="22uF 10V"/>
 <part name="SUPPLY3" library="supply2" deviceset="GND" device=""/>
@@
 <part name="SUPPLY68" library="supply2" deviceset="GND" device=""/>
 <part name="SUPPLY67" library="supply2" deviceset="GND" device=""/>
-<part name="U7" library="RoboJackets-ICs" deviceset="ADUM744X*RQZ-RL7" device="" package3d_urn="urn:adsk.eagle:package:12284950/1" technology="C"/>
-<part name="U6" library="RoboJackets-ICs" deviceset="ADUM744X*RQZ-RL7" device="" package3d_urn="urn:adsk.eagle:package:12284950/1" technology="A"/>
+<part name="U7" library="RoboJackets-ICs" deviceset="ADUM744X*RQZ-RL7" device="" package3d_urn="urn:adsk.eagle:package:12284950/1" technology="C" value="ADUM7441CRQZ-RL7"/>
+<part name="U6" library="RoboJackets-ICs" deviceset="ADUM744X*RQZ-RL7" device="" package3d_urn="urn:adsk.eagle:package:12284950/1" technology="A" value="ADUM7441ARQZ-RL7"/>
 <part name="SUPPLY72" library="supply2" deviceset="GND" device=""/>
 <part name="SUPPLY71" library="supply2" deviceset="+5V" device=""/>
@@
 <attribute name="VALUE" x="74.676" y="150.749" size="1.778" layer="96"/>
 </instance>
-<instance part="R24" gate="G$1" x="165.1" y="180.34" smashed="yes" rot="R180">
-<attribute name="NAME" x="168.91" y="178.8414" size="1.778" layer="95" rot="R180"/>
-<attribute name="VALUE" x="168.91" y="183.642" size="1.778" layer="96" rot="R180"/>
-</instance>
-<instance part="C25" gate="G$1" x="175.26" y="172.72" smashed="yes">
-<attribute name="NAME" x="176.276" y="173.355" size="1.778" layer="95"/>
-<attribute name="VALUE" x="176.276" y="168.529" size="1.778" layer="96"/>
-</instance>
-<instance part="SUPPLY39" gate="GND" x="175.26" y="157.48" smashed="yes">
-<attribute name="VALUE" x="173.355" y="154.305" size="1.778" layer="96"/>
+<instance part="R24" gate="G$1" x="177.8" y="180.34" smashed="yes" rot="R180">
+<attribute name="NAME" x="181.61" y="178.8414" size="1.778" layer="95" rot="R180"/>
+<attribute name="VALUE" x="181.61" y="183.642" size="1.778" layer="96" rot="R180"/>
+</instance>
+<instance part="C25" gate="G$1" x="167.64" y="172.72" smashed="yes">
+<attribute name="NAME" x="168.656" y="173.355" size="1.778" layer="95"/>
+<attribute name="VALUE" x="168.656" y="168.529" size="1.778" layer="96"/>
+</instance>
+<instance part="SUPPLY39" gate="GND" x="167.64" y="157.48" smashed="yes">
+<attribute name="VALUE" x="165.735" y="154.305" size="1.778" layer="96"/>
 </instance>
 <instance part="R23" gate="G$1" x="154.94" y="170.18" smashed="yes" rot="R90">
@@
 <segment>
 <pinref part="R24" gate="G$1" pin="2"/>
-<wire x1="160.02" y1="180.34" x2="154.94" y2="180.34" width="0.1524" layer="91"/>
+<wire x1="172.72" y1="180.34" x2="167.64" y2="180.34" width="0.1524" layer="91"/>
 <label x="139.7" y="180.34" size="1.27" layer="95" rot="R180" xref="yes"/>
 <pinref part="R23" gate="G$1" pin="2"/>
+<wire x1="167.64" y1="180.34" x2="154.94" y2="180.34" width="0.1524" layer="91"/>
 <wire x1="154.94" y1="180.34" x2="139.7" y2="180.34" width="0.1524" layer="91"/>
 <wire x1="154.94" y1="175.26" x2="154.94" y2="180.34" width="0.1524" layer="91"/>
 <junction x="154.94" y="180.34"/>
+<pinref part="C25" gate="G$1" pin="1"/>
+<wire x1="167.64" y1="175.26" x2="167.64" y2="180.34" width="0.1524" layer="91"/>
+<junction x="167.64" y="180.34"/>
 </segment>
 </net>
@@
 <segment>
 <pinref part="R24" gate="G$1" pin="1"/>
-<wire x1="170.18" y1="180.34" x2="175.26" y2="180.34" width="0.1524" layer="91"/>
 <label x="185.42" y="180.34" size="1.27" layer="95" rot="MR180" xref="yes"/>
-<pinref part="C25" gate="G$1" pin="1"/>
-<wire x1="175.26" y1="180.34" x2="185.42" y2="180.34" width="0.1524" layer="91"/>
-<wire x1="175.26" y1="175.26" x2="175.26" y2="180.34" width="0.1524" layer="91"/>
-<junction x="175.26" y="180.34"/>
+<wire x1="182.88" y1="180.34" x2="185.42" y2="180.34" width="0.1524" layer="91"/>
 </segment>
 </net>
@@
 <segment>
 <pinref part="C25" gate="G$1" pin="2"/>
-<wire x1="175.26" y1="167.64" x2="175.26" y2="160.02" width="0.1524" layer="91"/>
+<wire x1="167.64" y1="167.64" x2="167.64" y2="160.02" width="0.1524" layer="91"/>
 <pinref part="SUPPLY39" gate="GND" pin="GND"/>
 </segment>
@@
 </instance>
 <instance part="U7" gate="G$1" x="220.98" y="137.16" smashed="yes">
-<attribute name="NAME" x="209.55" y="156.21" size="2.54" layer="95"/>
-<attribute name="VALUE" x="209.55" y="123.19" size="2.54" layer="96" align="top-left"/>
+<attribute name="NAME" x="209.55" y="156.21" size="1.778" layer="95"/>
+<attribute name="VALUE" x="209.55" y="123.19" size="1.778" layer="96" align="top-left"/>
 </instance>
 <instance part="U6" gate="G$1" x="220.98" y="180.34" smashed="yes">
-<attribute name="NAME" x="209.55" y="199.39" size="2.54" layer="95"/>
-<attribute name="VALUE" x="209.55" y="166.37" size="2.54" layer="96" align="top-left"/>
+<attribute name="NAME" x="209.55" y="199.39" size="1.778" layer="95"/>
+<attribute name="VALUE" x="209.55" y="166.37" size="1.778" layer="96" align="top-left"/>
 </instance>
 <instance part="SUPPLY72" gate="GND" x="259.08" y="83.82" smashed="yes">
@@
 <junction x="144.78" y="104.14"/>
 <pinref part="SUPPLY66" gate="GND" pin="GND"/>
+</segment>
+<segment>
+<pinref part="SUPPLY68" gate="GND" pin="GND"/>
+<wire x1="203.2" y1="147.32" x2="180.34" y2="147.32" width="0.1524" layer="91"/>
+<wire x1="180.34" y1="147.32" x2="180.34" y2="144.78" width="0.1524" layer="91"/>
+<pinref part="U7" gate="G$1" pin="V_IA"/>
 </segment>
 </net>
@@
 </segment>
 </net>
-<net name="N$2" class="0">
-<segment>
-<pinref part="SUPPLY68" gate="GND" pin="GND"/>
-<wire x1="203.2" y1="147.32" x2="180.34" y2="147.32" width="0.1524" layer="91"/>
-<wire x1="180.34" y1="147.32" x2="180.34" y2="144.78" width="0.1524" layer="91"/>
-<pinref part="U7" gate="G$1" pin="V_IA"/>
-</segment>
-</net>

Commit message: final fixes and docs
Parts:
- removed C38, C39: 0.1uF, rcl:C-USC0603
- added C17, C18: 1uF, rcl:C-USC0603
- added R53: 10k, rcl:R-US_R0603
- C19: value 1uF -> 560uF; device rcl:C-USC0603 -> rcl:CPOL-USE7.5-18
- C20, C25: value 1uF -> 10uF (X7R); device rcl:C-USC0603 -> rcl:C-USC1210
- C21: value 560uF -> 10uF (X7R); device rcl:CPOL-USE7.5-18 -> rcl:C-USC1210
- C22: value 10uF (X7R) -> 1uF; device rcl:C-USC1210 -> rcl:C-USC0603
- C26: value 10uF (X7R) -> 0.1uF 35V; device rcl:C-USC1210 -> rcl:C-USC0603
- C27: value 10uF (X7R) -> 22uF 35V; device rcl:C-USC1210 -> rcl:C-USC0805
- C28: value 0.1uF 35V -> 0.1uF 50V
- C29: value 22uF 35V -> 0.1uF 50V; device rcl:C-USC0805 -> rcl:C-USC0603
- C30, C31: value 0.1uF 50V -> 0.1uF
- R17: value 187k -> 505k 0.1%; device rcl:R-US_R1206 -> rcl:R-US_R0603
- R18: value 931 -> 113k 0.1%; device rcl:R-US_R0805 -> rcl:R-US_R0603
- R19: value 100k -> 3.0k 0.1%
- R21, R24: value 160 -> 100k
- R23: value 100k -> 160
- R25: value 10k -> 160
- R27: value 160 -> 10k; device rcl:R-US_R1206 -> rcl:R-US_R0603
- R29: value 270k -> 160; device rcl:R-US_R0603 -> rcl:R-US_R1206
- R30: value 100k -> 270k
- R31: value ERJ-6GEYJ515V -> 100k; device rcl:R-US_R0805 -> rcl:R-US_R0603
- R33: value 1.5k 35W -> ERJ-6GEYJ515V; device RoboJackets-Resistors:PWR263S-35TO-263AB -> rcl:R-US_R0805
- R34: value 10k -> 1.5k 35W; device rcl:R-US_R0603 -> RoboJackets-Resistors:PWR263S-35TO-263AB
- R35: value ERJ-6GEYJ515V -> 10k; device rcl:R-US_R0805 -> rcl:R-US_R0603
- R37: value RC0603FR-07205KL -> ERJ-6GEYJ515V; device rcl:R-US_R0603 -> rcl:R-US_R0805
- R38: value 10k -> RC0603FR-07205KL
- R40: value 1k -> 10k
- R41, R44: value 330 -> 1k
- R43: value 1k -> 330
- R45: value ERJ-P06J274V -> 330; device rcl:R-US_R0805 -> rcl:R-US_R0603
- R46: value 60 -> ERJ-P06J274V; device rcl:R-US_R0603 -> rcl:R-US_R0805
- R47: value 51 -> 60
- R48: value 10k -> 51
Connections:
- new net N$2: R17.2, R18.1
- net !BTN_CHG: now also R53.1; no longer R52.1
- net !BTN_CHP: now also R51.1; no longer R50.1
- net !BTN_KCK: now also R52.1; no longer R51.1
- net !DONE!: now also C17.1, R22.1; no longer C19.1, R21.1
- net !DONE!_RAW: now also R20.1, R22.2; no longer R19.1, R21.2
- net !FAULT!: now also C18.1, R23.1; no longer C20.1, R22.1
- net !FAULT!_RAW: now also R21.1, R23.2; no longer R20.1, R22.2
- net !RESET: now also R35.1; no longer R34.1
- net +15.0V: now also C26.2, C27.2, R41.2; no longer C28.2, C29.2, R40.2
- net +5V: now also C30.2, C31.2, C36.2, C37.2, R21.2, R35.2, R45.2, R49.2, R53.2; no longer C34.2, C35.2, C38.2, C39.2, R19.2, R34.2, R41.2, R48.2, R50.2
- net 15V_PWR_BR: now also R41.1; no longer R40.1
- net BALL_SENSE: now also R47.2; no longer R46.2
- net BALL_SENSE_CL: now also R47.1; no longer R46.1
- net BB_RX: now also R49.1; no longer R48.1
- net BB_TX_CL: now also R48.2; no longer R47.2
- net CHARGE: now also R25.1; no longer R24.1
- net CHARGE_RAW: now also C22.1, R25.2; no longer C25.1, R23.2
- net CHIP: now also R40.2; no longer R39.2
- net CHIP_GATE: now also R26.2, R28.1; no longer R25.2, R27.1
- net CHIP_GATE_S: now also C28.1, R28.2; no longer C30.1, R27.2
- net DISCHARGE_DRAIN: now also R34.PIN2; no longer R33.PIN2
- net FAULT_INV_BR: now also R44.1; no longer R43.1
- net GND: now also C17.2, C18.2, C19.-, C21.2, C26.1, C27.1, C28.2, C29.2, C30.1, C31.1, C36.1, C37.1, R19.2, R24.1, R27.1, R31.1, R40.1; no longer C19.2, C21.-, C26.2, C27.2, C28.1, C29.1, C30.2, C31.2, C34.1, C35.1, C38.1, C39.1, R18.2, R23.1, R25.1, R30.1, R37.1
- net GND_LGC_EXT: now also C34.1, C35.1; no longer C36.1, C37.1
- net HV_FB: now also R18.2, R19.1; no longer R17.2, R18.1
- net HV_SENSE_DIV_BR: now also R36.1, R37.2; no longer R35.1, R36.2
- net KICK: now also R39.2; no longer R38.2
- net KICK_GATE: now also R27.2, R29.1; no longer R26.2, R28.1
- net KICK_GATE_S: now also C29.1, R29.2; no longer C31.1, R28.2
- net MODE_SELECT: now also R50.2; no longer R49.2
- net N$14: now also R50.1; no longer R49.1
- net N$20: now also R42.1; no longer R41.1
- net N$27: now also R45.1; no longer R44.1
- net N$29: now also R46.1; no longer R45.1
- net N$3: now also R48.1; no longer R47.1
- net N$5: now also R43.1; no longer R42.1
- net QD_GATE_CTRL: now also R30.1, R31.2; no longer R29.1, R30.2
- net QD_PU_BR: now also R32.1, R33.2; no longer R31.1, R32.2
- net QUICK_DISCHARGE: now also R33.1; no longer R32.1
- net V+: now also R32.2, R34.PIN1, R36.2, R46.2; no longer R31.2, R33.PIN1, R35.2, R45.2
- net VBATT: now also C19.+, C20.1, C21.1, C25.1, R30.2; no longer C21.+, C22.1, C26.1, C27.1, R29.2
- net VCC_LGC_EXT: now also C34.2, C35.2; no longer C36.2, C37.2
- net VMON: now also R37.1, R38.2; no longer R36.1, R37.2
Other:
- note added: "Desolder FBH and jump FBL->GND to enter capacitor charging mode. This is recommended."
- note added: "Double Zener/TVS protection internal to ATP302"
- note added: "FBH=((Vout-1.22)^2)/(Pd) FBH=((250-1.22)^2)/0.1) FBH=618.9kOhm FBL=(1.22/(Vout-1.22))*FBH FBL=(1.22/(250-1.22))*618900 FBL=3.0kOhm"
- note added: "This is a fairly dense bit, so an explanation is here. The IZ4427N is a FET gate drive. It turns a weakly driven lower voltage from the MCU into a strong high voltage signal that can quickly open a FET or IGBT. Next in line is a pull-down that prevents the gate from floating if the IC is powering up of the input is floating. The small valued resistor and following capacitor act as a snubber, prev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"
- note removed: "Desolder R17 and jump R18 to enter capacitor charging mode. This is recommended."
- moved on the sheet: C20, C22, C23, C24, C25, C28, C29, C32, C33, C34, C35, C36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
