File: boards/other/motortester-v1.0/motortester.sch (EAGLE design)
At the start: 16 parts, among them IC1 MEGA32-A, IC2 LM50, IC3 LM50, IC4 LM50

Commit message: Fixed motor tester issues
Parts:
- removed SV1: (no value), con-lstb:MA08-1
- added J1: MKS-1658, RoboJackets-Connectors:MKS-1658
- IC1: device atmel:MEGA32-A -> RoboJackets-ICs:MEGA32-A
- SV2: device con-lstb:MA04-1 -> RoboJackets-Connectors:MA04-1
- U$1: device HD44780LCD:LCD-HD447804-HOLES20X4-4HOLES -> RoboJackets-Boards:LCD-HD447804-HOLES20X4-4HOLES
Connections:
- net GND: now also J1.2; no longer SV1.2
- net H1: now also J1.1; no longer SV1.1
- net H2: now also J1.3; no longer SV1.3
- net H3: now also J1.5; no longer SV1.5
- net PHASEA: now also J1.7; no longer SV1.7
- net PHASEB: now also J1.8; no longer SV1.8
- net PHASEC: now also J1.6; no longer SV1.6
- net VCC: now also J1.4; no longer SV1.4
