File: boards/whiskers-breakouts-1.0/VL6180X_Design.brd (EAGLE design)
At the start: 80 x 37 mm, 19 parts, among them J2 6-PIN_2MM-V, Q3 BSS138, Q4 BSS138, U1 VL6180X, U2 MIC5225_2.8V, U3 VL6180X, U4 VL6180X

Commit message: Update VL6180X_Design.brd
Routing:
- net GND: track 23.0 -> 24.7 mm, vias 10 -> 11
Other:
- board size 80 x 37 mm -> 73 x 33 mm
Changed lines of the file:
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@@
 <board>
 <plain>
-<wire x1="16" y1="35" x2="96" y2="35" width="0" layer="20"/>
-<wire x1="96" y1="35" x2="96" y2="72" width="0" layer="20"/>
-<wire x1="96" y1="72" x2="16" y2="72" width="0" layer="20"/>
-<wire x1="16" y1="72" x2="16" y2="35" width="0" layer="20"/>
+<wire x1="19" y1="37" x2="92" y2="37" width="0" layer="20"/>
+<wire x1="92" y1="37" x2="92" y2="70" width="0" layer="20"/>
+<wire x1="92" y1="70" x2="19" y2="70" width="0" layer="20"/>
+<wire x1="19" y1="70" x2="19" y2="37" width="0" layer="20"/>
 </plain>
 <attributes>
@@
 <wire x1="87" y1="46.7" x2="86.875" y2="46.825" width="0.3" layer="1"/>
 <wire x1="86.875" y1="46.825" x2="86.875" y2="48.8" width="0.3" layer="1"/>
-<wire x1="68.8" y1="57.6" x2="62.94" y2="57.86" width="0" layer="19" extent="1-1"/>
-<wire x1="26.875" y1="48.8" x2="24.625" y2="48.8" width="0" layer="19" extent="1-1"/>
+<wire x1="62.94" y1="57.86" x2="61.24" y2="57.86" width="0.3" layer="1"/>
+<wire x1="61.24" y1="57.86" x2="61.2" y2="57.9" width="0.3" layer="1"/>
+<via x="61.2" y="57.9" extent="1-16" drill="0.35"/>
+<wire x1="24.625" y1="48.8" x2="26.875" y2="48.8" width="0" layer="19" extent="1-1"/>
 </signal>
 <signal name="+3.3V">
