File: boards/off-robot/battery-status-v2.0/Battery Status Device 2.0 organized.sch (EAGLE design)
At the start: 43 parts, among them IC1 4511D, IC2 4511D, IC3 4511D, J1 6PIN-0353620650, U1 AP1509-50SG-13

Commit message: Add files via upload
Parts:
- added C3, C4, C5, C6, C7: 10uF, rcl:C-USC0805
- added D2-R8: 330, RoboJackets-Resistors:R330-0603-1/10W-5%
- added JP1: (no value), pinhead:PINHD-2X4
- added T1, T2, T3, T4, T5: BC846, transistor:BC846
- added VD1: 35k, RoboJackets-Resistors:RESISTOR-0603-1/10W-5%
- added VD10, VD7: 20.0k, RoboJackets-Resistors:RESISTOR-0603-1/10W-5%
- added VD2, VD4: 10k, RoboJackets-Resistors:RESISTOR-0603-1/10W-5%
- added VD3: 50k, RoboJackets-Resistors:RESISTOR-0603-1/10W-5%
- added VD5: 71.5k, RoboJackets-Resistors:RESISTOR-0603-1/10W-5%
- added VD6: 11k, RoboJackets-Resistors:RESISTOR-0603-1/10W-5%
- added VD8, VD9: 10.0k, RoboJackets-Resistors:RESISTOR-0603-1/10W-5%
Connections:
- removed net 18V: C1.1, U1.VIN
- new net !RESET!: JP1.4
- new net 11.1V: J1.3, T1.C
- new net 14.8V: J1.2, T2.C
- new net 18.5V: J1.1, T3.C, U$1.1, U$1.4
- new net 18.5VB: F1.1, U$1.2, U$1.3
- new net 18.5VF: C1.1, F1.2, U1.VIN
- new net 3.7V: J1.5, T5.C
- new net 7.4V: J1.4, T4.C
- new net A1: D1-R1.2, U$3.P7-A
- new net A2: D2-R1.2, U$4.P7-A
- new net A3: D3-R1.2, U$5.P7-A
- new net AN1: C7.1, U$2.PINS10, VD10.2, VD9.1
- new net AN2: C6.1, U$2.PINS11, VD7.1, VD8.2
- new net AN3: C3.1, U$2.PINS12, VD1.1, VD2.2
- new net AN4: C4.1, U$2.PINS13, VD3.1, VD4.2
- new net AN5: C5.1, U$2.PINS14, VD5.1, VD6.2
- new net B1: D1-R2.2, U$3.P6-B
- new net B2: D2-R2.2, U$4.P6-B
- new net B3: D3-R2.2, U$5.P6-B
- new net C1: D1-R3.2, U$3.P4-C
- new net C2: D2-R3.2, U$4.P4-C
- new net C3: D3-R3.2, U$5.P4-C
- new net D1: D1-R4.2, U$3.P2-D
- new net D2: D2-R4.2, U$4.P2-D
- new net D3: D3-R4.2, U$5.P2-D
- new net DI1: LED1.A, U$2.PINS1
- new net DI10: IC2A.IB, U$2.PINS16
- new net DI11: IC2A.IC, U$2.PINS17
- new net DI12: IC2A.ID, U$2.PINS22
- new net DI13: D2-R8.2, U$2.PINS9
- new net DI14: IC3A.IA, U$2.PINS23
- new net DI15: IC3A.IB, U$2.PINS24
- new net DI16: IC3A.IC, U$2.PINS25
- new net DI17: IC3A.ID, U$2.PINS26
- new net DI2: LED2.A, U$2.PINS2
- new net DI3: LED3.A, U$2.PINS3
- new net DI4: U$2.PINS4, XTAL1.1
- new net DI5: IC1A.IA, U$2.PINS5
- new net DI6: IC1A.IB, U$2.PINS6
- new net DI7: IC1A.IC, U$2.PINS7
- new net DI8: IC1A.ID, U$2.PINS8
- new net DI9: IC2A.IA, U$2.PINS15
- new net E1: D1-R5.2, U$3.P1-E
- new net E2: D2-R5.2, U$4.P1-E
- new net E3: D3-R5.2, U$5.P1-E
- new net F1: D1-R6.2, U$3.P9-F
- new net F2: D2-R6.2, U$4.P9-F
- new net F3: D3-R6.2, U$5.P9-F
- new net G1: D1-R7.2, U$3.P10-G
- new net G2: D2-R7.2, U$4.P10-G
- new net G3: D3-R7.2, U$5.P10-G
- new net MISO: JP1.1
- new net MOSI: JP1.2
- new net N$10: D1-R5.1, IC1A.E
- new net N$11: D1-R7.1, IC1A.G
- new net N$12: D2-R1.1, IC2A.A
- new net N$13: D2-R2.1, IC2A.B
- new net N$14: D2-R3.1, IC2A.C
- new net N$15: D2-R4.1, IC2A.D
- new net N$16: D2-R5.1, IC2A.E
- new net N$17: D2-R6.1, IC2A.F
- new net N$18: D2-R7.1, IC2A.G
- new net N$19: D3-R1.1, IC3A.A
- new net N$2: LED1-R1.2, LED1.C
- new net N$20: D3-R2.1, IC3A.B
- new net N$21: D3-R3.1, IC3A.C
- new net N$22: D3-R4.1, IC3A.D
- new net N$23: D3-R5.1, IC3A.E
- new net N$24: D3-R6.1, IC3A.F
- new net N$25: D3-R7.1, IC3A.G
- new net N$26: D2-R8.1, U$4.P5-DP
- new net N$27: T5.E, VD9.2
- new net N$28: T4.E, VD7.2
- new net N$29: T1.E, VD1.2
- new net N$3: LED2-R1.2, LED2.C
- new net N$31: T2.E, VD3.2
- new net N$35: T3.E, VD5.2
- new net N$4: LED3-R1.2, LED3.C
- new net N$5: D1-R1.1, IC1A.A
- new net N$6: D1-R2.1, IC1A.B
- new net N$7: D1-R3.1, IC1A.C
- new net N$8: D1-R4.1, IC1A.D
- new net N$9: D1-R6.1, IC1A.F
- new net SCK: JP1.3
- net 3.3V: now also IC2A.BI, IC2A.LT, IC2P.VDD, IC3A.BI, IC3A.LT, IC3P.VDD, JP1.6, T1.B, T2.B, T3.B, T4.B, T5.B, U$2.PINS28
- net GND: now also C3.2, C4.2, C5.2, C6.2, C7.2, IC2A.LE, IC2P.VSS, IC3A.LE, IC3P.VSS, J1.6, JP1.5, LED1-R1.1, LED2-R1.1, LED3-R1.1, U$2.PINS19, U$2.PINS29, U$3.P3-GND, U$3.P8-GND, U$4.P3-GND, U$4.P8-GND, U$5.P3-GND, U$5.P8-GND, VD10.1, VD2.1, VD4.1, VD6.1, VD8.1, XTAL1.2
Other:
- note added: "Programming Header"
- moved on the sheet: IC2P, IC3P, LED1, LED1-R1, LED2, LED2-R1, LED3, LED3-R1, U$2, U$3

Commit message: Update Battery Status Device 2.0 organized.sch
Parts:
- added C10, C8: 10uF, rcl:C-USC0805
- added MOS-R1: 40.0k, RoboJackets-Resistors:RESISTOR-0603-1/10W-5%
- added MOS-R2: 10.0k, RoboJackets-Resistors:RESISTOR-0603-1/10W-5%
- added Q1: DMN65D8L-7, RoboJackets-Discrete:DMN65D8L-7
- D1-R1, D1-R2, D1-R3, D1-R4, D1-R5, D1-R6, D1-R7, D2-R1, D2-R2, D2-R3, D2-R4, D2-R5, D2-R6, D2-R7, D3-R1, D3-R2, D3-R3, D3-R4, D3-R5, D3-R6, D3-R7: value 330 -> 100
- D2-R8: value 330 -> 133
Connections:
- new net N$30: MOS-R1.1, MOS-R2.2, Q1.G
- new net N$32: F1.1, Q1.S
- net !RESET!: now also U$2.PINS26
- net 18.5V: now also Q1.D
- net 18.5VB: now also MOS-R1.2; no longer F1.1
- net 3.3V: now also C10.1, C8.1, U$2.PINS18
- net DI12: now also U$2.PINS21; no longer U$2.PINS22
- net DI14: now also U$2.PINS22; no longer U$2.PINS23
- net DI15: now also U$2.PINS23; no longer U$2.PINS24
- net DI16: now also U$2.PINS24; no longer U$2.PINS25
- net DI17: now also U$2.PINS25; no longer U$2.PINS26
- net DI6: now also U$2.PINS30; no longer U$2.PINS6
- net DI7: now also U$2.PINS31; no longer U$2.PINS7
- net DI8: now also U$2.PINS32; no longer U$2.PINS8
- net GND: now also C10.2, C8.2, MOS-R2.1
- net MISO: now also U$2.PINS7
- net MOSI: now also U$2.PINS6
- net SCK: now also U$2.PINS8
Other:
- note added: "MOSFET"
- note removed: "Fuse"
- moved on the sheet: F1, JP1, XTAL1
