File: boards/radio-v4.0/radio.sch (EAGLE design)
At the start: 29 parts, among them J2 SFW8, J3 FTSH-105-01-F-D-K, U1 ISM43340, U2 MPM3620GQV-P

Commit message: radio updates
Parts:
- added F1: 0805L200SLTHYR, RoboJackets-Fuses:CHIP_FUSE0805
Connections:
- new net PRE-FUSE: F1.1, R3.2, U2.OUT
- net +3.3V: now also F1.2; no longer R3.2, U2.OUT
Changed lines of the file:
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@@
 <part name="SUPPLY6" library="supply2" library_urn="urn:adsk.eagle:library:372" deviceset="GND" device=""/>
 <part name="J2" library="RoboJackets-Connectors" deviceset="SFW8" device=""/>
+<part name="F1" library="RoboJackets-Fuses" deviceset="CHIP_FUSE" device="0805" package3d_urn="urn:adsk.eagle:package:8760197/1" value="0805L200SLTHYR"/>
 </parts>
 <sheets>
@@
 <attribute name="VALUE" x="13.335" y="50.165" size="1.778" layer="96"/>
 </instance>
-<instance part="U1" gate="G$1" x="58.42" y="106.68" smashed="yes">
+<instance part="U1" gate="A" x="58.42" y="106.68" smashed="yes">
 <attribute name="NAME" x="26.67" y="156.21" size="1.778" layer="95"/>
 </instance>
@@
 <attribute name="VALUE" x="203.2" y="124.46" size="1.778" layer="96" font="vector"/>
 </instance>
+<instance part="F1" gate="G$1" x="99.06" y="238.76" smashed="yes">
+<attribute name="NAME" x="96.52" y="241.3" size="1.778" layer="95"/>
+<attribute name="VALUE" x="96.52" y="236.22" size="1.778" layer="96" align="top-left"/>
+</instance>
 </instances>
 <busses>
@@
 <net name="+3.3V" class="0">
 <segment>
-<pinref part="U2" gate="G$1" pin="OUT"/>
-<wire x1="81.28" y1="238.76" x2="93.98" y2="238.76" width="0.1524" layer="91"/>
-<pinref part="R3" gate="G$1" pin="2"/>
-<wire x1="93.98" y1="238.76" x2="93.98" y2="233.68" width="0.1524" layer="91"/>
-<wire x1="93.98" y1="238.76" x2="104.14" y2="238.76" width="0.1524" layer="91"/>
-<junction x="93.98" y="238.76"/>
 <wire x1="104.14" y1="238.76" x2="114.3" y2="238.76" width="0.1524" layer="91"/>
 <wire x1="114.3" y1="238.76" x2="114.3" y2="251.46" width="0.1524" layer="91"/>
 <pinref part="C11" gate="G$1" pin="1"/>
 <wire x1="104.14" y1="233.68" x2="104.14" y2="238.76" width="0.1524" layer="91"/>
-<junction x="104.14" y="238.76"/>
 <pinref part="C13" gate="G$1" pin="1"/>
 <wire x1="114.3" y1="233.68" x2="114.3" y2="238.76" width="0.1524" layer="91"/>
 <junction x="114.3" y="238.76"/>
 <pinref part="SUPPLY14" gate="P" pin="+3.3V"/>
+<pinref part="F1" gate="G$1" pin="2"/>
+<wire x1="101.6" y1="238.76" x2="104.14" y2="238.76" width="0.1524" layer="91"/>
+<junction x="104.14" y="238.76"/>
 </segment>
 <segment>
@@
 <junction x="15.24" y="149.86"/>
 <pinref part="SUPPLY1" gate="P" pin="+3.3V"/>
-<pinref part="U1" gate="G$1" pin="P02-VDD"/>
-<pinref part="U1" gate="G$1" pin="P14-VDD"/>
-<pinref part="U1" gate="G$1" pin="P15-VBAT"/>
+<pinref part="U1" gate="A" pin="P02-VDD"/>
+<pinref part="U1" gate="A" pin="P14-VDD"/>
+<pinref part="U1" gate="A" pin="P15-VBAT"/>
 </segment>
 <segment>
@@
 <junction x="15.24" y="93.98"/>
 <pinref part="SUPPLY2" gate="GND" pin="GND"/>
-<pinref part="U1" gate="G$1" pin="P01-GND"/>
-<pinref part="U1" gate="G$1" pin="P03-GND"/>
-<pinref part="U1" gate="G$1" pin="P17-GND"/>
-<pinref part="U1" gate="G$1" pin="P20-GND"/>
-<pinref part="U1" gate="G$1" pin="P35-GND"/>
-<pinref part="U1" gate="G$1" pin="P36-GND"/>
-<pinref part="U1" gate="G$1" pin="P37-GND"/>
-<pinref part="U1" gate="G$1" pin="P38-GND"/>
-<pinref part="U1" gate="G$1" pin="P39-GND"/>
-<pinref part="U1" gate="G$1" pin="P40-GND"/>
-<pinref part="U1" gate="G$1" pin="P41-GND"/>
-<pinref part="U1" gate="G$1" pin="P42-GND"/>
-<pinref part="U1" gate="G$1" pin="P43-GND"/>
-<pinref part="U1" gate="G$1" pin="P44-GND"/>
+<pinref part="U1" gate="A" pin="P01-GND"/>
+<pinref part="U1" gate="A" pin="P03-GND"/>
+<pinref part="U1" gate="A" pin="P17-GND"/>
+<pinref part="U1" gate="A" pin="P20-GND"/>
+<pinref part="U1" gate="A" pin="P35-GND"/>
+<pinref part="U1" gate="A" pin="P36-GND"/>
+<pinref part="U1" gate="A" pin="P37-GND"/>
+<pinref part="U1" gate="A" pin="P38-GND"/>
+<pinref part="U1" gate="A" pin="P39-GND"/>
+<pinref part="U1" gate="A" pin="P40-GND"/>
+<pinref part="U1" gate="A" pin="P41-GND"/>
+<pinref part="U1" gate="A" pin="P42-GND"/>
+<pinref part="U1" gate="A" pin="P43-GND"/>
+<pinref part="U1" gate="A" pin="P44-GND"/>
 </segment>
 <segment>
@@
 <wire x1="53.34" y1="160.02" x2="53.34" y2="162.56" width="0.1524" layer="91"/>
 <label x="53.34" y="162.56" size="1.27" layer="95" rot="R90" xref="yes"/>
-<pinref part="U1" gate="G$1" pin="P04-JTAG_TMS"/>
+<pinref part="U1" gate="A" pin="P04-JTAG_TMS"/>
 </segment>
 <segment>
@@
 <wire x1="55.88" y1="160.02" x2="55.88" y2="162.56" width="0.1524" layer="91"/>
 <label x="55.88" y="162.56" size="1.27" layer="95" rot="R90" xref="yes"/>
-<pinref part="U1" gate="G$1" pin="P05-JTAG_TCK"/>
+<pinref part="U1" gate="A" pin="P05-JTAG_TCK"/>
 </segment>
 <segment>
@@
 <wire x1="58.42" y1="160.02" x2="58.42" y2="162.56" width="0.1524" layer="91"/>
 <label x="58.42" y="162.56" size="1.27" layer="95" rot="R90" xref="yes"/>
-<pinref part="U1" gate="G$1" pin="P06-JTAG_TDI"/>
+<pinref part="U1" gate="A" pin="P06-JTAG_TDI"/>
 </segment>
 <segment>
@@
 <wire x1="60.96" y1="160.02" x2="60.96" y2="162.56" width="0.1524" layer="91"/>
 <label x="60.96" y="162.56" size="1.27" layer="95" rot="R90" xref="yes"/>
-<pinref part="U1" gate="G$1" pin="P07-JTAG_TDO"/>
+<pinref part="U1" gate="A" pin="P07-JTAG_TDO"/>
 </segment>
 <segment>
@@
 <wire x1="96.52" y1="111.76" x2="101.6" y2="111.76" width="0.1524" layer="91"/>
 <label x="101.6" y="111.76" size="1.27" layer="95" xref="yes"/>
-<pinref part="U1" gate="G$1" pin="P34-!RST!"/>
+<pinref part="U1" gate="A" pin="P34-!RST!"/>
 </segment>
 <segment>
@@
 <wire x1="96.52" y1="142.24" x2="101.6" y2="142.24" width="0.1524" layer="91"/>
 <label x="101.6" y="142.24" size="1.27" layer="95" xref="yes"/>
-<pinref part="U1" gate="G$1" pin="P09-SPI_MOSI/ADC_4"/>
+<pinref part="U1" gate="A" pin="P09-SPI_MOSI/ADC_4"/>
 </segment>
 <segment>
@@
 <wire x1="96.52" y1="137.16" x2="101.6" y2="137.16" width="0.1524" layer="91"/>
 <label x="101.6" y="137.16" size="1.27" layer="95" xref="yes"/>
-<pinref part="U1" gate="G$1" pin="P11-SPI_SCK/ADC_2"/>
+<pinref part="U1" gate="A" pin="P11-SPI_SCK/ADC_2"/>
 </segment>
 <segment>
@@
 <wire x1="96.52" y1="134.62" x2="101.6" y2="134.62" width="0.1524" layer="91"/>
 <label x="101.6" y="134.62" size="1.27" layer="95" xref="yes"/>
-<pinref part="U1" gate="G$1" pin="P12-SPI_!SS!/ADC_1"/>
+<pinref part="U1" gate="A" pin="P12-SPI_!SS!/ADC_1"/>
 </segment>
 </net>
@@
 <wire x1="96.52" y1="114.3" x2="101.6" y2="114.3" width="0.1524" layer="91"/>
 <label x="101.6" y="114.3" size="1.27" layer="95" xref="yes"/>
-<pinref part="U1" gate="G$1" pin="P13-SPI_DR/DR/ADC_0"/>
+<pinref part="U1" gate="A" pin="P13-SPI_DR/DR/ADC_0"/>
 </segment>
 </net>
@@
 <wire x1="96.52" y1="139.7" x2="101.6" y2="139.7" width="0.1524" layer="91"/>
 <label x="101.6" y="139.7" size="1.27" layer="95" xref="yes"/>
-<pinref part="U1" gate="G$1" pin="P10-SPI_MISO/ADC_3"/>
+<pinref part="U1" gate="A" pin="P10-SPI_MISO/ADC_3"/>
 </segment>
 </net>
@@
 <wire x1="96.52" y1="91.44" x2="101.6" y2="91.44" width="0.1524" layer="91"/>
 <label x="101.6" y="91.44" size="1.27" layer="95" xref="yes"/>
-<pinref part="U1" gate="G$1" pin="P26-GPIO_3"/>
+<pinref part="U1" gate="A" pin="P26-GPIO_3"/>
 </segment>
 <segment>
@@
 <wire x1="96.52" y1="88.9" x2="101.6" y2="88.9" width="0.1524" layer="91"/>
 <label x="101.6" y="88.9" size="1.27" layer="95" xref="yes"/>
-<pinref part="U1" gate="G$1" pin="P27-GPIO_4"/>
+<pinref part="U1" gate="A" pin="P27-GPIO_4"/>
 </segment>
 <segment>
@@
 <wire x1="96.52" y1="99.06" x2="101.6" y2="99.06" width="0.1524" layer="91"/>
 <label x="101.6" y="99.06" size="1.27" layer="95" xref="yes"/>
-<pinref part="U1" gate="G$1" pin="P23-GPIO_0"/>
+<pinref part="U1" gate="A" pin="P23-GPIO_0"/>
 </segment>
 <segment>
@@
 <wire x1="96.52" y1="96.52" x2="101.6" y2="96.52" width="0.1524" layer="91"/>
 <label x="101.6" y="96.52" size="1.27" layer="95" xref="yes"/>
-<pinref part="U1" gate="G$1" pin="P24-GPIO_1"/>
+<pinref part="U1" gate="A" pin="P24-GPIO_1"/>
 </segment>
 <segment>
@@
 </segment>
 </net>
+<net name="PRE-FUSE" class="0">
+<segment>
+<pinref part="R3" gate="G$1" pin="2"/>
+<wire x1="93.98" y1="238.76" x2="93.98" y2="233.68" width="0.1524" layer="91"/>
+<pinref part="U2" gate="G$1" pin="OUT"/>
+<wire x1="81.28" y1="238.76" x2="93.98" y2="238.76" width="0.1524" layer="91"/>
+<pinref part="F1" gate="G$1" pin="1"/>
+<wire x1="93.98" y1="238.76" x2="96.52" y2="238.76" width="0.1524" layer="91"/>
+<junction x="93.98" y="238.76"/>
+</segment>
+</net>
 </nets>
 </sheet>
 </sheets>
-<errors>
-</errors>
 </schematic>
 </drawing>

Commit message: Final radio revisions
Parts:
- removed C11: 22uF, rcl:C-USC1210
- removed C13: 0.1uF, rcl:C-USC0603
- removed D6: YELLOW, RoboJackets-LEDs:LED-SMD-YELLOW
- removed J3: FTSH-105-01-F-D-K, Jlink-Connector:FTSH-105-01-F-D-K
- removed R10: 200, resistor:R-US_R0603
- removed U2: MPM3620GQV-P, RoboJackets-PowerICs:MPM3620GQV-P
- added $$U1: ISM43340, RoboJackets-RF:ISM43340
- added C8: 10uF, rcl:C-USC0805
- added C9: 1uF, rcl:C-USC0603
- added J1: SFW8, RoboJackets-Connectors:SFW8
- C1: value 220uF -> 0.1uF; device RoboJackets-Capacitors:ECA-1HHG221 -> rcl:C-USC0603
- C2: value 10uF -> 10uF 16V; device rcl:C-USC0805 -> rcl:C-USC1210
- C3: value 10uF -> 22uF; device rcl:C-USC0805 -> rcl:C-USC1210
- C4: value 1uF -> 220uF; device rcl:C-USC0603 -> RoboJackets-Capacitors:ECA-1HHG221
- C5: value 0.1uF -> 10uF; device rcl:C-USC0603 -> rcl:C-USC0805
- C7: value 10uF 16V -> 0.1uF; device rcl:C-USC1210 -> rcl:C-USC0603
- D1: value GREEN -> RED; device RoboJackets-LEDs:LED-SMD-GREEN -> RoboJackets-LEDs:LED-SMD-RED
- D3: value RED -> GREEN; device RoboJackets-LEDs:LED-SMD-RED -> RoboJackets-LEDs:LED-SMD-GREEN
- D5: value GREEN -> YELLOW; device RoboJackets-LEDs:LED-SMD-GREEN -> RoboJackets-LEDs:LED-SMD-YELLOW
- J2: value SFW8 -> FTSH-105-01-F-D-K; device RoboJackets-Connectors:SFW8 -> Jlink-Connector:FTSH-105-01-F-D-K
- R1: value 88.7k 1% -> 100k
- R2: value 100k -> 88.7k 1%
- R3: value 143.0k 1% -> 45.3k 1%
- R4: value 45.3k 1% -> 143.0k 1%
- R5: value 1k -> 680
- R6: value 680 -> 1k
- U1: value ISM43340 -> MPM3620GQV-P; device RoboJackets-RF:ISM43340 -> RoboJackets-PowerICs:MPM3620GQV-P
Connections:
- removed net DBG_TLK_RAD: R8.1, U1.P24-GPIO_1
- removed net TLK: D4.A, R8.2
- net !CS!_RAD: now also $$U1.P12-SPI_!SS!/ADC_1, J1G$1.5; no longer J2G$1.5, U1.P12-SPI_!SS!/ADC_1
- net !RST!_GLB: now also $$U1.P34-!RST!, J1G$1.6, J2.2; no longer J2G$1.6, J3.2, U1.P34-!RST!
- net +3.3V: now also $$U1.P02-VDD, $$U1.P14-VDD, $$U1.P15-VBAT, C1.1, C4.11, C7.1, C8.1, C9.1, J2.1, R5.2; no longer C1.11, C11.1, C13.1, C2.1, C4.1, J3.1, R6.2, U1.P02-VDD, U1.P14-VDD, U1.P15-VBAT
- net +5.0V: now also C2.1, J1G$1.1, R1.1, R6.2, U1.IN; no longer C7.1, J2G$1.1, R2.1, R5.2, U2.IN
- net 3V3_PWR_IND: now also D4.A, R5.1; no longer D2.A, R6.1
- net 5V_PWR_IND: now also D3.A, R6.1; no longer D1.A, R5.1
- net AAM: now also R2.2, U1.AAM; no longer R1.2, U2.AAM
- net DBG_ACT_RAD: now also $$U1.P27-GPIO_4, R7.1; no longer R10.1, U1.P27-GPIO_4
- net DBG_ERR: now also D1.A, R9.2; no longer D3.A, R7.2
- net DBG_ERR_RAD: now also $$U1.P23-GPIO_0, R9.1; no longer R7.1, U1.P23-GPIO_0
- net DBG_LNK_RAD: now also $$U1.P26-GPIO_3, R8.1; no longer R9.1, U1.P26-GPIO_3
- net DGB_ACT: now also D5.A, R7.2; no longer D6.A, R10.2
- net DGB_LNK: now also D2.A, R8.2; no longer D5.A, R9.2
- net EN: now also R1.2, U1.EN; no longer R2.2, U2.EN
- net FB: now also R3.2, R4.1, U1.FB; no longer R3.1, R4.2, U2.FB
- net GND: now also $$U1.P01-GND, $$U1.P03-GND, $$U1.P17-GND, $$U1.P20-GND, $$U1.P35-GND, $$U1.P36-GND, $$U1.P37-GND, $$U1.P38-GND, $$U1.P39-GND, $$U1.P40-GND, $$U1.P41-GND, $$U1.P42-GND, $$U1.P43-GND, $$U1.P44-GND, C1.2, C4.22, C8.2, C9.2, J1G$1.2, J2.4, J2.5, J2.9, R2.1, R3.1, U1.AGND, U1.PGND; no longer C1.22, C11.2, C13.2, C4.2, D6.K, J2G$1.2, J3.4, J3.5, J3.9, R1.1, R4.1, U1.P01-GND, U1.P03-GND, U1.P17-GND, U1.P20-GND, U1.P35-GND, U1.P36-GND, U1.P37-GND, U1.P38-GND, U1.P39-GND, U1.P40-GND, U1.P41-GND, U1.P42-GND, U1.P43-GND, U1.P44-GND, U2.AGND, U2.PGND
- net INT_RAD: now also $$U1.P13-SPI_DR/DR/ADC_0, J1G$1.4; no longer J2G$1.4, U1.P13-SPI_DR/DR/ADC_0
- net MISO: now also $$U1.P10-SPI_MISO/ADC_3, J1G$1.3; no longer J2G$1.3, U1.P10-SPI_MISO/ADC_3
- net MOSI: now also $$U1.P09-SPI_MOSI/ADC_4, J1G$1.7; no longer J2G$1.7, U1.P09-SPI_MOSI/ADC_4
- net PRE-FUSE: now also R4.2, U1.OUT; no longer R3.2, U2.OUT
- net SCK: now also $$U1.P11-SPI_SCK/ADC_2, J1G$1.8; no longer J2G$1.8, U1.P11-SPI_SCK/ADC_2
- net TCK_RAD: now also $$U1.P05-JTAG_TCK, J2.7; no longer J3.7, U1.P05-JTAG_TCK
- net TDI_RAD: now also $$U1.P06-JTAG_TDI, J2.6; no longer J3.6, U1.P06-JTAG_TDI
- net TDO_RAD: now also $$U1.P07-JTAG_TDO, J2.10; no longer J3.10, U1.P07-JTAG_TDO
- net THERMAL_DNC: now also U1.SW; no longer U2.SW
- net TMS_RAD: now also $$U1.P04-JTAG_TMS, J2.3; no longer J3.3, U1.P04-JTAG_TMS
Other:
- note added: "ACT = activity (Indicates whether network traffic is flowing)"
- note added: "ERR = error (fucked)"
- note added: "LNK = link (indicates active connection to the router)"
- note added: "TLK = Arbitrary LED (technically means talk)"
- moved on the sheet: C2, C3, C5, C7, D1, D2, D3, D4, D5, R1, R2, R3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
