File: boards/on-robot/kicad/motorboard-v1.0/_autosave-motorboard-v1.0.kicad_pcb (KiCad board)
At the start: 4 copper layers, 306 parts, among them J1 52901-0274, J10 Conn_01x08, J11 XT60PW-M, J12 Conn_01x08, J13 39301080, J14 N2510-6002RB, J15 39301080, J16 N2510-6002RB, J17 39301080, J18 N2510-6002RB, J19 39301080, J2 52901-0274, J20 N2510-6002RB, J21 S8B-PH-SM4-TB, J3 52901-0274, J4 52901-0274, J5 XT30PW-M, J6 HFW8R-1STE1H1LF, J7 Conn_01x08, J8 Conn_01x08, J9 Conn_01x08, Q1 STD140N6F7, Q10 STD140N6F7, Q11 STD140N6F7, Q12 STD140N6F7, Q13 STD140N6F7, Q14 STD140N6F7, Q15 STD140N6F7, Q16 BSS123, Q17 BSS123, Q18 BSS123, Q19 STD140N6F7, Q2 STD140N6F7, Q20 STD140N6F7, Q21 STD140N6F7, Q22 STD140N6F7, Q23 STD140N6F7, Q24 STD140N6F7, Q25 BSS123, Q26 BSS123, Q27 BSS123, Q28 STD140N6F7, Q29 STD140N6F7, Q3 STD140N6F7, Q30 STD140N6F7, Q31 STD140N6F7, Q32 STD140N6F7, Q33 STD140N6F7, Q34 BSS123, Q35 BSS123, Q36 BSS123, Q37 STD140N6F7, Q38 STD140N6F7, Q39 STD140N6F7, Q4 STD140N6F7, Q40 STD140N6F7, Q41 STD140N6F7, Q42 STD140N6F7, Q43 BSS123, Q44 BSS123, Q45 BSS123, Q5 STD140N6F7, Q6 STD140N6F7, Q7 BSS123, Q8 BSS123, Q9 BSS123, SW1 TL1105VF100Q, U1 MC3486DR, U10 SN74LVC3G17DCTR, U11 STSPIN32F0A, U12 SN74LVC3G17DCTR, U13 SN74LVC3G17DCTR, U14 STSPIN32F0A, U15 SN74LVC3G17DCTR, U16 SN74LVC3G17DCTR, U17 STSPIN32F0A, U18 SN74LVC3G17DCTR, U19 SN74LVC3G17DCTR, U2 MC3486DR, U20 STSPIN32F0A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

Commit message: Status 10/29/2024
Edits made to overall motorboard schematic
Parts:
- Q1, Q3: moved to B.Cu
- moved C13 387.6 mm to (-345.8, 209.2)
- moved D1 387.6 mm to (-363.1, 257.4)
- moved R23 387.6 mm to (-385.9, 246.4)
- moved R24 387.6 mm to (-385.9, 248.9)
- moved R25 387.6 mm to (-385.9, 251.4)
- moved R26 387.6 mm to (-385.9, 254.0)
- moved R27 387.6 mm to (-385.9, 256.5)
- moved C10 387.6 mm to (-345.8, 201.7)
- moved C11 387.6 mm to (-345.8, 204.2)
- moved C12 387.6 mm to (-345.8, 206.7)
- moved C14 387.6 mm to (-345.8, 211.7)
- moved C16 387.6 mm to (-345.8, 216.8)
- moved C20 387.6 mm to (-367.7, 208.1)
- moved C21 387.6 mm to (-367.7, 211.4)
- moved C22 387.6 mm to (-367.7, 214.8)
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