File: boards/development/kicker-v3.4/hv_bank.kicad_sch (KiCad schematic)
At the start: 16 parts, among them Q3 AOD1N60, Q4 BSS127S

Commit message: some graphics
Other:
- moved on the sheet: D6, R20
Changed lines of the file:
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@@
 	(title_block
 		(title "High Voltage Cap Bank w/ Safety Auto Discharge")
-		(date "2026-02-24")
+		(date "2026-02-26")
 		(rev "3.4-dev")
 		(company "RoboJackets - RoboCup")
@@
 	)
 	(rectangle
-		(start 153.67 24.13)
-		(end 186.69 58.42)
+		(start 153.67 17.78)
+		(end 186.69 52.07)
 		(stroke
 			(width 0)
@@
 	(text "Safety Discharge Indicator"
 		(exclude_from_sim no)
-		(at 153.924 23.622 0)
+		(at 153.924 17.272 0)
 		(effects
 			(font
@@
 	(text "Only on when discharging"
 		(exclude_from_sim no)
-		(at 169.418 57.15 0)
+		(at 169.418 50.8 0)
 		(effects
 			(font
@@
 	(wire
 		(pts
-			(xy 162.56 30.48) (xy 162.56 29.21)
+			(xy 162.56 24.13) (xy 162.56 22.86)
 		)
 		(stroke
@@
 	(wire
 		(pts
-			(xy 162.56 38.1) (xy 162.56 40.64)
+			(xy 162.56 31.75) (xy 162.56 34.29)
 		)
 		(stroke
@@
 	(wire
 		(pts
-			(xy 162.56 48.26) (xy 162.56 54.61)
+			(xy 162.56 41.91) (xy 162.56 48.26)
 		)
 		(stroke
@@
 	)
 	(label "DISCHG_DRAIN"
-		(at 162.56 54.61 0)
+		(at 162.56 48.26 0)
 		(effects
 			(font
@@
 	(hierarchical_label "HV"
 		(shape bidirectional)
-		(at 162.56 29.21 180)
+		(at 162.56 22.86 180)
 		(effects
 			(font
@@
 	(symbol
 		(lib_id "Device:R")
-		(at 162.56 34.29 0)
+		(at 162.56 27.94 0)
 		(unit 1)
 		(exclude_from_sim no)
@@
 		(fields_autoplaced yes)
 		(property "Reference" "R20"
-			(at 165.1 33.0199 0)
+			(at 165.1 26.6699 0)
 			(effects
 				(font
@@
 		)
 		(property "Value" "270k"
-			(at 165.1 35.5599 0)
+			(at 165.1 29.2099 0)
 			(effects
 				(font
@@
 		)
 		(property "Footprint" "Resistor_SMD:R_0603_1608Metric"
-			(at 160.782 34.29 90)
+			(at 160.782 27.94 90)
 			(effects
 				(font
@@
 		)
 		(property "Datasheet" "~"
-			(at 162.56 34.29 0)
+			(at 162.56 27.94 0)
 			(effects
 				(font
@@
 		)
 		(property "Description" "Resistor"
-			(at 162.56 34.29 0)
+			(at 162.56 27.94 0)
 			(effects
 				(font
@@
 	(symbol
 		(lib_id "Device:LED")
-		(at 162.56 44.45 90)
+		(at 162.56 38.1 90)
 		(unit 1)
 		(exclude_from_sim no)
@@
 		(fields_autoplaced yes)
 		(property "Reference" "D6"
-			(at 166.37 44.7674 90)
+			(at 166.37 38.4174 90)
 			(effects
 				(font
@@
 		)
 		(property "Value" "HV_MID"
-			(at 166.37 47.3074 90)
+			(at 166.37 40.9574 90)
 			(effects
 				(font
@@
 		)
 		(property "Footprint" "LED_SMD:LED_0603_1608Metric"
-			(at 162.56 44.45 0)
+			(at 162.56 38.1 0)
 			(effects
 				(font
@@
 		)
 		(property "Datasheet" "~"
-			(at 162.56 44.45 0)
+			(at 162.56 38.1 0)
 			(effects
 				(font
@@
 		)
 		(property "Description" "Light emitting diode"
-			(at 162.56 44.45 0)
+			(at 162.56 38.1 0)
 			(effects
 				(font
@@
 		)
 		(property "Sim.Pins" "1=K 2=A"
-			(at 162.56 44.45 0)
-			(effects
-				(font
+			(at 162.56 38.1 0)
+			(effects
+				(font

Commit message: lock in part assignments
Parts:
- Q3: Manufacturer P/N (none) -> AOD1N60; Vendor P/N (none) -> 785-1179-1-ND
- Q4: Manufacturer P/N (none) -> BSS127S; Vendor P/N (none) -> BSS127S-7DICT-ND
Changed lines of the file:
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@@
+			)
+		)
+		(property "Manufacturer P/N" "BSS127S"
+			(at 41.91 48.26 0)
+			(effects
+				(font
+					(size 1.27 1.27)
+				)
+				(hide yes)
+			)
+		)
+		(property "Vendor P/N" "BSS127S-7DICT-ND"
+			(at 41.91 48.26 0)
+			(effects
+				(font
+					(size 1.27 1.27)
+				)
+				(hide yes)
 			)
 		)
@@
 			(at 124.46 41.91 0)
 			(effects
+				(font
+					(size 1.27 1.27)
+				)
+				(hide yes)
+			)
+		)
+		(property "Manufacturer P/N" "AOD1N60"
+			(at 124.46 41.91 0)
+			(effects
+				(font
+					(size 1.27 1.27)
+				)
+				(hide yes)
+			)
+		)
+		(property "Vendor P/N" "785-1179-1-ND"
+			(at 124.46 41.91 0)
+			(effects

Commit message: Production revision 2_26_26
Other:
- note added: "(Order 2/26/26) Replaced with 1.5k due to parts shortage This is only safe for charge voltage @ 200V or below. 3.3k is safe for up to 250V"
Changed lines of the file:
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@@
+		)
+	)
+	(text "(Order 2/26/26) Replaced with 1.5k due to parts shortage\nThis is only safe for charge voltage @ 200V or below.\n3.3k is safe for up to 250V"
+		(exclude_from_sim no)
+		(at 124.968 28.194 0)
+		(effects
+			(font
+				(size 1.27 1.27)
+				(color 255 0 0 1)
+			)
+			(justify right)
 		)
 	)
