File: boards/develop-2027/drive-motorboard/development/integration-test/enc_sense.kicad_sch (KiCad schematic)
At the start: 6 parts, among them J4 PROG SPI, U6 AS5047P

Commit message: Resolve all ERC, tweak formatting
Connections:
- net 3.3V_DEBUG renamed 3.3V DEBUG
Other:
- moved on the sheet: D14
Changed lines of the file:
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@@
 	(paper "A4")
 	(title_block
-		(date "2026-05-25")
+		(date "2026-07-16")
 		(rev "v1.0")
 		(company "Robojackets - RoboCup")
@@
 	)
 	(junction
+		(at 49.53 92.71)
+		(diameter 0)
+		(color 0 0 0 0)
+	)
+	(junction
 		(at 52.07 95.25)
 		(diameter 0)
@@
 	)
 	(junction
-		(at 49.53 92.71)
+		(at 50.8 25.4)
+		(diameter 0)
+		(color 0 0 0 0)
+	)
+	(junction
+		(at 36.83 25.4)
 		(diameter 0)
 		(color 0 0 0 0)
@@
 	)
 	(junction
-		(at 50.8 25.4)
-		(diameter 0)
-		(color 0 0 0 0)
-	)
-	(junction
-		(at 36.83 25.4)
-		(diameter 0)
-		(color 0 0 0 0)
-	)
-	(junction
 		(at 54.61 97.79)
 		(diameter 0)
@@
 	(wire
 		(pts
-			(xy 50.8 111.125) (xy 50.8 113.03)
+			(xy 50.8 111.76) (xy 50.8 113.03)
 		)
 		(stroke
@@
 	(wire
 		(pts
-			(xy 52.07 95.25) (xy 52.07 99.695)
+			(xy 52.07 95.25) (xy 52.07 100.33)
 		)
 		(stroke
@@
 	(wire
 		(pts
-			(xy 46.99 90.17) (xy 46.99 99.695)
+			(xy 46.99 90.17) (xy 46.99 100.33)
 		)
 		(stroke
@@
 	(bus
 		(pts
-			(xy 97.79 48.26) (xy 109.855 48.26)
+			(xy 97.79 48.26) (xy 99.06 48.26)
 		)
 		(stroke
@@
 	(wire
 		(pts
+			(xy 31.75 86.36) (xy 31.75 87.63)
+		)
+		(stroke
+			(width 0)
+			(type default)
+		)
+	)
+	(wire
+		(pts
 			(xy 31.75 102.87) (xy 31.75 100.33)
 		)
@@
 	(wire
 		(pts
+			(xy 33.02 86.36) (xy 31.75 86.36)
+		)
+		(stroke
+			(width 0)
+			(type default)
+		)
+	)
+	(wire
+		(pts
 			(xy 50.8 50.8) (xy 50.8 53.34)
 		)
@@
 	(wire
 		(pts
-			(xy 54.61 97.79) (xy 54.61 99.695)
+			(xy 54.61 97.79) (xy 54.61 100.33)
 		)
 		(stroke
@@
 	(wire
 		(pts
-			(xy 49.53 92.71) (xy 49.53 99.695)
+			(xy 49.53 92.71) (xy 49.53 100.33)
 		)
 		(stroke
@@
 		)
 	)
-	(label "ENC{A B}"
-		(at 107.95 48.26 180)
-		(effects
-			(font
-				(size 1.27 1.27)
-			)
-			(justify right bottom)
-		)
-	)
 	(label "ENC.A"
 		(at 93.98 43.18 180)
@@
 		)
 	)
-	(label "3.3V_DEBUG"
-		(at 31.75 87.63 0)
-		(effects
-			(font
-				(size 1.27 1.27)
-			)
-			(justify left bottom)
-		)
-	)
 	(label "PROGSPI.MOSI"
 		(at 53.34 41.91 180)
@@
 		)
 	)
-	(hierarchical_label "ENC"
+	(hierarchical_label "ENC{A B}"
 		(shape output)
-		(at 109.855 48.26 0)
+		(at 99.06 48.26 0)
+		(effects
+			(font
+				(size 1.27 1.27)
+			)
+			(justify left)
+		)
+	)
+	(hierarchical_label "3.3V DEBUG"
+		(shape output)
+		(at 33.02 86.36 0)
 		(effects
 			(font
@@
 	(symbol
 		(lib_id "RJ-Diodes:PUSB3FR4")
-		(at 50.8 103.505 0)
+		(at 50.8 104.14 0)
 		(unit 1)
 		(body_style 1)
@@
 		(fields_autoplaced yes)
 		(property "Reference" "D14"
-			(at 56.515 103.5049 0)
+			(at 56.515 104.1399 0)
 			(show_name no)
 			(do_not_autoplace no)
@@
 		)
 		(property "Value" "PUSB3FR4Z"
-			(at 56.515 106.0449 0)
+			(at 56.515 106.6799 0)
 			(show_name no)
 			(do_not_autoplace no)
@@
 		)
 		(property "Footprint" "Package_DFN_QFN:Diodes_UDFN-10_1x2.5mm_P0.5mm"
-			(at 50.8 75.565 0)
+			(at 50.8 76.2 0)
 			(hide yes)
 			(show_name no)
@@
 		)
 		(property "Datasheet" "https://assets.nexperia.com/documents/data-sheet/PUSB3FR4.pdf"
-			(at 51.435 73.025 0)
+			(at 51.435 73.66 0)
 			(hide yes)
 			(show_name no)
@@
 		)
 		(property "Description" "3V (Typ) Clamp 5A (8/20µs) Ipp Tvs Diode Surface Mount DFN2510A-10"
-			(at 50.8 78.105 0)
+			(at 50.8 78.74 0)
 			(hide yes)
 			(show_name no)
@@
 		)
 		(property "Manufacturer P/N" "PUSB3FR4Z"
-			(at 50.8 83.185 0)
+			(at 50.8 83.82 0)
 			(hide yes)
 			(show_name no)
@@
 		)
 		(property "Vendor" "DigiKey"
-			(at 50.8 85.725 0)
+			(at 50.8 86.36 0)
 			(hide yes)
 			(show_name no)
@@
 		)
 		(property "Vendor P/N" "1727-2026-1-ND"
-			(at 50.8 80.645 0)
-			(hide yes)
-			(show_name no)
+			(at 50.8 81.28 0)
+			(hide yes)
+			(show_name no)

Commit message: WIP placement & routing
Other:
- note added: "TODO: Unused SPI requires a certain resistor configuration"
- moved on the sheet: D14, J4

Commit message: Layout & Routing done
Parts:
- added R51, R52, R53: 4.7k, Resistor_SMD:R_0402_1005Metric, symbol Device:R
Connections:
- net 3.3V DEBUG: now also R51.1
- net GND: now also R52.2, R53.2
- net PROGSPI.CLK: now also R53.1
- net PROGSPI.CSN: now also R51.2
- net PROGSPI.MOSI: now also R52.1
