File: boards/develop-2027/dribbler-motorboard/dribbler-board-v0.1/current_sense.kicad_sch (KiCad schematic)
At the start: 8 parts

Commit message: Add motor temp sensor sheet and retune analogs
Introduces a new `motor_temp_sense.kicad_sch` sub-sheet with thermistor connector/divider circuitry and wires it into the integration schematic as `TEMP_SENSE`. The update also retunes current-sense and overcurrent component values for the new 16CL41-12-P2-7300 motor, removes unused magnetic encoder and motor mounting-hole schematic content, and refreshes project/sheet metadata and labeling.
Parts:
- R1: value 8.25k ±0.1% -> 120k ±0.1%
- R3, R7: value 1.13k ±0.1% -> 30k ±0.1%
- R5, R9: value 16.5k ±0.1% -> 240k ±0.1%
Changed lines of the file:
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@@
 	(title_block
 		(title "Current Sense Op-Amp")
-		(date "2026-09-02")
+		(date "2026-09-07")
 		(rev "v1.0")
 		(company "Robojackets - RoboCup")
-		(comment 1 "Aiden Lee [piman PCB]")
+		(comment 1 "Niko Cornell & Miles Schuler")
 	)
 	(rectangle
@@
 		)
 	)
-	(text_box "Differental amplifier with low pass filtered output. Design derived from EVLSPIN32G0A2 Evaluation Board.\nIntended for Field-Oriented Control of the Nanotec DF45 65W (10 A peak) or DF45 50W (7 A peak).\nAll Resistors except for R_{LP}: ±0.1% 25ppm/°C or better.\n\nIdeal Characteristics:\nVoltage Gain (G_{V/V}): 7.301 V/V\nCurrent Gain (G_{V/A}): 109.5 mV/A (15 mΩ shunt)\nCurrent Sense Range (I_{RANGE}): ±15.07 A\nOutput Offset (I_{SHUNT} = 0 A): 1.65 V\nLow Pass Filter Cutoff (-3 dB gain): 4.82 kHz\n\nSee ST Manual on EVLSPIN32G0A2, Section 4.4 for derivation"
+	(text_box "Differental amplifier with low pass filtered output. Design derived from EVLSPIN32G0A2 Evaluation Board.\nIntended for Field-Oriented Control of the 16CL41-12-P2-7300 (11 A peak).\nAll Resistors except for R_{LP}: ±0.1% 25ppm/°C or better.\n\nIdeal Characteristics:\nVoltage Gain (G_{V/V}): 4.0 V/V\nCurrent Gain (G_{V/A}): 60 mV/A (15 mΩ shunt)\nCurrent Sense Range (I_{RANGE}): ±27.5 A\nOutput Offset (I_{SHUNT} = 0 A): 1.65 V\nLow Pass Filter Cutoff (-3 dB gain): 4.82 kHz\n\nSee ST Manual on EVLSPIN32G0A2, Section 4.4 for derivation"
 		(exclude_from_sim no)
 		(at 53.34 105.41 0)
@@
 			)
 		)
-		(property "Value" "16.5k ±0.1%"
+		(property "Value" "240k ±0.1%"
 			(at 87.63 72.3899 0)
 			(show_name no)
@@
 			)
 		)
-		(property "Value" "1.13k ±0.1%"
+		(property "Value" "30k ±0.1%"
 			(at 104.14 60.96 90)
 			(show_name no)
@@
 			)
 		)
-		(property "Value" "1.13k ±0.1%"
+		(property "Value" "30k ±0.1%"
 			(at 66.04 73.66 90)
 			(show_name no)
@@
 			)
 		)
-		(property "Value" "8.25k ±0.1%"
+		(property "Value" "120k ±0.1%"
 			(at 129.54 48.26 90)
 			(show_name no)
@@
 			)
 		)
-		(property "Value" "16.5k ±0.1%"
+		(property "Value" "240k ±0.1%"
 			(at 87.63 85.0899 0)
 			(show_name no)

Commit message: Updated for BOM consolidation
Updated component references and part numbers for BOM consolidation
Parts:
- removed C2: 100n, Capacitor_SMD:C_0402_1005Metric, symbol Device:C
- added C18: 100n 25V, Capacitor_SMD:C_0402_1005Metric, symbol Device:C
- renumbered R1 to R27, R3 to R28, R5 to R29, R6 to R30, R7 to R31, R9 to R32, TP1 to TP24
Connections:
- net GND: now also C18.2
- net I_{SENSE}: now also C18.1
