File: boards/develop-2027/dribbler-motorboard/dribbler-board-v0.1/temp_sens.kicad_sch (KiCad schematic)
At the start: 7 parts, among them U5 LM75ADP

Commit message: Updated for BOM consolidation
Updated component references and part numbers for BOM consolidation
Parts:
- renumbered D12 to D11, R42 to R21, R43 to R22, R44 to R23, TP31 to TP22, TP32 to TP23, U5 to U3
Changed lines of the file:
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@@
 		(dnp no)
 		(fields_autoplaced yes)
-		(property "Reference" "TP31"
+		(property "Reference" "TP22"
 			(at 195.58 74.9299 90)
 			(show_name no)
@@
 			(project "integration-test"
 				(path "/2f9570f4-e846-4a86-b134-ae7438cb1d91/d4780e5d-8897-4fbd-a4f0-0cae90768857"
-					(reference "TP31")
+					(reference "TP22")
 					(unit 1)
 				)
@@
 		(dnp no)
 		(fields_autoplaced yes)
-		(property "Reference" "TP32"
+		(property "Reference" "TP23"
 			(at 195.58 81.2799 90)
 			(show_name no)
@@
 			(project "integration-test"
 				(path "/2f9570f4-e846-4a86-b134-ae7438cb1d91/d4780e5d-8897-4fbd-a4f0-0cae90768857"
-					(reference "TP32")
+					(reference "TP23")
 					(unit 1)
 				)
@@
 		(dnp no)
 		(fields_autoplaced yes)
-		(property "Reference" "R44"
+		(property "Reference" "R23"
 			(at 170.18 91.4399 0)
 			(show_name no)
@@
 			(project "integration-test"
 				(path "/2f9570f4-e846-4a86-b134-ae7438cb1d91/d4780e5d-8897-4fbd-a4f0-0cae90768857"
-					(reference "R44")
+					(reference "R23")
 					(unit 1)
 				)
@@
 		(dnp no)
 		(fields_autoplaced yes)
-		(property "Reference" "R42"
+		(property "Reference" "R21"
 			(at 144.78 85.0899 0)
 			(show_name no)
@@
 			(project "integration-test"
 				(path "/2f9570f4-e846-4a86-b134-ae7438cb1d91/d4780e5d-8897-4fbd-a4f0-0cae90768857"
-					(reference "R42")
+					(reference "R21")
 					(unit 1)
 				)
@@
 		(dnp no)
 		(fields_autoplaced yes)
-		(property "Reference" "D12"
+		(property "Reference" "D11"
 			(at 146.05 95.5674 90)
 			(show_name no)
@@
 			(project "integration-test"
 				(path "/2f9570f4-e846-4a86-b134-ae7438cb1d91/d4780e5d-8897-4fbd-a4f0-0cae90768857"
-					(reference "D12")
+					(reference "D11")
 					(unit 1)
 				)
@@
 		(dnp no)
 		(fields_autoplaced yes)
-		(property "Reference" "#PWR054"
+		(property "Reference" "#PWR049"
 			(at 142.24 83.82 0)
 			(hide yes)
@@
 			(project "integration-test"
 				(path "/2f9570f4-e846-4a86-b134-ae7438cb1d91/d4780e5d-8897-4fbd-a4f0-0cae90768857"
-					(reference "#PWR054")
+					(reference "#PWR049")
 					(unit 1)
 				)
@@
 		(dnp no)
 		(fields_autoplaced yes)
-		(property "Reference" "#PWR056"
+		(property "Reference" "#PWR051"
 			(at 167.64 88.9 0)
 			(hide yes)
@@
 			(project "integration-test"
 				(path "/2f9570f4-e846-4a86-b134-ae7438cb1d91/d4780e5d-8897-4fbd-a4f0-0cae90768857"
-					(reference "#PWR056")
+					(reference "#PWR051")
 					(unit 1)
 				)
@@
 		(in_pos_files yes)
 		(dnp no)
-		(property "Reference" "R43"
+		(property "Reference" "R22"
 			(at 158.75 91.4399 0)
 			(show_name no)
@@
 			(project "integration-test"
 				(path "/2f9570f4-e846-4a86-b134-ae7438cb1d91/d4780e5d-8897-4fbd-a4f0-0cae90768857"
-					(reference "R43")
+					(reference "R22")
 					(unit 1)
 				)
@@
 		(dnp no)
 		(fields_autoplaced yes)
-		(property "Reference" "#PWR055"
+		(property "Reference" "#PWR050"
 			(at 161.29 88.9 0)
 			(hide yes)
@@
 			(project "integration-test"
 				(path "/2f9570f4-e846-4a86-b134-ae7438cb1d91/d4780e5d-8897-4fbd-a4f0-0cae90768857"
-					(reference "#PWR055")
+					(reference "#PWR050")
 					(unit 1)
 				)
@@
 		(dnp no)
 		(fields_autoplaced yes)
-		(property "Reference" "U5"
+		(property "Reference" "U3"
 			(at 129.54 91.44 0)
 			(show_name no)
@@
 			(project "integration-test"
 				(path "/2f9570f4-e846-4a86-b134-ae7438cb1d91/d4780e5d-8897-4fbd-a4f0-0cae90768857"
-					(reference "U5")
+					(reference "U3")
 					(unit 1)
 				)
@@
 		(dnp no)
 		(fields_autoplaced yes)
-		(property "Reference" "#PWR058"
+		(property "Reference" "#PWR053"
 			(at 116.84 121.92 0)
 			(hide yes)
@@
 			(project "integration-test"
 				(path "/2f9570f4-e846-4a86-b134-ae7438cb1d91/d4780e5d-8897-4fbd-a4f0-0cae90768857"
-					(reference "#PWR058")
+					(reference "#PWR053")
 					(unit 1)
 				)
@@
 		(dnp no)
 		(fields_autoplaced yes)
-		(property "Reference" "#PWR057"
+		(property "Reference" "#PWR052"
 			(at 116.84 99.06 0)
 			(hide yes)
@@
 			(project "integration-test"
 				(path "/2f9570f4-e846-4a86-b134-ae7438cb1d91/d4780e5d-8897-4fbd-a4f0-0cae90768857"
-					(reference "#PWR057")
+					(reference "#PWR052")
 					(unit 1)
 				)
