File: boards/develop-2027/power-board/power_management.kicad_sch (KiCad schematic)
At the start: 43 parts, among them U3 LMR51430XDDCR, U4 LMR51430XDDCR, U5 SIC437AED-T1-GE3, U6 ${SIM.PARAMS}

Commit message: 12v rail buck external circuitry done
Connections:
- net VBAT_FUSED: no longer U5.19 (EN)
- new net RAIL_EN_12V: U5.19 (EN)
- no-connect marks 0 -> 1
Other:
- note added: "not connected in datasheet"
Changed lines of the file:
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@@
+		)
+	)
+	(text "not connected\nin datasheet"
+		(exclude_from_sim no)
+		(at 129.032 165.1 0)
+		(effects
+			(font
+				(size 0.8 0.8)
+			)
+			(justify left)
 		)
 	)
@@
 	)
 	(junction
-		(at 115.57 144.78)
-		(diameter 0)
-		(color 0 0 0 0)
-	)
-	(junction
 		(at 309.88 49.53)
 		(diameter 0)
@@
 		(color 0 0 0 0)
 	)
+	(no_connect
+		(at 128.27 165.1)
+	)
 	(wire
 		(pts
@@
 	(wire
 		(pts
-			(xy 102.87 152.4) (xy 102.87 144.78)
-		)
-		(stroke
-			(width 0)
-			(type default)
-		)
-	)
-	(wire
-		(pts
 			(xy 307.34 44.45) (xy 309.88 44.45)
 		)
@@
 	(wire
 		(pts
-			(xy 102.87 144.78) (xy 115.57 144.78)
+			(xy 80.01 152.4) (xy 102.87 152.4)
 		)
 		(stroke
@@
 		)
 	)
+	(hierarchical_label "RAIL_EN_12V"
+		(shape input)
+		(at 80.01 152.4 180)
+		(effects
+			(font
+				(size 1.27 1.27)
+			)
+			(justify right)
+		)
+	)

Commit message: some changes
Connections:
- net +12V_SOURCE: no longer R15.1, U5.17 (FB)
- net -BATT: no longer R16.2
- new net: R15.1, R16.2, U5.17 (FB)
Other:
- note added: "<--- use electrolytic instead of ceramic cuz better price for the ratings you get (for the 44µF)"
- note added: "five 22µF parts at 12V bias give roughly 55µF effective"
- note added: "put close to Vin"
- note removed: "add up to 100µF plus margin (so 110µF)"
- moved on the sheet: R16
Changed lines of the file:
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@@
 		)
 	)
+	(text "put close to Vin"
+		(exclude_from_sim no)
+		(at 50.8 141.224 0)
+		(effects
+			(font
+				(size 1.27 1.27)
+			)
+			(justify left)
+		)
+	)
 	(text "TODO: replace with fuse mount if this isn't the mount"
 		(exclude_from_sim no)
@@
 	(text "From datasheet:\nR_{_FB_H} = (R_{_FB_L}(V_{OUT} - V_{FB})) / V_{FB}\n\"Where V_{FB} is 0.6 V for the SiC43X.\"\n\n= 10000*(12-0.6)/0.6 = 190kΩ"
 		(exclude_from_sim no)
-		(at 149.098 183.642 0)
+		(at 155.702 164.084 0)
 		(effects
 			(font
@@
 		)
 	)
-	(text "add up to 100µF plus margin (so 110µF)"
+	(text "five 22µF parts at 12V bias give roughly 55µF effective"
 		(exclude_from_sim no)
-		(at 167.64 135.636 0)
+		(at 162.56 135.89 0)
 		(effects
 			(font
@@
 		)
 	)
+	(text "<--- use electrolytic instead of ceramic\ncuz better price for the ratings you\nget (for the 44µF)"
+		(exclude_from_sim no)
+		(at 124.968 63.246 0)
+		(effects
+			(font
+				(size 1.27 1.27)
+			)
+			(justify left)
+		)
+	)
 	(junction
 		(at 168.91 147.32)
@@
 	(wire
 		(pts
-			(xy 147.32 177.8) (xy 147.32 190.5)
-		)
-		(stroke
-			(width 0)
-			(type default)
-		)
-	)
-	(wire
-		(pts
 			(xy 307.34 44.45) (xy 309.88 44.45)
 		)
@@
 	(wire
 		(pts
-			(xy 191.77 137.16) (xy 191.77 139.7)
+			(xy 191.77 134.62) (xy 191.77 139.7)
 		)
 		(stroke
@@
 	(wire
 		(pts
-			(xy 147.32 170.18) (xy 147.32 172.72)
-		)
-		(stroke
-			(width 0)
-			(type default)
-		)
-	)
-	(wire
-		(pts
 			(xy 87.63 58.42) (xy 90.17 58.42)
 		)
@@
 	(wire
 		(pts
+			(xy 147.32 166.37) (xy 147.32 170.18)
+		)
+		(stroke
+			(width 0)
+			(type default)
+		)
+	)
+	(wire
+		(pts
 			(xy 33.02 127) (xy 43.18 127)
 		)
@@
 	(wire
 		(pts
-			(xy 147.32 160.02) (xy 147.32 170.18)
+			(xy 147.32 160.02) (xy 147.32 161.29)
 		)
 		(stroke
@@
 	)
 	(label "+12V_SOURCE"
-		(at 191.77 137.16 0)
+		(at 191.77 134.62 0)
 		(effects
 			(font
@@
 	(symbol
 		(lib_id "Device:R_Small")
-		(at 147.32 175.26 0)
+		(at 147.32 163.83 0)
 		(unit 1)
 		(body_style 1)
@@
 		(dnp no)
 		(property "Reference" "R16"
-			(at 148.082 174.2439 0)
+			(at 148.082 162.8139 0)
 			(show_name no)
 			(do_not_autoplace no)
@@
 		)
 		(property "Value" "190kΩ"
-			(at 148.082 175.768 0)
+			(at 148.082 164.338 0)
 			(show_name no)
 			(do_not_autoplace no)
@@
 		)
 		(property "Footprint" ""
-			(at 147.32 175.26 0)
+			(at 147.32 163.83 0)
 			(hide yes)
 			(show_name no)
@@
 		)
 		(property "Datasheet" ""
-			(at 147.32 175.26 0)
+			(at 147.32 163.83 0)
 			(hide yes)
 			(show_name no)
@@
 		)
 		(property "Description" "Resistor, small symbol"
-			(at 147.32 175.26 0)
+			(at 147.32 163.83 0)
 			(hide yes)
 			(show_name no)
@@
 		)
 		(property "Datasheet Label" "R_{_FB_H}"
-			(at 151.13 177.546 0)
+			(at 151.13 166.116 0)
 			(show_name no)
 			(do_not_autoplace no)
@@
 		(dnp no)
 		(property "Reference" "R15"
-			(at 152.4 166.878 90)
+			(at 152.4 171.958 90)
 			(show_name no)
 			(do_not_autoplace no)
@@
 		)
 		(property "Value" "10kΩ"
-			(at 152.4 168.402 90)
+			(at 152.4 173.482 90)
 			(show_name no)
 			(do_not_autoplace no)
@@
 					(unit 1)
 				)
-			)
-		)
-	)
-	(symbol
-		(lib_id "power:GND")
-		(at 147.32 190.5 0)
-		(unit 1)
-		(body_style 1)
-		(exclude_from_sim no)
-		(in_bom yes)
-		(on_board yes)
-		(in_pos_files yes)
-		(dnp no)
-		(fields_autoplaced yes)
-		(property "Reference" "#PWR016"
-			(at 147.32 196.85 0)
-			(hide yes)
-			(show_name no)
-			(do_not_autoplace no)
-			(effects
-				(font
-					(size 1.27 1.27)
-				)
-			)
-		)
-		(property "Value" "GND"
-			(at 147.32 195.58 0)
-			(show_name no)
-			(do_not_autoplace no)
-			(effects
-				(font
-					(size 1.27 1.27)
-				)
-			)
-		)
-		(property "Footprint" ""
-			(at 147.32 190.5 0)
-			(hide yes)
-			(show_name no)
-			(do_not_autoplace no)
-			(effects
-				(font
-					(size 1.27 1.27)
-				)
-			)
-		)
-		(property "Datasheet" ""
-			(at 147.32 190.5 0)
-			(hide yes)
-			(show_name no)
-			(do_not_autoplace no)
-			(effects
-				(font
-					(size 1.27 1.27)
-				)
-			)
-		)
-		(property "Description" "Power symbol creates a global label with name \"GND\" , ground"
-			(at 147.32 190.5 0)
-			(hide yes)
-			(show_name no)
-			(do_not_autoplace no)
-			(effects
-				(font
-					(size 1.27 1.27)
-				)
-			)
-		)
-		(pin "1"
-		)
-		(instances
-			(project "power-board"
-				(path "/cb63459b-b5eb-4b1b-8316-cdcb6a76275f/78bc56ac-35bc-4a48-b190-7d489bf5b351"
-					(reference "#PWR016")
-					(unit 1)
-				)

Commit message: add current sense circuit; add connector sheet, wip; add some hierarchical labels; organization; etc
Parts:
- removed R17, R18: R, symbol Device:R
- removed R19, R_Shunt?: R_Small, symbol Device:R_Small
- removed U6: ${SIM.PARAMS}, Package_SO:SOIC-8_3.9x4.9mm_P1.27mm, symbol Simulation_SPICE:OPAMP
- added R_Shunt1, R_Shunt2: 10mΩ, symbol Device:R_Small
- added R_Shunt3: 2.5mΩ, symbol Device:R_Small
- added U7: INA4180A3IPWR, symbol Amplifier_Current:INA4180A3IPWR
Connections:
- net +12V: now also R_Shunt3.2, U7.9 (IN-3)
- net +12V_SOURCE: now also R_Shunt3.1, U7.10 (IN+3)
- net +3V3: now also R_Shunt1.2, U7.2 (IN-1)
- net +3V3_SOURCE: now also R_Shunt1.1, U7.3 (IN+1)
- net +5V: now also R_Shunt2.2, U7.6 (IN-2)
- net +5V_SOURCE: now also R_Shunt2.1, U7.5 (IN+2)
- net -BATT: now also U7.11 (GND), U7.12 (IN+4), U7.13 (IN-4)
- net I_SENSE_3V3: now also U7.1 (OUT1)
- new net I_SENSE_12V: U7.8 (OUT3)
- new net I_SENSE_5V: U7.7 (OUT2)
- no-connect marks 1 -> 2
Other:
- note added: "f_{SW} = 500kHz for 3V3 and 5V rail bucks"
- note added: "f_{SW}=500kHz"
- note added: "requirements: (shunt voltage drop) * (gain) = 3V (under max ADC in of 3.3V); gain of the quad amp is 100; 3V / 100 = 0.03 V max shunt drop. 3V3 and 5V rails are 3A: 0.03 V / 3A = 0.01Ω = 10mΩ; 12V rail is 12A: 0.03V / 12A = 0.0025 = 2.5mΩ. shunt rating requirement: 3V3 and 5V rails: 0.03V * 3A = 0.09W; 12V rail: 0.03V * 12A = 0.36W. (plus margin for safety)"
- note removed: "TODO finish this, determine the values needed for shunt resistor, and the op amp resistors accordingly. and make sure i sense output is such that it is max 3.3v (cuz adc input max). then duplicate for other rails"

Commit message: power dist: 12v rail external circuitry attached footprints and digikey parts; and other changes
Parts:
- removed C15, C28: 100nF, RF_Module:CMWX1ZZABZ, symbol Device:C_Small
- removed C16, C26, C27: 10µF, RF_Module:CMWX1ZZABZ, symbol Device:C_Small
- removed C17: 0.1µF, symbol Device:C_Small
- removed C20, C21, C22, C23, C24: 22µF, RF_Module:CMWX1ZZABZ, symbol Device:C_Small
- removed C29: 100µF, RF_Module:CMWX1ZZABZ, symbol Device:C_Small
- added C30: 10u, symbol Device:C
- added C31, C59, C65: 0.1µF, Capacitor_SMD:C_0402_1005Metric_Pad0.74x0.62mm_HandSolder, symbol Device:C_Small
- added C32, C33, C34, C35, C57, C58: 10µF, Capacitor_SMD:C_1210_3225Metric_Pad1.33x2.70mm_HandSolder, symbol Device:C_Small
- added C36, C37, C38, C55, C56, C60, C61, C62, C63, C64: 22µF, Capacitor_SMD:CAPAE660X600N - A768EB226M1HLAE048, symbol Device:C_Polarized_Small_US
- added Q1: PMOS, symbol Simulation_SPICE:PMOS
- added R17: 1k, symbol Device:R
- added TP21: 3.3V DEBUG, TestPoint:TestPoint_Pad_D1.0mm, symbol Connector:TestPoint
- added TP22: 3.3V_REG, TestPoint:TestPoint_Pad_D1.0mm, symbol Connector:TestPoint
- added TP23: 3.3V, TestPoint:TestPoint_Pad_D1.0mm, symbol Connector:TestPoint
- added U6, U8: LM66100DCK, Package_TO_SOT_SMD:SOT-363_SC-70-6, symbol Power_Management:LM66100DCK
- C18: footprint (none) -> Capacitor_SMD:C_1210_3225Metric_Pad1.33x2.70mm_HandSolder; DigiKey Part # (none) -> 490-1864-1-ND; Part # (none) -> GRM32ER71H475KA88L
- C19: footprint RF_Module:CMWX1ZZABZ -> Capacitor_SMD:C_0402_1005Metric_Pad0.74x0.62mm_HandSolder; DigiKey Part # (none) -> 490-10017-1-ND; Part # (none) -> GRM155R61E105KA12D
- C25: value 10µF -> 4.7µF; footprint RF_Module:CMWX1ZZABZ -> Capacitor_SMD:C_1210_3225Metric_Pad1.33x2.70mm_HandSolder; Datasheet Label C_{IN} -> (none); DigiKey Part # (none) -> 490-1864-1-ND; Part # (none) -> GRM32ER71H475KA88L
- L4: footprint Package_DFN_QFN:Vishay_PowerPAK_MLP44-24L_ThermalVias -> (none)
- R15, R23: footprint (none) -> Resistor_SMD:R_0402_1005Metric_Pad0.72x0.64mm_HandSolder; DigiKey Part # (none) -> RMCF0402FT10K0CT-ND; Part # (none) -> RMCF0402FT10K0
- R16: value 190kΩ -> 191kΩ; footprint (none) -> Resistor_SMD:R_0201_0603Metric_Pad0.64x0.40mm_HandSolder; DigiKey Part # (none) -> YAG2460CT-ND; Part # (none) -> RC0201FR-07191KL
- R20: footprint (none) -> Resistor_SMD:R_0402_1005Metric_Pad0.72x0.64mm_HandSolder; DigiKey Part # (none) -> 311-100KLRCT-ND; Part # (none) -> RC0402FR-07100KL
- R21: footprint (none) -> Resistor_SMD:R_0805_2012Metric_Pad1.20x1.40mm_HandSolder; DigiKey Part # (none) -> RG20P499KBCT-ND; Part # (none) -> RG2012P-4993-B-T5
- R22: footprint (none) -> Resistor_SMD:R_0402_1005Metric_Pad0.72x0.64mm_HandSolder; DigiKey Part # (none) -> 541-2.20LLCT-ND; Part # (none) -> CRCW04022R20FKED
Connections:
- net +12V_SOURCE: now also C60.1, C61.1, C62.1, C63.1, C64.1
- net +3V3_SOURCE: now also C30.1, TP23.1, U6.6 (VOUT), U8.6 (VOUT); no longer C11.1, L2.2, R11.1
- net +5V_SOURCE: now also U7.4 (VS)
- net -BATT: now also C25.1, C30.2, C31.2, C32.2, C33.2, C34.2, C35.2, C36.2, C37.2, C38.2, C55.2, C56.2, C57.2, C58.2, C59.2, C60.2, C61.2, C62.2, C63.2, C64.2, U6.2 (GND), U8.2 (GND), U8.5 (ST); no longer C18.1, C25.2
- net at U5.23 (BOOT): now also C65.1
- net at L4.1, U5.5 (SW), U5.6 (SW)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: now also C59.1
- net at R22.1: now also C65.2
- net VBAT_FUSED renamed BAT_FUSED
- net BAT_FUSED: now also C31.1, C32.1, C33.1, C34.1, C35.1, C36.1, C37.1, C38.1, C55.1, C56.1, C57.1, C58.1, Q1.3 (S); no longer C25.1
- new net: C18.1, C25.2
- new net: R17.2, U6.5 (ST), U8.3 (~{CE})
- new net 3.3V_DEBUG: R17.1, TP21.1, U6.1 (VIN)
- new net 3.3V_REG: C11.1, L2.2, R11.1, TP22.1, U6.3 (~{CE}), U8.1 (VIN)
- new net RAIL_BAT: Q1.1 (D)
Other:
- note added: "(copied from rev-2026/kicker-v3.4)"
- note added: "3.3V Dual-Supply ORing Power Mux"
- note added: "BULK CAPACITORS (Electrolytic, lower res freq): 5*22 = 110µF"
- note added: "Calculations for SIC437 external circuitry: https://www.desmos.com/calculator/lv8rmnqqm9 (NOTE: this was used initially, not all of the calculations here are still relevant)"
- note added: "DECOUPLING CAPACITORS (ceramic, higher res freq):"
- note added: "TODO: decide if using this is fine for the VS (power supply)"
- note added: "This isn't strictly nessesary, but it's additional protection for USB/SWD"
- note added: "as of making this schematic, 190kΩ not in stock. so using 191kΩ"
- note added: "https://www.vishay.com/docs/76801/sic43x_usermanual.pdf for SiC437 external circuitry and layout reference"
- note added: "link to frequency characteristics for 10µF caps, CL32B106KMVNNWE (CLICK ME)"
- note removed: "Calculations for SIC437 external circuitry: https://www.desmos.com/calculator/lv8rmnqqm9"
- note removed: "put close to Vin"
- moved on the sheet: C11, C12, C13, C14, C18, C19, C8, C9, F1, L2, L3, L4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

Commit message: put in parts for shunt resistors (TODO: put in footprints)
Parts:
- R_Shunt1, R_Shunt2: DigikeyPart# (none) -> P17098CT-ND; Part# (none) -> ERJ-MS4HF10MU
- R_Shunt3: DigikeyPart# (none) -> 541-10116-1-ND; Part# (none) -> WSL25122L500FEA
Other:
- note added: "TODO: Find footprints for parts"
Changed lines of the file:
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@@
 		)
 	)
+	(text "TODO: Find footprints for parts"
+		(exclude_from_sim no)
+		(at 256.286 88.138 0)
+		(effects
+			(font
+				(size 1.27 1.27)
+			)
+		)
+	)
 	(junction
 		(at 31.75 35.56)
@@
 			)
 		)
-		(property "Datasheet" ""
+		(property "Datasheet" "https://www.vishay.com/docs/30100/wsl.pdf"
 			(at 306.07 76.2 0)
 			(hide yes)
@@
 			)
 		)
+		(property "Part#" "WSL25122L500FEA"
+			(at 306.07 76.2 90)
+			(hide yes)
+			(show_name no)
+			(do_not_autoplace no)
+			(effects
+				(font
+					(size 1.27 1.27)
+				)
+			)
+		)
+		(property "DigikeyPart#" "541-10116-1-ND"
+			(at 306.07 76.2 90)
+			(hide yes)
+			(show_name no)
+			(do_not_autoplace no)
+			(effects
+				(font
+					(size 1.27 1.27)
+				)
+			)
+		)
 		(pin "1"
 		)
@@
 			)
 		)
-		(property "Datasheet" ""
+		(property "Datasheet" "https://industrial.panasonic.com/cdbs/www-data/pdf/RDN0000/AOA0000C319.pdf"
 			(at 257.81 76.2 0)
 			(hide yes)
@@
 			)
 		)
+		(property "Part#" "ERJ-MS4HF10MU"
+			(at 257.81 76.2 90)
+			(hide yes)
+			(show_name no)
+			(do_not_autoplace no)
+			(effects
+				(font
+					(size 1.27 1.27)
+				)
+			)
+		)
+		(property "DigikeyPart#" "P17098CT-ND"
+			(at 257.81 76.2 90)
+			(hide yes)
+			(show_name no)
+			(do_not_autoplace no)
+			(effects
+				(font
+					(size 1.27 1.27)
+				)
+			)
+		)
 		(pin "1"
 		)
@@
 			)
 		)
-		(property "Datasheet" ""
+		(property "Datasheet" "https://industrial.panasonic.com/cdbs/www-data/pdf/RDN0000/AOA0000C319.pdf"
 			(at 257.81 63.5 0)
 			(hide yes)
@@
 			(hide yes)
 			(show_name no)
+			(do_not_autoplace no)
+			(effects
+				(font
+					(size 1.27 1.27)
+				)
+			)
+		)
+		(property "Part#" "ERJ-MS4HF10MU"
+			(at 257.81 63.5 90)
+			(hide yes)
+			(show_name no)
+			(do_not_autoplace no)
+			(effects
+				(font
+					(size 1.27 1.27)
+				)
+			)
+		)
+		(property "DigikeyPart#" "P17098CT-ND"
+			(at 257.81 63.5 90)
+			(hide yes)
+			(show_name no)

Commit message: finished power dist. board (TODO: add footprints to everything)
Parts:
- C11, C14: DigikeyPart# (none) -> 399-A768EB476M1VLAE042CT-ND; Part# (none) -> A768EB476M1VLAE042
- C12, C8: DigikeyPart# (none) -> 490-12332-1-ND; Part# (none) -> GRT188R61H225KE13D
- C13, C9: DigikeyPart# (none) -> 490-10700-1-ND; Part# (none) -> GRM155R71H104KE14D
- L2: DigikeyPart# (none) -> 4044-CSHB0540R-5R6MCT-ND; Part# (none) -> CSHB0540R-5R6M
- L3: DigikeyPart# (none) -> 4044-CSBA1060-6R8MCT-ND; Part# (none) -> CSBA1060-6R8M
- L4: DigikeyPart# (none) -> 4044-CSHB0540R-3R3MCT-ND; Part# (none) -> CSHB0540R-3R3M
- R11, R13: DigikeyPart# (none) -> 311-100KLRCT-ND; Part# (none) -> RC0402FR-07100KL
- R12: DigikeyPart# (none) -> 311-22.1KHRCT-ND; Part# (none) -> RC0603FR-0722K1L
- R14: DigikeyPart# (none) -> 311-13.7KHRCT-ND; Part# (none) -> RC0603FR-0713K7L
- U7: DigikeyPart# (none) -> 296-49096-1-ND; Part# (none) -> INA4180A3IPWR
