File: boards/develop-2027/controlboard/ControlBoard2027/03_USB_Debug.kicad_sch (KiCad schematic)
At the start: 12 parts, among them J2 USB-C_DFU, J3 SWD_5pin, SW1 RESET, SW2 BOOT0_DFU, U5 USBLC6-2SC6

Commit message: post design review changes
post design review changes
Connections:
- net GND: now also J3.4 (Pin_4); no longer J3.5 (Pin_5)
- net NRST: now also J3.5 (Pin_5); no longer J3.4 (Pin_4)
- net SWCLK: now also R39.1; no longer R40.1
- net SWDIO: now also R40.1; no longer R39.1
Other:
- note added: "R39/R40 22R: series resistors on SWCLK/SWDIO. Damp ringing on the probe cable and limit current into PA13/PA14 from ESD or a bad probe. Not critical (0R works)."
- note added: "ROUTING - USB FS USB_DP/USB_DM: 90R differential pair, length-matched within 1mm, over solid GND, no vias if possible, no stubs. Join J2 A6/B6 and A7/B7 at the connector. U5 right at J2, then to PA11/PA12. R8/R9 near J2. SWD to J3 short."

Commit message: added comments. Grouped submodules in ways that make more sense
Parts:
- F1: value 500mA_PTC -> MF-MSMF050; footprint (none) -> Fuse:Fuse_1812_4532Metric; MPN (none) -> Bourns MF-MSMF050-2
- J2: footprint (none) -> Connector_USB:USB_C_Receptacle_GCT_USB4110; MPN (none) -> GCT USB4110-GF-A

Commit message: fixed minor errors
Parts:
- F1: value MF-MSMF050 -> MF-MSMF075; MPN Bourns MF-MSMF050-2 -> Bourns MF-MSMF075-2
Connections:
- net +3V3: now also U5.5 (VBUS)
- net VBUS: no longer U5.5 (VBUS)
Other:
- note added: "R39/R40 22R: series resistors on SWCLK/SWDIO. Damp ringing on the probe cable. They do not protect against a mis-plugged 5V probe (~50mA). Not critical (0R works). J3 must be keyed. U5 pin 5 on +3V3 (not VBUS): stops D+ back-feeding VBUS when unplugged."
- note removed: "R39/R40 22R: series resistors on SWCLK/SWDIO. Damp ringing on the probe cable and limit current into PA13/PA14 from ESD or a bad probe. Not critical (0R works)."

Commit message: Updated comments. Claude did an audit. Take it with huge grains of salt
Other:
- note added: "R39/R40 22R damp ringing on the SWD cable (0R also works). They do not protect against a mis-plugged 5V probe, so J3 must be keyed. U5 rail pin on +3V3 so an unplugged USB cable is detected. DESIGN_NOTES.md §7."
- note removed: "R39/R40 22R: series resistors on SWCLK/SWDIO. Damp ringing on the probe cable. They do not protect against a mis-plugged 5V probe (~50mA). Not critical (0R works). J3 must be keyed. U5 pin 5 on +3V3 (not VBUS): stops D+ back-feeding VBUS when unplugged."
Changed lines of the file:
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@@
 		)
 	)
-  (text "R39/R40 22R: series resistors on SWCLK/SWDIO.\nDamp ringing on the probe cable. They do not protect against a mis-plugged\n5V probe (~50mA). Not critical (0R works). J3 must be keyed.\nU5 pin 5 on +3V3 (not VBUS): stops D+ back-feeding VBUS when unplugged."
+  (text "R39/R40 22R damp ringing on the SWD cable (0R also works). They do not\nprotect against a mis-plugged 5V probe, so J3 must be keyed.\nU5 rail pin on +3V3 so an unplugged USB cable is detected.\nDESIGN_NOTES.md §7."
     (at 199.39 156.21 0)
     (effects (font (size 1.27 1.27)) (justify left bottom))

Commit message: boxing goes brrr
Parts:
- removed D8: BAT54_VTref, symbol Device:D_Schottky
- added D12: TVS0500DRV, symbol Power_Protection:TVS0500DRV
- F1: value MF-MSMF075 -> MF-MSMF075/16X; MPN Bourns MF-MSMF075-2 -> Bourns MF-MSMF075/16X-2
- U5: MPN (none) -> ST USBLC6-2SC6
Connections:
- net +3V3: now also J3.1 (Pin_1)
- net GND: now also D12.1 (GND), D12.2 (GND), D12.3 (GND), D12.7 (GND); no longer J2.SH (SHIELD)
- net at F1.2, J2.A4 (VBUS), J2.A9 (VBUS)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: now also D12.4 (IN), D12.5 (IN), D12.6 (IN)
- no-connect marks 2 -> 3
Other:
- note added: "SWD DEBUG J3, RESET AND BOOT BUTTONS"
- note added: "USB-C J2: TVS, FUSE, CC RESISTORS, ESD"
Changed lines of the file:
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@@
 		(color 0 0 0 0)
+	)
+	(junction
+		(at 99.06 99.06)
+		(diameter 0)
 	)
 	(no_connect
@@
 		(at 91.44 129.54)
 	)
+	(no_connect
+		(at 68.58 137.16)
+	)
 	(wire
 		(pts
@@
 	(wire
 		(pts
-			(xy 68.58 137.16)
-			(xy 63.5 137.16)
-		)
-		(stroke
-			(width 0)
-			(type default)
-		)
-	)
-	(wire
-		(pts
 			(xy 219.71 114.3)
 			(xy 228.6 114.3)
@@
 		)
 	)
-	(text "ROUTING - USB FS\nUSB_DP/USB_DM: 90R differential pair, length-matched within 1mm,\nover solid GND, no vias if possible, no stubs.\nJoin J2 A6/B6 and A7/B7 at the connector. U5 right at J2, then to PA11/PA12.\nR8/R9 near J2. SWD to J3 short."
-		(at 110.49 83.82 0)
+	(wire
+		(pts
+			(xy 212.09 102.87)
+			(xy 219.71 102.87)
+		)
+	)
+	(text "R39/R40 22R damp ringing on the SWD cable (0R also works). They do not\nprotect against a mis-plugged 5V probe, so J3 must be keyed.\nU5 rail pin on +3V3 so an unplugged USB cable is detected.\nDESIGN_NOTES.md §7."
+		(at 199.39 156.21 0)
 		(effects
 			(font
 				(size 1.27 1.27)
-				(bold yes)
-				(color 255 0 0 1)
 			)
 			(justify left bottom)
@@
 	)
 	(label "CC1"
-		(at 104.14 104.14 0)
+		(at 91.44 104.14 0)
 		(effects
 			(font
@@
 		)
 	)
-  (text "R39/R40 22R damp ringing on the SWD cable (0R also works). They do not\nprotect against a mis-plugged 5V probe, so J3 must be keyed.\nU5 rail pin on +3V3 so an unplugged USB cable is detected.\nDESIGN_NOTES.md §7."
-    (at 199.39 156.21 0)
-    (effects (font (size 1.27 1.27)) (justify left bottom))
+  (text "ROUTING - USB FS\nUSB_DP/USB_DM: 90R differential pair, length-matched within 1mm,\nover solid GND, no vias if possible, no stubs.\nJoin J2 A6/B6 and A7/B7 at the connector. U5 right at J2, then to PA11/PA12.\nR8/R9 near J2. SWD to J3 short."
+    (at 105.41 83.82 0)
+    (effects (font (size 1.27 1.27) (bold yes) (color 255 0 0 1)) (justify left bottom))
+  )
+  (text "USB-C J2: TVS, FUSE, CC RESISTORS, ESD"
+    (at 60.96 71.12 0)
+    (effects (font (size 2 2) (thickness 0.4) (bold yes) (color 0 0 132 1)) (justify left bottom))
+  )
+  (text "SWD DEBUG J3, RESET AND BOOT BUTTONS"
+    (at 191.77 91.44 0)
+    (effects (font (size 2 2) (thickness 0.4) (bold yes) (color 0 0 132 1)) (justify left bottom))
   )
 	(symbol
@@
 			)
 		)
-		(property "Description" "GCT USB4110-GF-A, USB 2.0 Type-C 16P SMT receptacle. VBUS 5A total, GND 6.25A total, 0.25A per signal pin, 48VDC, 20,000 cycles. Same series as the rev-2026 control board (C5143397). Footprint pads match the symbol (A1-B12, SH)."
+		(property "Description" "GCT USB4110-GF-A, USB 2.0 Type-C 16P SMT receptacle. VBUS 5A total, GND 6.25A total, 0.25A per signal pin. Shield (SH) left floating by design choice."
 			(at 76.2 114.3 0)
 			(hide yes)
@@
 	)
 	(symbol
-		(lib_id "Device:D_Schottky")
-		(at 215.9 102.87 180)
-		(unit 1)
-		(exclude_from_sim no)
-		(in_bom yes)
-		(on_board yes)
-		(dnp no)
-		(property "Reference" "D8"
-			(at 215.9 105.41 0)
-			(show_name no)
-			(do_not_autoplace no)
-			(effects
-				(font
-					(size 1.27 1.27)
-				)
-			)
-		)
-		(property "Value" "BAT54_VTref"
-			(at 215.9 100.33 0)
-			(show_name no)
-			(do_not_autoplace no)
-			(effects
-				(font
-					(size 1.27 1.27)
-				)
-			)
-		)
-		(property "Footprint" ""
-			(at 215.9 102.87 0)
-			(hide yes)
-			(show_name no)
-			(do_not_autoplace no)
-			(effects
-				(font
-					(size 1.27 1.27)
-				)
-			)
-		)
-		(property "Datasheet" ""
-			(at 215.9 102.87 0)
-			(hide yes)
-			(show_name no)
-			(do_not_autoplace no)
-			(effects
-				(font
-					(size 1.27 1.27)
-				)
-			)
-		)
-		(property "Description" "Schottky diode"
-			(at 215.9 102.87 0)
-			(hide yes)
-			(show_name no)
-			(do_not_autoplace no)
-			(effects
-				(font
-					(size 1.27 1.27)
-				)
-			)
-		)
-		(body_style 1)
-		(in_pos_files yes)
-		(pin "1"
-		)
-		(pin "2"
-		)
-		(instances
-			(project "ControlBoard2027"
-				(path "/2be89789-dd04-494d-960d-2531c7ce8a2f/b44198b9-a21d-475d-9b21-d8da342bbbd1"
-					(reference "D8")
-					(unit 1)
-				)
-			)
-		)
-	)
-	(symbol
 		(lib_id "Device:R")
 		(at 116.84 107.95 0)
@@
 			)
 		)
-	)
+		(property "MPN" "ST USBLC6-2SC6"
+			(at 152.4 119.38 0)
+			(hide yes)
+			(effects
+				(font
+					(size 1.27 1.27)
+				)
+			)
+		))
 	(symbol
 		(lib_id "Device:R")
@@
 	)
 	(symbol
-		(lib_id "power:GND")
-		(at 63.5 137.16 0)
-		(unit 1)
-		(exclude_from_sim no)
-		(in_bom yes)
-		(on_board yes)
-		(dnp no)
-		(property "Reference" "#PWR301"
-			(at 63.5 143.51 0)
-			(hide yes)
-			(show_name no)
-			(do_not_autoplace no)
-			(effects
-				(font
-					(size 1.27 1.27)
-				)
-			)
-		)
-		(property "Value" "GND"
-			(at 63.5 140.97 0)
-			(show_name no)
-			(do_not_autoplace no)
-			(effects
-				(font
-					(size 1.27 1.27)
-				)
-			)
-		)
-		(property "Footprint" ""
-			(at 63.5 137.16 0)
-			(hide yes)
-			(show_name no)
-			(do_not_autoplace no)
-			(effects
-				(font
-					(size 1.27 1.27)
-				)
-			)
-		)
-		(property "Datasheet" ""
-			(at 63.5 137.16 0)
-			(hide yes)
-			(show_name no)
-			(do_not_autoplace no)
-			(effects
-				(font
-					(size 1.27 1.27)
-				)
-			)
-		)
-		(property "Description" "Power symbol creates a global label with name \"GND\" , ground"
-			(at 63.5 137.16 0)
-			(hide yes)
-			(show_name no)
-			(do_not_autoplace no)
-			(effects
-				(font
-					(size 1.27 1.27)
-				)
-			)
-		)
-		(body_style 1)
-		(in_pos_files yes)
-		(pin "1"
-		)
-		(instances
-			(project "ControlBoard2027"
-				(path "/2be89789-dd04-494d-960d-2531c7ce8a2f/b44198b9-a21d-475d-9b21-d8da342bbbd1"
-					(reference "#PWR301")
-					(unit 1)
-				)
-			)
-		)
-	)
-	(symbol
 		(lib_id "Device:Polyfuse")
 		(at 110.49 99.06 270)
@@
 			)
 		)
-		(property "Value" "MF-MSMF075"
+		(property "Value" "MF-MSMF075/16X"
 			(at 110.49 101.6 90)
 			(show_name no)
@@
 			)
 		)
-		(property "Description" "Bourns MF-MSMF075-2 PTC, 1812, on USB VBUS. Ihold 0.75A / Itrip 1.50A at 23C, 0.60A hold at 50C, R 0.11-0.45 Ohm (Bourns derating table). U13 limits USB current to 0.455-0.560A first; F1 is backup for a U13 or cable short. MF-MSMF050 was replaced because its 0.40A hold at 50C tripped below U13's limit."
+		(property "Description" "USB VBUS PTC, 1812. Ihold 0.75A / Itrip 1.50A at 23C, 0.55A hold at 50C, 0.11-0.45 Ohm, 8A trips in 0.2s max (Bourns MF-MSMF Rev BD). Holds a USB 2.0 port's 0.5A and trips on a board or cable short. Motor modules on USB may trip it (DESIGN_NOTES.md §7)."
 			(at 110.49 99.06 0)
 			(hide yes)
@@
 			)
 		)
-		(property "MPN" "Bourns MF-MSMF075-2"
+		(property "MPN" "Bourns MF-MSMF075/16X-2"
 			(at 110.49 99.06 0)
 			(hide yes)
@@
 		)
 	)
+	(symbol
+		(lib_id "Power_Protection:TVS0500DRV")
+		(at 99.06 91.44 180)
+		(unit 1)
+		(in_bom yes)
+		(on_board yes)
+		(dnp no)
+		(property "Reference" "D12"
+			(at 96.52 92.71 0)
+			(effects
+				(font
+					(size 1.27 1.27)
+				)
+				(justify left)
+			)
+		)
+		(property "Value" "TVS0500DRV"
+			(at 96.52 90.17 0)
+			(effects
+				(font
+					(size 1.27 1.27)
+				)
+				(justify left)
+			)
+		)
+		(property "Footprint" ""
+			(at 99.06 91.44 0)
+			(hide yes)
+			(effects
+				(font
+					(size 1.27 1.27)
+				)
+			)
+		)
+		(property "Datasheet" "http://www.ti.com/lit/ds/symlink/tvs0500.pdf"
+			(at 99.06 91.44 0)
+			(hide yes)
+			(effects
+				(font
+					(size 1.27 1.27)
+				)
+			)
+		)
+		(property "Description" "USB VBUS TVS at J2, same part as D9/D10. TVS0500: VRWM 5V, VBR 7.5-8.4V, flat clamp 9.2V at 43A. Place right at J2 VBUS pins with a short GND via."
+			(at 99.06 91.44 0)
+			(hide yes)
+			(effects
+				(font
+					(size 1.27 1.27)
+				)
+			)
+		)
+		(instances
+			(project "ControlBoard2027"
+				(path "/2be89789-dd04-494d-960d-2531c7ce8a2f/b44198b9-a21d-475d-9b21-d8da342bbbd1"
+					(reference "D12")
+					(unit 1)
+				)
+			)
+		)
+		(property "MPN" "TI TVS0500DRVR"
+			(at 99.06 91.44 0)
+			(hide yes)
+			(effects
+				(font
+					(size 1.27 1.27)
+				)
+			)
+		))
+	(symbol
+		(lib_id "power:GND")
+		(at 99.06 83.82 180)
+		(unit 1)
+		(in_bom yes)
+		(on_board yes)
+		(dnp no)
+		(property "Reference" "#PWR313"
+			(at 99.06 77.47 0)
+			(hide yes)
+			(effects
+				(font
+					(size 1.27 1.27)
+				)
+			)
+		)
+		(property "Value" "GND"
+			(at 99.06 80.01 0)
+			(effects
+				(font
+					(size 1.27 1.27)
+				)
+			)
+		)
+		(property "Footprint" ""
+			(at 99.06 83.82 0)
+			(hide yes)
+			(effects
+				(font
+					(size 1.27 1.27)
+				)
+			)
+		)
+		(property "Datasheet" ""
+			(at 99.06 83.82 0)
+			(hide yes)
+			(effects
+				(font
+					(size 1.27 1.27)
+				)
+			)
+		)
+		(property "Description" "Power symbol creates a global label with name \"GND\" , ground"
+			(at 99.06 83.82 0)
+			(hide yes)
+			(effects
+				(font
+					(size 1.27 1.27)
+				)
+			)
+		)
+		(instances
+			(project "ControlBoard2027"
+				(path "/2be89789-dd04-494d-960d-2531c7ce8a2f/b44198b9-a21d-475d-9b21-d8da342bbbd1"
+					(reference "#PWR313")
+					(unit 1)
+				)
+			)
+		)
+	)
+	(rectangle
+		(start 60 67)
+		(end 186 153)
+		(stroke
+			(width 0.254)
+			(type dash)
+			(color 0 0 132 1)
+		)
+		(fill
+			(type none)
+		)
+	)
+	(rectangle
+		(start 190 88)
+		(end 278 159)
+		(stroke
+			(width 0.254)
+			(type dash)
+			(color 0 0 132 1)
+		)
+		(fill
+			(type none)
+		)
+	)

Commit message: updated schematics based on feedback
Parts:
- removed R39, R40: 22R, symbol Device:R
Connections:
- net SWCLK: now also J3.2 (Pin_2)
- net SWDIO: now also J3.3 (Pin_3)
Other:
- note added: "SWD: R39/R40 removed; direct SWCLK/SWDIO connections. Use short GND-referenced probe wiring; start SWCLK at 1MHz. Series damping is optional SI tuning, not required DC matching. NRST: internal 30-50k pull-up + C32 100nF (DS13313 section 6.3.17). J3 must be keyed. U5 rail pin stays on +3V3."
- note added: "USB POWER LIMIT: F1 holds 0.55A at 50C. ~0.85A concurrent base + Wi-Fi + LEDs exceeds this. Use powerboard for full operation; USB bench mode restricted. A larger fuse alone does not increase allowed USB current."
- note removed: "R39/R40 22R damp ringing on the SWD cable (0R also works). They do not protect against a mis-plugged 5V probe, so J3 must be keyed. U5 rail pin on +3V3 so an unplugged USB cable is detected. DESIGN_NOTES.md §7."
Changed lines of the file:
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@@
 		)
 	)
-	(text "R39/R40 22R damp ringing on the SWD cable (0R also works). They do not\nprotect against a mis-plugged 5V probe, so J3 must be keyed.\nU5 rail pin on +3V3 so an unplugged USB cable is detected.\nDESIGN_NOTES.md §7."
-		(at 199.39 156.21 0)
+	(wire
+		(pts
+			(xy 212.09 109.22)
+			(xy 219.71 109.22)
+		)
+	)
+	(wire
+		(pts
+			(xy 212.09 114.3)
+			(xy 219.71 114.3)
+		)
+	)
+	(text "ROUTING - USB FS\nUSB_DP/USB_DM: 90R differential pair, length-matched within 1mm,\nover solid GND, no vias if possible, no stubs.\nJoin J2 A6/B6 and A7/B7 at the connector. U5 right at J2, then to PA11/PA12.\nR8/R9 near J2. SWD to J3 short."
+		(at 105.41 83.82 0)
 		(effects
 			(font
 				(size 1.27 1.27)
+				(bold yes)
+				(color 255 0 0 1)
+			)
+			(justify left bottom)
+		)
+	)
+	(text "USB-C J2: TVS, FUSE, CC RESISTORS, ESD"
+		(at 60.96 71.12 0)
+		(effects
+			(font
+				(size 2 2)
+				(thickness 0.4)
+				(bold yes)
+				(color 0 0 132 1)
+			)
+			(justify left bottom)
+		)
+	)
+	(text "SWD DEBUG J3, RESET AND BOOT BUTTONS"
+		(at 191.77 91.44 0)
+		(effects
+			(font
+				(size 2 2)
+				(thickness 0.4)
+				(bold yes)
+				(color 0 0 132 1)
 			)
 			(justify left bottom)
@@
 		)
 	)
-  (text "ROUTING - USB FS\nUSB_DP/USB_DM: 90R differential pair, length-matched within 1mm,\nover solid GND, no vias if possible, no stubs.\nJoin J2 A6/B6 and A7/B7 at the connector. U5 right at J2, then to PA11/PA12.\nR8/R9 near J2. SWD to J3 short."
-    (at 105.41 83.82 0)
-    (effects (font (size 1.27 1.27) (bold yes) (color 255 0 0 1)) (justify left bottom))
+  (text "SWD: R39/R40 removed; direct SWCLK/SWDIO connections.\nUse short GND-referenced probe wiring; start SWCLK at 1MHz.\nSeries damping is optional SI tuning, not required DC matching.\nNRST: internal 30-50k pull-up + C32 100nF (DS13313 section 6.3.17).\nJ3 must be keyed. U5 rail pin stays on +3V3."
+    (at 199.39 156.21 0)
+    (effects (font (size 1.27 1.27)) (justify left bottom))
   )
-  (text "USB-C J2: TVS, FUSE, CC RESISTORS, ESD"
-    (at 60.96 71.12 0)
-    (effects (font (size 2 2) (thickness 0.4) (bold yes) (color 0 0 132 1)) (justify left bottom))
-  )
-  (text "SWD DEBUG J3, RESET AND BOOT BUTTONS"
-    (at 191.77 91.44 0)
-    (effects (font (size 2 2) (thickness 0.4) (bold yes) (color 0 0 132 1)) (justify left bottom))
+  (text "USB POWER LIMIT: F1 holds 0.55A at 50C.\n~0.85A concurrent base + Wi-Fi + LEDs exceeds this.\nUse powerboard for full operation; USB bench mode restricted.\nA larger fuse alone does not increase allowed USB current."
+    (at 60.96 170.18 0)
+    (effects (font (size 1.27 1.27)) (justify left bottom))
   )
 	(symbol
@@
 			)
 		)
-		(body_style 1)
-		(in_pos_files yes)
-		(pin "4"
-		)
-		(pin "2"
-		)
-		(pin "3"
-		)
-		(pin "6"
-		)
-		(pin "1"
-		)
-		(pin "5"
-		)
-		(instances
-			(project "ControlBoard2027"
-				(path "/2be89789-dd04-494d-960d-2531c7ce8a2f/b44198b9-a21d-475d-9b21-d8da342bbbd1"
-					(reference "U5")
-					(unit 1)
-				)
-			)
-		)
 		(property "MPN" "ST USBLC6-2SC6"
 			(at 152.4 119.38 0)
@@
 				)
 			)
-		))
+		)
+		(body_style 1)
+		(in_pos_files yes)
+		(pin "4"
+		)
+		(pin "2"
+		)
+		(pin "3"
+		)
+		(pin "6"
+		)
+		(pin "1"
+		)
+		(pin "5"
+		)
+		(instances
+			(project "ControlBoard2027"
+				(path "/2be89789-dd04-494d-960d-2531c7ce8a2f/b44198b9-a21d-475d-9b21-d8da342bbbd1"
+					(reference "U5")
+					(unit 1)
+				)
+			)
+		)
+	)
 	(symbol
 		(lib_id "Device:R")
@@
 			)
 		)
-		(property "Description" "USB VBUS PTC, 1812. Ihold 0.75A / Itrip 1.50A at 23C, 0.55A hold at 50C, 0.11-0.45 Ohm, 8A trips in 0.2s max (Bourns MF-MSMF Rev BD). Holds a USB 2.0 port's 0.5A and trips on a board or cable short. Motor modules on USB may trip it (DESIGN_NOTES.md §7)."
+		(property "Description" "Bourns MF-MSMF075/16X-2: 0.75A hold/1.5A trip at 23C; 0.55A hold at 50C. Retained for restricted USB bench use only. Estimated 0.85A concurrent board/radio/LED load exceeds hot hold and legacy USB allowance; see DESIGN_NOTES sections 4/7. Not an active current limiter."
 			(at 110.49 99.06 0)
 			(hide yes)
@@
 	)
 	(symbol
-		(lib_id "Device:R")
-		(at 215.9 109.22 90)
-		(unit 1)
-		(exclude_from_sim no)
-		(in_bom yes)
-		(on_board yes)
-		(dnp no)
-		(property "Reference" "R39"
-			(at 215.9 107.188 90)
-			(show_name no)
-			(do_not_autoplace no)
-			(effects
-				(font
-					(size 1.27 1.27)
-				)
-			)
-		)
-		(property "Value" "22R"
-			(at 215.9 109.22 90)
-			(show_name no)
-			(do_not_autoplace no)
-			(effects
-				(font
-					(size 1.27 1.27)
-				)
-			)
-		)
-		(property "Footprint" ""
-			(at 215.9 109.22 0)
-			(hide yes)
-			(show_name no)
-			(do_not_autoplace no)
-			(effects
-				(font
-					(size 1.27 1.27)
-				)
-			)
-		)
-		(property "Datasheet" ""
-			(at 215.9 109.22 0)
-			(hide yes)
-			(show_name no)
-			(do_not_autoplace no)
-			(effects
-				(font
-					(size 1.27 1.27)
-				)
-			)
-		)
-		(property "Description" "22R series on SWCLK. Damps ringing on the probe cable and limits current into PA14 from ESD or a mis-plugged probe. SWD is slow, so the value is not critical; 0R also works."
-			(at 215.9 109.22 0)
-			(hide yes)
-			(show_name no)
-			(do_not_autoplace no)
-			(effects
-				(font
-					(size 1.27 1.27)
-				)
-			)
-		)
-		(body_style 1)
-		(in_pos_files yes)
-		(pin "1"
-		)
-		(pin "2"
-		)
-		(instances
-			(project "ControlBoard2027"
-				(path "/2be89789-dd04-494d-960d-2531c7ce8a2f/b44198b9-a21d-475d-9b21-d8da342bbbd1"
-					(reference "R39")
-					(unit 1)
-				)
-			)
-		)
-	)
-	(symbol
 		(lib_id "power:GND")
 		(at 226.06 116.84 270)
@@
 	)
 	(symbol
-		(lib_id "Device:R")
-		(at 215.9 114.3 90)
-		(unit 1)
-		(exclude_from_sim no)
-		(in_bom yes)
-		(on_board yes)
-		(dnp no)
-		(property "Reference" "R40"
-			(at 215.9 112.268 90)
-			(show_name no)
-			(do_not_autoplace no)
-			(effects
-				(font
-					(size 1.27 1.27)
-				)
-			)
-		)
-		(property "Value" "22R"
-			(at 215.9 114.3 90)
-			(show_name no)
-			(do_not_autoplace no)
-			(effects
-				(font
-					(size 1.27 1.27)
-				)
-			)
-		)
-		(property "Footprint" ""
-			(at 215.9 114.3 0)
-			(hide yes)
-			(show_name no)
-			(do_not_autoplace no)
-			(effects
-				(font
-					(size 1.27 1.27)
-				)
-			)
-		)
-		(property "Datasheet" ""
-			(at 215.9 114.3 0)
-			(hide yes)
-			(show_name no)
-			(do_not_autoplace no)
-			(effects
-				(font
-					(size 1.27 1.27)
-				)
-			)
-		)
-		(property "Description" "22R series on SWDIO. Same role as R39: cable ringing damping and PA13 protection at the SWD header."
-			(at 215.9 114.3 0)
-			(hide yes)
-			(show_name no)
-			(do_not_autoplace no)
-			(effects
-				(font
-					(size 1.27 1.27)
-				)
-			)
-		)
-		(body_style 1)
-		(in_pos_files yes)
-		(pin "1"
-		)
-		(pin "2"
-		)
-		(instances
-			(project "ControlBoard2027"
-				(path "/2be89789-dd04-494d-960d-2531c7ce8a2f/b44198b9-a21d-475d-9b21-d8da342bbbd1"
-					(reference "R40")
-					(unit 1)
-				)
-			)
-		)
-	)
-	(symbol
 		(lib_id "power:+3V3")
 		(at 152.4 114.3 0)
@@
 			)
 		)
-		(instances
-			(project "ControlBoard2027"
-				(path "/2be89789-dd04-494d-960d-2531c7ce8a2f/b44198b9-a21d-475d-9b21-d8da342bbbd1"
-					(reference "D12")
-					(unit 1)
-				)
-			)
-		)
 		(property "MPN" "TI TVS0500DRVR"
 			(at 99.06 91.44 0)
@@
 				)
 			)
-		))
+		)
+		(instances
+			(project "ControlBoard2027"
+				(path "/2be89789-dd04-494d-960d-2531c7ce8a2f/b44198b9-a21d-475d-9b21-d8da342bbbd1"
+					(reference "D12")
+					(unit 1)
+				)
+			)
+		)
+	)
 	(symbol
 		(lib_id "power:GND")
