File: boards/develop-2027/controlboard/ControlBoard2027/03_USB_Debug.kicad_sch (KiCad schematic)
At the start: 10 parts, among them J2 USB-C_DFU, J3 SWD_5pin, SW1 RESET, SW2 BOOT0_DFU, U5 USBLC6-2SC6

Commit message: review changes
Parts:
- D1: renamed from D12; footprint (none) -> Package_SON:WSON-6-1EP_2x2mm_P0.65mm_EP1x1.6mm
- U3: renamed from U5; footprint (none) -> Package_TO_SOT_SMD:SOT-23-6
- renumbered R9 to R22, R8 to R23
Other:
- note added: "SWD is direct; damping depends on probe/cable edges and layout. DS13313 does not prescribe a universal 22R or 55R series resistor. NRST has an internal 30-50k pull-up; C32 = 100nF (DS13313 NRST data). U5 clamp rail is +3V3: validate rail injection and power-off behavior. USBLC6-2 DS4260 pinout/topology; short return path required."
- note added: "USB LAYOUT: keep DP/DM coupled over an uninterrupted ground reference. Join duplicate Type-C data contacts at J2; U5 close to connector. Final impedance/skew depend on stackup and PHY timing, not series R alone. DS4260 Figures 6/17: minimize ESD path inductance. No routed PCB yet."
- note added: "USB LOAD: MF-MSMF075/16X Ihold = 0.75 A at 23C, 0.55 A at 50C. Actual concurrent worst-case board/external current is not established. Restricted bench use until host current, startup and thermal budget are checked. F1 does not negotiate USB current; replacing it alone cannot approve more load."
- note removed: "ROUTING - USB FS USB_DP/USB_DM: 90R differential pair, length-matched within 1mm, over solid GND, no vias if possible, no stubs. Join J2 A6/B6 and A7/B7 at the connector. U5 right at J2, then to PA11/PA12. R8/R9 near J2. SWD to J3 short."
- note removed: "SWD: R39/R40 removed; direct SWCLK/SWDIO connections. Use short GND-referenced probe wiring; start SWCLK at 1MHz. Series damping is optional SI tuning, not required DC matching. NRST: internal 30-50k pull-up + C32 100nF (DS13313 section 6.3.17). J3 must be keyed. U5 rail pin stays on +3V3."
- note removed: "USB POWER LIMIT: F1 holds 0.55A at 50C. ~0.85A concurrent base + Wi-Fi + LEDs exceeds this. Use powerboard for full operation; USB bench mode restricted. A larger fuse alone does not increase allowed USB current."
