File: boards/develop-2027/controlboard/ControlBoard2027/09_Buttons.kicad_sch (KiCad schematic)
At the start: 12 parts, among them SW4 USER_BTN0, SW5 USER_BTN1, SW6 USER_BTN2

Commit message: post design review changes
post design review changes
Parts:
- R27, R28, R29: value 100R -> 10k
Connections:
- net BTN0_DB: no longer C37.1
- net BTN1_DB: no longer C38.1
- net BTN2_DB: no longer C39.1
- net USER_EXTI0: now also C37.1
- net USER_EXTI1: now also C38.1
- net USER_EXTI2: now also C39.1
Other:
- moved on the sheet: C37, C38, C39

Commit message: boxing goes brrr
Other:
- note added: "BUTTON DEBOUNCE (same for SW4, SW5, SW6) Pull-up R24/R25/R26 = 10k, series R27/R28/R29 = 10k, C37/C38/C39 = 100nF, no inductor. Press (C discharges through series R): tau = R27 x C37 = 10k x 100nF = 1.0ms Release (C charges through pull-up + series R): tau = (R24 + R27) x C37 = 20k x 100nF = 2.0ms With 1% resistors and 10% caps: press 0.9-1.1ms, release 1.8-2.2ms. Settles in ~5 tau. The RC remove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"
- note added: "USER BUTTONS SW4-SW6 WITH RC DEBOUNCE"
Changed lines of the file:
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@@
 		)
 	)
+  (text "BUTTON DEBOUNCE (same for SW4, SW5, SW6)\nPull-up R24/R25/R26 = 10k, series R27/R28/R29 = 10k, C37/C38/C39 = 100nF, no inductor.\nPress (C discharges through series R):   tau = R27 x C37 = 10k x 100nF = 1.0ms\nRelease (C charges through pull-up + series R):   tau = (R24 + R27) x C37 = 20k x 100nF = 2.0ms\nWith 1% resistors and 10% caps: press 0.9-1.1ms, release 1.8-2.2ms. Settles in ~5 tau.\nThe RC removes sub-millisecond bounce spikes; firmware ignores re-triggers for ~10ms.\nThe series R also limits current into the MCU pin from the discharging cap.\nDESIGN_NOTES.md §9."
+    (at 60.96 175.26 0)
+    (effects (font (size 1.27 1.27)) (justify left bottom))
+  )
+  (text "USER BUTTONS SW4-SW6 WITH RC DEBOUNCE"
+    (at 57.15 80.01 0)
+    (effects (font (size 2 2) (thickness 0.4) (bold yes) (color 0 0 132 1)) (justify left bottom))
+  )
 	(symbol
 		(lib_id "Switch:SW_Push")
@@
 		)
 	)
+	(rectangle
+		(start 56 76)
+		(end 168 180)
+		(stroke
+			(width 0.254)
+			(type dash)
+			(color 0 0 132 1)
+		)
+		(fill
+			(type none)
+		)
+	)

Commit message: review changes
Parts:
- renumbered C37 to C50, C38 to C51, C39 to C52, R24 to R59, R25 to R60, R26 to R61, R27 to R62, R28 to R63, R29 to R64
Other:
- note added: "BUTTONS: R24-R26 pull up with 10k; R27-R29 series 10k; C37-C39 = 100nF. Calculated nominal time constants: press 1 ms, release 2 ms. At +/-1% R and +/-10% C: 0.891-1.111 ms and 1.782-2.222 ms. These tolerances must be specified in the BOM; current generic values do not prove them. RC filtering does not guarantee removal of all bounce; qualify switch and firmware. Series R is between switch node a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"
- note removed: "BUTTON DEBOUNCE (same for SW4, SW5, SW6) Pull-up R24/R25/R26 = 10k, series R27/R28/R29 = 10k, C37/C38/C39 = 100nF, no inductor. Press (C discharges through series R): tau = R27 x C37 = 10k x 100nF = 1.0ms Release (C charges through pull-up + series R): tau = (R24 + R27) x C37 = 20k x 100nF = 2.0ms With 1% resistors and 10% caps: press 0.9-1.1ms, release 1.8-2.2ms. Settles in ~5 tau. The RC remove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"

Commit message: preliminary layout
Parts:
- C50, C51, C52: footprint (none) -> Capacitor_SMD:C_0402_1005Metric
- R59, R60, R61, R62, R63, R64: footprint (none) -> Resistor_SMD:R_0603_1608Metric
- SW4, SW5, SW6: footprint (none) -> Button_Switch_SMD:SW_SPST_TL3305A
Changed lines of the file:
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@@
 			)
 		)
-		(property "Footprint" ""
+		(property "Footprint" "Button_Switch_SMD:SW_SPST_TL3305A"
 			(at 71.12 96.52 0)
 			(hide yes)
@@
 			)
 		)
-		(property "Footprint" ""
+		(property "Footprint" "Button_Switch_SMD:SW_SPST_TL3305A"
 			(at 71.12 142.24 0)
 			(hide yes)
@@
 			)
 		)
-		(property "Footprint" ""
+		(property "Footprint" "Capacitor_SMD:C_0402_1005Metric"
 			(at 114.3 123.19 0)
 			(hide yes)
@@
 			)
 		)
-		(property "Footprint" ""
+		(property "Footprint" "Resistor_SMD:R_0603_1608Metric"
 			(at 81.28 115.57 0)
 			(hide yes)
@@
 			)
 		)
-		(property "Footprint" ""
+		(property "Footprint" "Resistor_SMD:R_0603_1608Metric"
 			(at 81.28 138.43 0)
 			(hide yes)
@@
 			)
 		)
-		(property "Footprint" ""
+		(property "Footprint" "Resistor_SMD:R_0603_1608Metric"
 			(at 105.41 119.38 0)
 			(hide yes)
@@
 			)
 		)
-		(property "Footprint" ""
+		(property "Footprint" "Capacitor_SMD:C_0402_1005Metric"
 			(at 114.3 146.05 0)
 			(hide yes)
@@
 			)
 		)
-		(property "Footprint" ""
+		(property "Footprint" "Button_Switch_SMD:SW_SPST_TL3305A"
 			(at 71.12 119.38 0)
 			(hide yes)
@@
 			)
 		)
-		(property "Footprint" ""
+		(property "Footprint" "Resistor_SMD:R_0603_1608Metric"
 			(at 105.41 96.52 0)
 			(hide yes)
@@
 			)
 		)
-		(property "Footprint" ""
+		(property "Footprint" "Capacitor_SMD:C_0402_1005Metric"
 			(at 114.3 100.33 0)
 			(hide yes)
@@
 			)
 		)
-		(property "Footprint" ""
+		(property "Footprint" "Resistor_SMD:R_0603_1608Metric"
 			(at 81.28 92.71 0)
 			(hide yes)
@@
 			)
 		)
-		(property "Footprint" ""
+		(property "Footprint" "Resistor_SMD:R_0603_1608Metric"
 			(at 105.41 142.24 0)
 			(hide yes)

Commit message: some routing fixes :)
Parts:
- SW4, SW5, SW6: footprint Button_Switch_SMD:SW_SPST_TL3305A -> Button_Switch_THT:SW_PUSH_1P1T_6x3.5mm_H4.3_APEM_MJTP1243; MPN (none) -> APEM MJTP1243
Changed lines of the file:
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@@
 			)
 		)
-		(property "Footprint" "Button_Switch_SMD:SW_SPST_TL3305A"
+		(property "Footprint" "Button_Switch_THT:SW_PUSH_1P1T_6x3.5mm_H4.3_APEM_MJTP1243"
 			(at 71.12 96.52 0)
 			(hide yes)
@@
 			)
 		)
-		(property "Datasheet" ""
+		(property "Datasheet" "https://www.apem.com/int/mjtp-series-1-1-1-1.html"
+			(at 71.12 96.52 0)
+			(hide yes)
+			(show_name no)
+			(do_not_autoplace no)
+			(effects
+				(font
+					(size 1.27 1.27)
+				)
+			)
+		)
+		(property "MPN" "APEM MJTP1243"
 			(at 71.12 96.52 0)
 			(hide yes)
@@
 			)
 		)
-		(property "Footprint" "Button_Switch_SMD:SW_SPST_TL3305A"
+		(property "Footprint" "Button_Switch_THT:SW_PUSH_1P1T_6x3.5mm_H4.3_APEM_MJTP1243"
 			(at 71.12 142.24 0)
 			(hide yes)
@@
 			)
 		)
-		(property "Datasheet" ""
+		(property "Datasheet" "https://www.apem.com/int/mjtp-series-1-1-1-1.html"
+			(at 71.12 142.24 0)
+			(hide yes)
+			(show_name no)
+			(do_not_autoplace no)
+			(effects
+				(font
+					(size 1.27 1.27)
+				)
+			)
+		)
+		(property "MPN" "APEM MJTP1243"
 			(at 71.12 142.24 0)
 			(hide yes)
@@
 			)
 		)
-		(property "Footprint" "Button_Switch_SMD:SW_SPST_TL3305A"
+		(property "Footprint" "Button_Switch_THT:SW_PUSH_1P1T_6x3.5mm_H4.3_APEM_MJTP1243"
 			(at 71.12 119.38 0)
 			(hide yes)
@@
 			)
 		)
-		(property "Datasheet" ""
+		(property "Datasheet" "https://www.apem.com/int/mjtp-series-1-1-1-1.html"
 			(at 71.12 119.38 0)
 			(hide yes)
+			(show_name no)
+			(do_not_autoplace no)
+			(effects
+				(font
+					(size 1.27 1.27)
+				)
+			)
+		)
+		(property "MPN" "APEM MJTP1243"
+			(at 71.12 119.38 0)
+			(hide yes)

Commit message: added VPNs to non-passives
Parts:
- SW4, SW5, SW6: Vendor PN (none) -> 679-2452-ND
Changed lines of the file:
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@@
+			)
+		)
+		(property "Description" "Push button switch, generic, two pins"
+			(at 71.12 96.52 0)
+			(hide yes)
+			(show_name no)
+			(do_not_autoplace no)
+			(effects
+				(font
+					(size 1.27 1.27)
+				)
 			)
 		)
@@
 			)
 		)
-		(property "Description" "Push button switch, generic, two pins"
+		(property "Vendor PN" "679-2452-ND"
 			(at 71.12 96.52 0)
 			(hide yes)
@@
 			)
 		)
+		(property "Description" "Push button switch, generic, two pins"
+			(at 71.12 142.24 0)
+			(hide yes)
+			(show_name no)
+			(do_not_autoplace no)
+			(effects
+				(font
+					(size 1.27 1.27)
+				)
+			)
+		)
 		(property "MPN" "APEM MJTP1243"
 			(at 71.12 142.24 0)
@@
 			)
 		)
-		(property "Description" "Push button switch, generic, two pins"
+		(property "Vendor PN" "679-2452-ND"
 			(at 71.12 142.24 0)
 			(hide yes)
@@
 			)
 		)
+		(property "Vendor PN" ""
+			(at 114.3 123.19 0)
+			(hide yes)
+			(show_name no)
+			(do_not_autoplace no)
+			(effects
+				(font
+					(size 1.27 1.27)
+				)
+			)
+		)
 		(pin "2"
 		)
@@
 			)
 		)
+		(property "Vendor PN" ""
+			(at 81.28 115.57 90)
+			(hide yes)
+			(show_name no)
+			(do_not_autoplace no)
+			(effects
+				(font
+					(size 1.27 1.27)
+				)
+			)
+		)
 		(pin "2"
 		)
@@
 			)
 		)
+		(property "Vendor PN" ""
+			(at 81.28 138.43 90)
+			(hide yes)
+			(show_name no)
+			(do_not_autoplace no)
+			(effects
+				(font
+					(size 1.27 1.27)
+				)
+			)
+		)
 		(pin "1"
 		)
@@
 			)
 		)
+		(property "Vendor PN" ""
+			(at 105.41 119.38 90)
+			(hide yes)
+			(show_name no)
+			(do_not_autoplace no)
+			(effects
+				(font
+					(size 1.27 1.27)
+				)
+			)
+		)
 		(pin "2"
 		)
@@
 			)
 		)
+		(property "Vendor PN" ""
+			(at 114.3 146.05 0)
+			(hide yes)
+			(show_name no)
+			(do_not_autoplace no)
+			(effects
+				(font
+					(size 1.27 1.27)
+				)
+			)
+		)
 		(pin "1"
 		)
@@
 			)
 		)
+		(property "Description" "Push button switch, generic, two pins"
+			(at 71.12 119.38 0)
+			(hide yes)
+			(show_name no)
+			(do_not_autoplace no)
+			(effects
+				(font
+					(size 1.27 1.27)
+				)
+			)
+		)
 		(property "MPN" "APEM MJTP1243"
 			(at 71.12 119.38 0)
@@
 			)
 		)
-		(property "Description" "Push button switch, generic, two pins"
+		(property "Vendor PN" "679-2452-ND"
 			(at 71.12 119.38 0)
 			(hide yes)
@@
 			)
 		)
+		(property "Vendor PN" ""
+			(at 105.41 96.52 90)
+			(hide yes)
+			(show_name no)
+			(do_not_autoplace no)
+			(effects
+				(font
+					(size 1.27 1.27)
+				)
+			)
+		)
 		(pin "2"
 		)
@@
 			)
 		)
+		(property "Vendor PN" ""
+			(at 114.3 100.33 0)
+			(hide yes)
+			(show_name no)
+			(do_not_autoplace no)
+			(effects
+				(font
+					(size 1.27 1.27)
+				)
+			)
+		)
 		(pin "1"
 		)
@@
 			)
 		)
+		(property "Vendor PN" ""
+			(at 81.28 92.71 90)
+			(hide yes)
+			(show_name no)
+			(do_not_autoplace no)
+			(effects
+				(font
+					(size 1.27 1.27)
+				)
+			)
+		)
 		(pin "1"
 		)
@@
 			(hide yes)
 			(show_name no)
+			(do_not_autoplace no)
+			(effects
+				(font
+					(size 1.27 1.27)
+				)
+			)
+		)
+		(property "Vendor PN" ""
+			(at 105.41 142.24 90)
+			(hide yes)
+			(show_name no)

Commit message: final changes
Parts:
- C50, C51, C52: Rating (none) -> 16V X7R
- R59, R60, R61, R62, R63, R64: Rating (none) -> 1%
Other:
- note added: "BUTTONS: R59-R61 pull up with 10k; R62-R64 series 10k; C50-C52 = 100nF. Calculated nominal time constants: press 1 ms, release 2 ms. At +/-1% R and +/-10% C: 0.891-1.111 ms and 1.782-2.222 ms. BOM: R59-R64 are 1%; C50-C52 need a +/-10% X7R part. RC filtering does not guarantee removal of all bounce; qualify switch and firmware. Series R is between switch node and MCU/cap node, not between cap and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"
- note removed: "BUTTONS: R24-R26 pull up with 10k; R27-R29 series 10k; C37-C39 = 100nF. Calculated nominal time constants: press 1 ms, release 2 ms. At +/-1% R and +/-10% C: 0.891-1.111 ms and 1.782-2.222 ms. These tolerances must be specified in the BOM; current generic values do not prove them. RC filtering does not guarantee removal of all bounce; qualify switch and firmware. Series R is between switch node a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"
Changed lines of the file:
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@@
-		)
-	)
-	(text "BUTTONS: R24-R26 pull up with 10k; R27-R29 series 10k; C37-C39 = 100nF.\nCalculated nominal time constants: press 1 ms, release 2 ms.\nAt +/-1% R and +/-10% C: 0.891-1.111 ms and 1.782-2.222 ms.\nThese tolerances must be specified in the BOM; current generic values do not prove them.\nRC filtering does not guarantee removal of all bounce; qualify switch and firmware.\nSeries R is between switch node and MCU/cap node, not between cap and MCU.\nInput leakage check uses STM32H723 DS13313 Table 51."
-		(exclude_from_sim no)
-		(at 60.96 175.26 0)
-		(effects
-			(font
-				(size 1.1 1.1)
-			)
-			(justify left bottom)
 		)
 	)
@@
 		)
 	)
+  (text "BUTTONS: R59-R61 pull up with 10k; R62-R64 series 10k; C50-C52 = 100nF.\nCalculated nominal time constants: press 1 ms, release 2 ms.\nAt +/-1% R and +/-10% C: 0.891-1.111 ms and 1.782-2.222 ms.\nBOM: R59-R64 are 1%; C50-C52 need a +/-10% X7R part.\nRC filtering does not guarantee removal of all bounce; qualify switch and firmware.\nSeries R is between switch node and MCU/cap node, not between cap and MCU.\nInput leakage check uses STM32H723 DS13313 Table 51."
+    (at 60.96 175.26 0)
+    (effects (font (size 1.1 1.1)) (justify left bottom))
+  )
 	(symbol
 		(lib_id "Switch:SW_Push")
@@
 			)
 		)
-		(property "Datasheet" "https://www.apem.com/int/mjtp-series-1-1-1-1.html"
+		(property "Datasheet" "https://www.farnell.com/datasheets/1598766.pdf"
 			(at 71.12 96.52 0)
 			(hide yes)
@@
 			)
 		)
-		(property "Datasheet" "https://www.apem.com/int/mjtp-series-1-1-1-1.html"
+		(property "Datasheet" "https://www.farnell.com/datasheets/1598766.pdf"
 			(at 71.12 142.24 0)
 			(hide yes)
@@
 			)
 		)
-		(property "Description" "Debounce cap at the MCU pin side of R28."
+		(property "Description" "Debounce cap at the MCU pin side of R63."
 			(at 114.3 123.19 0)
 			(hide yes)
@@
 			)
 		)
-	)
+		(property "Rating" "16V X7R"
+			(at 114.3 123.19 0)
+			(hide yes)
+			(effects
+				(font
+					(size 1.27 1.27)
+				)
+			)
+		))
 	(symbol
 		(lib_id "Device:R")
@@
 			)
 		)
-	)
+		(property "Rating" "1%"
+			(at 81.28 115.57 0)
+			(hide yes)
+			(effects
+				(font
+					(size 1.27 1.27)
+				)
+			)
+		))
 	(symbol
 		(lib_id "power:GND")
@@
 			)
 		)
-	)
+		(property "Rating" "1%"
+			(at 81.28 138.43 0)
+			(hide yes)
+			(effects
+				(font
+					(size 1.27 1.27)
+				)
+			)
+		))
 	(symbol
 		(lib_id "Device:R")
@@
 			)
 		)
-		(property "Description" "Debounce R, see R27."
+		(property "Description" "Debounce R, see R62."
 			(at 105.41 119.38 0)
 			(hide yes)
@@
 			)
 		)
-	)
+		(property "Rating" "1%"
+			(at 105.41 119.38 0)
+			(hide yes)
+			(effects
+				(font
+					(size 1.27 1.27)
+				)
+			)
+		))
 	(symbol
 		(lib_id "Device:C")
@@
 			)
 		)
-		(property "Description" "Debounce cap at the MCU pin side of R29."
+		(property "Description" "Debounce cap at the MCU pin side of R64."
 			(at 114.3 146.05 0)
 			(hide yes)
@@
 			)
 		)
-	)
+		(property "Rating" "16V X7R"
+			(at 114.3 146.05 0)
+			(hide yes)
+			(effects
+				(font
+					(size 1.27 1.27)
+				)
+			)
+		))
 	(symbol
 		(lib_id "power:+3V3")
@@
 			)
 		)
-		(property "Datasheet" "https://www.apem.com/int/mjtp-series-1-1-1-1.html"
+		(property "Datasheet" "https://www.farnell.com/datasheets/1598766.pdf"
 			(at 71.12 119.38 0)
 			(hide yes)
@@
 			)
 		)
-		(property "Description" "Debounce R. SW press: C37 discharges through 10k (tau 1ms); release: 20k (tau 2ms). Limits switch current."
+		(property "Description" "Debounce R. SW press: C50 discharges through 10k (tau 1ms); release: 20k (tau 2ms). Limits switch current."
 			(at 105.41 96.52 0)
 			(hide yes)
@@
 			)
 		)
-	)
+		(property "Rating" "1%"
+			(at 105.41 96.52 0)
+			(hide yes)
+			(effects
+				(font
+					(size 1.27 1.27)
+				)
+			)
+		))
 	(symbol
 		(lib_id "Device:C")
@@
 			)
 		)
-		(property "Description" "Debounce cap at the MCU pin side of R27."
+		(property "Description" "Debounce cap at the MCU pin side of R62."
 			(at 114.3 100.33 0)
 			(hide yes)
@@
 			)
 		)
-	)
+		(property "Rating" "16V X7R"
+			(at 114.3 100.33 0)
+			(hide yes)
+			(effects
+				(font
+					(size 1.27 1.27)
+				)
+			)
+		))
 	(symbol
 		(lib_id "Device:R")
@@
 			)
 		)
-	)
+		(property "Rating" "1%"
+			(at 81.28 92.71 0)
+			(hide yes)
+			(effects
+				(font
+					(size 1.27 1.27)
+				)
+			)
+		))
 	(symbol
 		(lib_id "power:+3V3")
@@
 			)
 		)
-		(property "Description" "Debounce R, see R27."
+		(property "Description" "Debounce R, see R62."
 			(at 105.41 142.24 0)
 			(hide yes)
@@
 			)
 		)
-	)
+		(property "Rating" "1%"
+			(at 105.41 142.24 0)
+			(hide yes)
+			(effects
+				(font
+					(size 1.27 1.27)
+				)
+			)
+		))
 	(symbol
 		(lib_id "power:GND")
