File: boards/develop-2027/controlboard/RadioBoard2027/RadioBoard2027.kicad_sch (KiCad schematic)
At the start: 0 parts

Commit message: radioboard fixes
Other:
- sheet Controlboard Link ports: added ESP_DATA_READY, ESP_EN, ESP_HANDSHAKE, ESP_SPI_CS, ESP_SPI_MISO, ESP_SPI_MOSI, ESP_SPI_SCK; removed none
- sheet ESP32-C5 ports: added ESP_DATA_READY, ESP_EN, ESP_HANDSHAKE, ESP_SPI_CS, ESP_SPI_MISO, ESP_SPI_MOSI, ESP_SPI_SCK, PWR_SRC_HOST, USB_DN, USB_DP; removed none
- sheet Power ports: added PWR_SRC_HOST; removed none
- sheet USB ports: added USB_DN, USB_DP; removed none
- note added: "RADIOBOARD2027 - ESP32-C5 Wi-Fi co-processor for ControlBoard2027 (ESP-Hosted over SPI) Power: controlboard +3V3 over the J2 cable, or USB-C alone for flashing (TPS2116 mux). Signals cross sheets through sheet pins (hierarchical labels); rails (+3V3_HOST, GND) use global labels and power symbols. Design justification: DESIGN_NOTES.md."
- note removed: "RADIOBOARD2027 - ESP32-C5 Wi-Fi co-processor for ControlBoard2027 (ESP-Hosted over SPI) Power: controlboard +3V3 over the J2 cable, or USB-C alone for flashing (TPS2116 mux). Cross-sheet nets use global labels. Design justification: DESIGN_NOTES.md."
