File: boards/develop-2027/controlboard/RadioBoard2027/03_USB.kicad_sch (KiCad schematic)
At the start: 6 parts, among them J1 USB_C, U2 USBLC6-2SC6

Commit message: Preliminary daughterboard layout
Parts:
- D2: footprint (none) -> Package_SON:WSON-6-1EP_2x2mm_P0.65mm_EP1x1.6mm
- F1: value MF-MSMF075/16X -> MF-MSMF075/33X; MPN Bourns MF-MSMF075/16X-2 -> Bourns MF-MSMF075/33X-2
- R10, R9: footprint (none) -> Resistor_SMD:R_0402_1005Metric
- U2: footprint (none) -> Package_TO_SOT_SMD:SOT-23-6
Other:
- note added: "ROUTING - USB USB_DP/USB_DN 90R differential, in parallel at equal length. Join A6/B6 and A7/B7 at J1. U2 right at J1, D2 right at J1 VBUS, short GND vias."
- note removed: "ROUTING - USB USB_DP/USB_DN 90R differential, length-matched within 1mm. Join A6/B6 and A7/B7 at J1. U2 right at J1, D2 right at J1 VBUS, short GND vias."
Changed lines of the file:
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@@
     (effects (font (size 1.27 1.27)) (justify left bottom))
-  )
-  (text "ROUTING - USB\nUSB_DP/USB_DN 90R differential, length-matched within 1mm. Join A6/B6 and A7/B7 at J1.\nU2 right at J1, D2 right at J1 VBUS, short GND vias."
-    (at 71.12 208.28 0)
-    (effects (font (size 1.27 1.27) (bold yes) (color 255 0 0 1)) (justify left bottom))
   )
   (text "USB-C J1: TVS, FUSE, CC, ESD"
@@
     (effects (font (size 2 2) (thickness 0.4) (bold yes) (color 0 0 132 1)) (justify left bottom))
   )
+  (text "ROUTING - USB\nUSB_DP/USB_DN 90R differential, in parallel at equal length. Join A6/B6 and A7/B7 at J1.\nU2 right at J1, D2 right at J1 VBUS, short GND vias."
+    (at 71.12 208.28 0)
+    (effects (font (size 1.27 1.27) (bold yes) (color 255 0 0 1)) (justify left bottom))
+  )
 	(symbol
 		(lib_id "Connector:USB_C_Receptacle_USB2.0_16P")
@@
 			)
 		)
-		(property "Footprint" ""
+		(property "Footprint" "Resistor_SMD:R_0402_1005Metric"
 			(at 132.08 144.78 0)
 			(hide yes)
@@
 			)
 		)
-		(property "Footprint" ""
+		(property "Footprint" "Resistor_SMD:R_0402_1005Metric"
 			(at 121.92 144.78 0)
 			(hide yes)
@@
 			)
 		)
-		(property "Footprint" ""
+		(property "Footprint" "Package_TO_SOT_SMD:SOT-23-6"
 			(at 172.72 160.02 0)
 			(hide yes)
@@
 			)
 		)
-		(property "Footprint" ""
+		(property "Footprint" "Package_SON:WSON-6-1EP_2x2mm_P0.65mm_EP1x1.6mm"
 			(at 121.92 116.84 0)
 			(hide yes)
@@
 			)
 		)
-		(property "Value" "MF-MSMF075/16X"
+		(property "Value" "MF-MSMF075/33X"
 			(at 142.24 127 90)
 			(effects
@@
 			)
 		)
-		(property "Description" "USB VBUS PTC. Hold 0.75A (0.55A at 50C), trip 1.50A (Bourns MF-MSMF Rev BD). Module peak 403mA fits under the hold current."
+		(property "Description" "USB VBUS PTC. Hold 0.75A (0.56A at 50C), trip 1.50A, 33V (Bourns MF-MSMF Rev BD). /33X used because /16X is not stocked at LCSC. Module peak 403mA fits under the hold current."
 			(at 142.24 124.46 0)
 			(hide yes)
@@
 			)
 		)
-		(property "MPN" "Bourns MF-MSMF075/16X-2"
+		(property "MPN" "Bourns MF-MSMF075/33X-2"
 			(at 142.24 124.46 0)
 			(hide yes)

Commit message: radioboard fixes
Parts:
- D2: LCSC (none) -> C609571
- F1: LCSC (none) -> C3760814
- J1: LCSC (none) -> C5143397
- R10, R9: LCSC (none) -> C25905; MPN (none) -> UniOhm 0402WGF5101TCE; Rating (none) -> 1%
- U2: LCSC (none) -> C7519
Other:
- note added: "ROUTING - USB J1 -> U2 (flow-through) -> R5/R6 -> module in one direction, no vias; Full-Speed, so 90R coupling is not required. Join A6/B6 and A7/B7 at J1. U2 right at J1, D2 right at J1 VBUS, short GND vias."
- note removed: "ROUTING - USB USB_DP/USB_DN 90R differential, in parallel at equal length. Join A6/B6 and A7/B7 at J1. U2 right at J1, D2 right at J1 VBUS, short GND vias."
Changed lines of the file:
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@@
+		)
+	)
+	(text "USB-C J1\nNative USB Serial/JTAG on GPIO13/14 for flashing and logs; no USB-UART bridge.\nCC 5.1k Rd = sink. Shell floating, same as ControlBoard2027.\nD2 surge clamp and F1 PTC on VBUS; VBUS feeds only the U4 LDO.\nDESIGN_NOTES.md §4."
+		(at 71.12 195.58 0)
+		(effects
+			(font
+				(size 1.27 1.27)
+			)
+			(justify left bottom)
+		)
+	)
+	(text "USB-C J1: TVS, FUSE, CC, ESD"
+		(at 69.85 96.52 0)
+		(effects
+			(font
+				(size 2 2)
+				(thickness 0.4)
+				(bold yes)
+				(color 0 0 132 1)
+			)
+			(justify left bottom)
 		)
 	)
@@
 		)
 	)
-	(global_label "USB_DN"
-		(shape input)
+	(hierarchical_label "USB_DN"
+		(shape bidirectional)
 		(at 180.34 160.02 0)
 		(effects
@@
 		)
 	)
-	(global_label "USB_DP"
-		(shape input)
+	(hierarchical_label "USB_DP"
+		(shape bidirectional)
 		(at 180.34 162.56 0)
 		(effects
@@
 		)
 	)
-  (text "USB-C J1\nNative USB Serial/JTAG on GPIO13/14 for flashing and logs; no USB-UART bridge.\nCC 5.1k Rd = sink. Shell floating, same as ControlBoard2027.\nD2 surge clamp and F1 PTC on VBUS; VBUS feeds only the U4 LDO.\nDESIGN_NOTES.md §4."
-    (at 71.12 195.58 0)
-    (effects (font (size 1.27 1.27)) (justify left bottom))
-  )
-  (text "USB-C J1: TVS, FUSE, CC, ESD"
-    (at 69.85 96.52 0)
-    (effects (font (size 2 2) (thickness 0.4) (bold yes) (color 0 0 132 1)) (justify left bottom))
-  )
-  (text "ROUTING - USB\nUSB_DP/USB_DN 90R differential, in parallel at equal length. Join A6/B6 and A7/B7 at J1.\nU2 right at J1, D2 right at J1 VBUS, short GND vias."
+  (text "ROUTING - USB\nJ1 -> U2 (flow-through) -> R5/R6 -> module in one direction, no vias; Full-Speed, so 90R coupling is not required.\nJoin A6/B6 and A7/B7 at J1. U2 right at J1, D2 right at J1 VBUS, short GND vias."
     (at 71.12 208.28 0)
     (effects (font (size 1.27 1.27) (bold yes) (color 255 0 0 1)) (justify left bottom))
@@
 			)
 		)
-		(property "Datasheet" "https://www.usb.org/sites/default/files/documents/usb_type-c.zip"
+		(property "Datasheet" "https://www.lcsc.com/product-detail/C5143397.html"
 			(at 88.9 139.7 0)
 			(hide yes)
@@
 		)
 		(property "Description" "USB-C for programming (native USB Serial/JTAG) and standalone power. Same part as ControlBoard2027 J2. Shield left floating."
+			(at 88.9 139.7 0)
+			(hide yes)
+			(effects
+				(font
+					(size 1.27 1.27)
+				)
+			)
+		)
+		(property "MPN" "GCT USB4110-GF-A"
 			(at 88.9 139.7 0)
 			(hide yes)
@@
 			)
 		)
-		(property "MPN" "GCT USB4110-GF-A"
+		(property "LCSC" "C5143397"
 			(at 88.9 139.7 0)
 			(hide yes)
@@
 			)
 		)
-		(property "Datasheet" ""
+		(property "Datasheet" "https://www.lcsc.com/product-detail/C25905.html"
 			(at 132.08 144.78 0)
 			(hide yes)
@@
 			)
 		)
-	)
+		(property "LCSC" "C25905"
+			(at 132.08 144.78 0)
+			(hide yes)
+			(effects
+				(font
+					(size 1.27 1.27)
+				)
+			)
+		)
+		(property "MPN" "UniOhm 0402WGF5101TCE"
+			(at 132.08 144.78 0)
+			(hide yes)
+			(effects
+				(font
+					(size 1.27 1.27)
+				)
+			)
+		)
+		(property "Rating" "1%"
+			(at 132.08 144.78 0)
+			(hide yes)
+			(effects
+				(font
+					(size 1.27 1.27)
+				)
+			)
+		))
 	(symbol
 		(lib_id "Device:R")
@@
 			)
 		)
-		(property "Datasheet" ""
+		(property "Datasheet" "https://www.lcsc.com/product-detail/C25905.html"
 			(at 121.92 144.78 0)
 			(hide yes)
@@
 			)
 		)
-	)
+		(property "LCSC" "C25905"
+			(at 121.92 144.78 0)
+			(hide yes)
+			(effects
+				(font
+					(size 1.27 1.27)
+				)
+			)
+		)
+		(property "MPN" "UniOhm 0402WGF5101TCE"
+			(at 121.92 144.78 0)
+			(hide yes)
+			(effects
+				(font
+					(size 1.27 1.27)
+				)
+			)
+		)
+		(property "Rating" "1%"
+			(at 121.92 144.78 0)
+			(hide yes)
+			(effects
+				(font
+					(size 1.27 1.27)
+				)
+			)
+		))
 	(symbol
 		(lib_id "Power_Protection:USBLC6-2SC6")
@@
 			)
 		)
+		(property "MPN" "ST USBLC6-2SC6"
+			(at 172.72 160.02 0)
+			(hide yes)
+			(effects
+				(font
+					(size 1.27 1.27)
+				)
+			)
+		)
 		(instances
 			(project "RadioBoard2027"
@@
 			)
 		)
-		(property "MPN" "ST USBLC6-2SC6"
+		(property "LCSC" "C7519"
 			(at 172.72 160.02 0)
 			(hide yes)
@@
 			)
 		)
+		(property "MPN" "TI TVS0500DRVR"
+			(at 121.92 116.84 0)
+			(hide yes)
+			(effects
+				(font
+					(size 1.27 1.27)
+				)
+			)
+		)
 		(instances
 			(project "RadioBoard2027"
@@
 			)
 		)
-		(property "MPN" "TI TVS0500DRVR"
+		(property "LCSC" "C609571"
 			(at 121.92 116.84 0)
 			(hide yes)
@@
 			)
 		)
-		(property "Datasheet" ""
+		(property "Datasheet" "https://www.bourns.com/docs/product-datasheets/mf-msmf.pdf"
 			(at 142.24 124.46 0)
 			(hide yes)
@@
 		)
 		(property "Description" "USB VBUS PTC. Hold 0.75A (0.56A at 50C), trip 1.50A, 33V (Bourns MF-MSMF Rev BD). /33X used because /16X is not stocked at LCSC. Module peak 403mA fits under the hold current."
+			(at 142.24 124.46 0)
+			(hide yes)
+			(effects
+				(font
+					(size 1.27 1.27)
+				)
+			)
+		)
+		(property "MPN" "Bourns MF-MSMF075/33X-2"
 			(at 142.24 124.46 0)
 			(hide yes)
@@
 			)
 		)
-		(property "MPN" "Bourns MF-MSMF075/33X-2"
+		(property "LCSC" "C3760814"
 			(at 142.24 124.46 0)
 			(hide yes)

Commit message: radioboard parts goes brrr
Parts:
- D2: Vendor PN (none) -> 296-48382-1-ND
- F1: Vendor PN (none) -> 118-MF-MSMF075/33X-2CT-ND
- J1: Vendor PN (none) -> 2073-USB4110-GF-A-1-ND
- R10, R9: LCSC C25905 -> (none); MPN UniOhm 0402WGF5101TCE -> Yageo RC0402FR-075K1L; Vendor PN (none) -> 311-5.10KLRCT-ND
- U2: Vendor PN (none) -> 497-5235-1-ND
Changed lines of the file:
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@@
 			)
 		)
-		(property "Datasheet" "https://www.lcsc.com/product-detail/C5143397.html"
+		(property "Datasheet" "https://gct.co/files/drawings/usb4110.pdf"
 			(at 88.9 139.7 0)
 			(hide yes)
@@
 		)
 		(property "LCSC" "C5143397"
+			(at 88.9 139.7 0)
+			(hide yes)
+			(effects
+				(font
+					(size 1.27 1.27)
+				)
+			)
+		)
+		(property "Vendor PN" "2073-USB4110-GF-A-1-ND"
 			(at 88.9 139.7 0)
 			(hide yes)
@@
 			)
 		)
-		(property "Datasheet" "https://www.lcsc.com/product-detail/C25905.html"
+		(property "Datasheet" "https://www.digikey.com/en/products/detail/yageo/RC0402FR-075K1L/726624"
 			(at 132.08 144.78 0)
 			(hide yes)
@@
 			)
 		)
-		(property "LCSC" "C25905"
-			(at 132.08 144.78 0)
-			(hide yes)
-			(effects
-				(font
-					(size 1.27 1.27)
-				)
-			)
-		)
-		(property "MPN" "UniOhm 0402WGF5101TCE"
+		(property "LCSC" ""
+			(at 132.08 144.78 0)
+			(hide yes)
+			(effects
+				(font
+					(size 1.27 1.27)
+				)
+			)
+		)
+		(property "MPN" "Yageo RC0402FR-075K1L"
 			(at 132.08 144.78 0)
 			(hide yes)
@@
 		)
 		(property "Rating" "1%"
+			(at 132.08 144.78 0)
+			(hide yes)
+			(effects
+				(font
+					(size 1.27 1.27)
+				)
+			)
+		)
+		(property "Vendor PN" "311-5.10KLRCT-ND"
 			(at 132.08 144.78 0)
 			(hide yes)
@@
 			)
 		)
-		(property "Datasheet" "https://www.lcsc.com/product-detail/C25905.html"
+		(property "Datasheet" "https://www.digikey.com/en/products/detail/yageo/RC0402FR-075K1L/726624"
 			(at 121.92 144.78 0)
 			(hide yes)
@@
 			)
 		)
-		(property "LCSC" "C25905"
-			(at 121.92 144.78 0)
-			(hide yes)
-			(effects
-				(font
-					(size 1.27 1.27)
-				)
-			)
-		)
-		(property "MPN" "UniOhm 0402WGF5101TCE"
+		(property "LCSC" ""
+			(at 121.92 144.78 0)
+			(hide yes)
+			(effects
+				(font
+					(size 1.27 1.27)
+				)
+			)
+		)
+		(property "MPN" "Yageo RC0402FR-075K1L"
 			(at 121.92 144.78 0)
 			(hide yes)
@@
 		)
 		(property "Rating" "1%"
+			(at 121.92 144.78 0)
+			(hide yes)
+			(effects
+				(font
+					(size 1.27 1.27)
+				)
+			)
+		)
+		(property "Vendor PN" "311-5.10KLRCT-ND"
 			(at 121.92 144.78 0)
 			(hide yes)
@@
 				)
 			)
+		)
+		(property "Vendor PN" "497-5235-1-ND"
+			(at 172.72 160.02 0)
+			(hide yes)
+			(effects
+				(font
+					(size 1.27 1.27)
+				)
+			)
 		))
 	(symbol
@@
 				)
 			)
+		)
+		(property "Vendor PN" "296-48382-1-ND"
+			(at 121.92 116.84 0)
+			(hide yes)
+			(effects
+				(font
+					(size 1.27 1.27)
+				)
+			)
 		))
 	(symbol
@@
 			)
 		)
-		(property "Description" "USB VBUS PTC. Hold 0.75A (0.56A at 50C), trip 1.50A, 33V (Bourns MF-MSMF Rev BD). /33X used because /16X is not stocked at LCSC. Module peak 403mA fits under the hold current."
+		(property "Description" "USB VBUS PTC. Hold 0.75A (0.56A at 50C), trip 1.50A, 33V (Bourns MF-MSMF Rev BD). Module peak 403mA fits under the hold current."
 			(at 142.24 124.46 0)
 			(hide yes)
@@
 			(at 142.24 124.46 0)
 			(hide yes)
+			(effects
+				(font
+					(size 1.27 1.27)
+				)
+			)
+		)
+		(property "Vendor PN" "118-MF-MSMF075/33X-2CT-ND"
+			(at 142.24 124.46 0)
+			(hide yes)
