File: boards/develop-2027/controlboard/RadioBoard2027/RadioBoard2027.kicad_pcb (KiCad board)
At the start: 2 copper layers, 0 parts

Commit message: Preliminary daughterboard layout
Parts:
- added C1: 22uF 25V, Capacitor_SMD:C_0805_2012Metric, F.Cu at (107.0, 102.3)
- added C2: 100nF, Capacitor_SMD:C_0402_1005Metric, F.Cu at (107.5, 104.6)
- added C3: 1uF, Capacitor_SMD:C_0402_1005Metric, F.Cu at (104.4, 106.3)
- added C4: 15pF DNP, Capacitor_SMD:C_0402_1005Metric, F.Cu at (132.0, 121.5)
- added C5: 4.7uF 25V, Capacitor_SMD:C_0805_2012Metric, F.Cu at (113.0, 135.5)
- added C6: 10uF 10V, Capacitor_SMD:C_0603_1608Metric, F.Cu at (121.0, 134.3)
- added C7: 10uF 10V, Capacitor_SMD:C_0603_1608Metric, F.Cu at (119.6, 138.5)
- added C8: 22uF 25V, Capacitor_SMD:C_0805_2012Metric, F.Cu at (125.8, 138.5)
- added C9: 100nF, Capacitor_SMD:C_0402_1005Metric, F.Cu at (127.8, 138.5)
- added D1: GREEN, LED_SMD:LED_0603_1608Metric, F.Cu at (132.5, 112.0)
- added D2: TVS0500DRV, Package_SON:WSON-6-1EP_2x2mm_P0.65mm_EP1x1.6mm, F.Cu at (111.8, 126.5)
- added D3: RED, LED_SMD:LED_0603_1608Metric, F.Cu at (132.5, 117.0)
- added D4: TVS0500DRV, Package_SON:WSON-6-1EP_2x2mm_P0.65mm_EP1x1.6mm, F.Cu at (110.5, 144.8)
- added F1: MF-MSMF075/33X, Fuse:Fuse_1812_4532Metric, F.Cu at (113.2, 130.8)
- added H1: MountingHole_2.2mm_M2, MountingHole:MountingHole_2.2mm_M2, F.Cu at (103.0, 103.0)
- added H2: MountingHole_2.2mm_M2, MountingHole:MountingHole_2.2mm_M2, F.Cu at (133.0, 103.0)
- added H3: MountingHole_2.2mm_M2, MountingHole:MountingHole_2.2mm_M2, F.Cu at (103.0, 151.0)
- added H4: MountingHole_2.2mm_M2, MountingHole:MountingHole_2.2mm_M2, F.Cu at (133.0, 151.0)
- added J1: USB_C, Connector_USB:USB_C_Receptacle_GCT_USB4110, F.Cu at (103.7, 131.0)
- added J2: RADIO_LINK, Connector_JST:JST_GH_BM15B-GHS-TBT_1x15-1MP_P1.25mm_Vertical, F.Cu at (118.0, 150.2)
- added R1: 10k, Resistor_SMD:R_0402_1005Metric, F.Cu at (105.6, 106.3)
- added R10: 5.1k, Resistor_SMD:R_0402_1005Metric, F.Cu at (117.2, 138.2)
- added R11: 100k, Resistor_SMD:R_0402_1005Metric, F.Cu at (119.5, 141.8)
- added R12: 68k, Resistor_SMD:R_0402_1005Metric, F.Cu at (121.5, 141.8)
- added R13: 10k, Resistor_SMD:R_0402_1005Metric, F.Cu at (123.5, 141.8)
- added R14: 1M, Resistor_SMD:R_0402_1005Metric, F.Cu at (125.5, 141.8)
- added R15: 1.5k, Resistor_SMD:R_0402_1005Metric, F.Cu at (132.5, 119.0)
- added R2: 470, Resistor_SMD:R_0402_1005Metric, F.Cu at (102.9, 106.4)
- added R3: 10k, Resistor_SMD:R_0402_1005Metric, F.Cu at (129.9, 121.5)
- added R4: 33, Resistor_SMD:R_0402_1005Metric, F.Cu at (107.2, 107.1)
- added R5: 22, Resistor_SMD:R_0402_1005Metric, F.Cu at (107.3, 118.5)
- added R6: 22, Resistor_SMD:R_0402_1005Metric, F.Cu at (107.3, 119.8)
- added R7: 499, Resistor_SMD:R_0402_1005Metric, F.Cu at (132.4, 106.5)
- added R8: 1.5k, Resistor_SMD:R_0402_1005Metric, F.Cu at (132.5, 114.0)
- added R9: 5.1k, Resistor_SMD:R_0402_1005Metric, F.Cu at (115.8, 138.2)
- added SW1: TS-1187A, Button_Switch_SMD:SW_Push_1P1T_XKB_TS-1187A, F.Cu at (132.0, 127.8)
- added SW2: TS-1187A, Button_Switch_SMD:SW_Push_1P1T_XKB_TS-1187A, F.Cu at (132.0, 134.5)
- added TP1: U0TXD, TestPoint:TestPoint_Pad_D1.0mm, F.Cu at (129.8, 106.5)
- added TP2: U0RXD, TestPoint:TestPoint_Pad_D1.0mm, F.Cu at (129.8, 108.6)
- added U1: ESP32-C5-WROOM-1U-N8R8, RadioBoard2027:ESP32-C5-WROOM-1U, F.Cu at (118.0, 112.2)
- added U2: USBLC6-2SC6, Package_TO_SOT_SMD:SOT-23-6, F.Cu at (111.6, 139.5)
- added U3: TPS2116DRL, Package_TO_SOT_SMD:SOT-583-8, F.Cu at (122.5, 138.5)
- added U4: AP7361C-33E, Package_TO_SOT_SMD:SOT-223-3_TabPin2, F.Cu at (121.8, 128.8)
- added U5: TPD4E05U06DQA, Package_SON:USON-10_2.5x1.0mm_P0.5mm, F.Cu at (116.5, 144.8)
- added U6: TPD4E05U06DQA, Package_SON:USON-10_2.5x1.0mm_P0.5mm, F.Cu at (124.0, 144.8)
Routing:
- net ESP_HANDSHAKE: track 0.00 -> 77.5 mm, vias 0 -> 3
- net ESP_EN: track 0.00 -> 75.6 mm, vias 0 -> 2
- net Net-(U1-EN/CHIP_PU): track 0.00 -> 66.8 mm, vias 0 -> 2
- net ESP_SPI_MISO: track 0.00 -> 59.2 mm, vias 0 -> 2
- net ESP_SPI_SCK: track 0.00 -> 50.2 mm, vias 0 -> 2
- net ESP_SPI_MOSI: track 0.00 -> 49.9 mm, vias 0 -> 2
- net ESP_DATA_READY: track 0.00 -> 49.8 mm, vias 0 -> 2
- net ESP_SPI_CS: track 0.00 -> 47.7 mm, vias 0 -> 2
- net PWR_SRC_HOST: track 0.00 -> 42.1 mm, vias 0 -> 3
- net GND: track 0.00 -> 31.9 mm, vias 0 -> 38
- net USB_DP: track 0.00 -> 31.0 mm
- net USB_DN: track 0.00 -> 30.8 mm
- net +3V3_HOST: track 0.00 -> 28.3 mm, vias 0 -> 2
- net Net-(U1-GPIO28): track 0.00 -> 27.8 mm
- net Net-(J1-CC1): track 0.00 -> 25.7 mm, vias 0 -> 2
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- added copper zone on In2.Cu, net +3V3
- added copper zone on B.Cu, net GND
- added copper zone on F.Cu, net GND
- added copper zone on In1.Cu, net GND
Other:
- board outline added: 36 x 54 mm
- copper layers 2 -> 4

Commit message: radioboard fixes
Parts:
- moved U2 13.8 mm to (110.3, 125.8), turned to 90 degrees
- moved R9 9.62 mm to (113.0, 129.0), turned to 0 degrees
- moved C5 9.46 mm to (115.6, 126.4), turned to 90 degrees
- moved R10 9.20 mm to (108.0, 138.4), turned to 180 degrees
- moved D2 8.58 mm to (110.6, 135.0), turned to 90 degrees
- moved F1 4.11 mm to (115.0, 134.5), turned to 180 degrees
- moved U6 3.61 mm to (127.6, 144.6)
- moved R7 3.45 mm to (129.0, 107.1), turned to 0 degrees
- moved R5 2.28 mm to (106.6, 120.7), turned to -90 degrees
- moved TP2 1.22 mm to (131.0, 108.4)
- moved TP1 1.22 mm to (131.0, 106.3)
- moved R6 1.03 mm to (107.8, 120.7), turned to -90 degrees
- moved U5 0.84 mm to (116.8, 145.6), turned to 90 degrees
Connections:
- net PWR_SRC_HOST renamed /ESP32-C5/PWR_SRC_HOST
- net USB_DN renamed /ESP32-C5/USB_DN
- net USB_DP renamed /ESP32-C5/USB_DP
- J2 pad 10: ESP_SPI_CS -> /Controlboard Link/ESP_SPI_CS
- J2 pad 12: ESP_HANDSHAKE -> /Controlboard Link/ESP_HANDSHAKE
- J2 pad 13: ESP_DATA_READY -> /Controlboard Link/ESP_DATA_READY
- J2 pad 14: ESP_EN -> /Controlboard Link/ESP_EN
- J2 pad 4: ESP_SPI_SCK -> /Controlboard Link/ESP_SPI_SCK
- J2 pad 6: ESP_SPI_MOSI -> /Controlboard Link/ESP_SPI_MOSI
- J2 pad 8: ESP_SPI_MISO -> /Controlboard Link/ESP_SPI_MISO
- R2 pad 1: ESP_EN -> /Controlboard Link/ESP_EN
- R4 pad 1: ESP_SPI_MISO -> /Controlboard Link/ESP_SPI_MISO
- U1 pad 12: ESP_SPI_CS -> /Controlboard Link/ESP_SPI_CS
- U1 pad 17: ESP_DATA_READY -> /Controlboard Link/ESP_DATA_READY
- U1 pad 5: ESP_HANDSHAKE -> /Controlboard Link/ESP_HANDSHAKE
- U1 pad 8: ESP_SPI_SCK -> /Controlboard Link/ESP_SPI_SCK
- U1 pad 9: ESP_SPI_MOSI -> /Controlboard Link/ESP_SPI_MOSI
- U5 pad 1: ESP_SPI_SCK -> /Controlboard Link/ESP_SPI_SCK
- U5 pad 10: unconnected-(U5-NC-Pad10) -> /Controlboard Link/ESP_SPI_SCK
- U5 pad 2: ESP_SPI_MOSI -> /Controlboard Link/ESP_SPI_MOSI
- U5 pad 4: ESP_SPI_MISO -> /Controlboard Link/ESP_SPI_MISO
- U5 pad 5: ESP_SPI_CS -> /Controlboard Link/ESP_SPI_CS
- U5 pad 6: unconnected-(U5-NC-Pad6) -> /Controlboard Link/ESP_SPI_CS
- U5 pad 7: unconnected-(U5-NC-Pad7) -> /Controlboard Link/ESP_SPI_MISO
- U5 pad 9: unconnected-(U5-NC-Pad9) -> /Controlboard Link/ESP_SPI_MOSI
- U6 pad 1: ESP_HANDSHAKE -> /Controlboard Link/ESP_HANDSHAKE
- U6 pad 10: unconnected-(U6-NC-Pad10) -> /Controlboard Link/ESP_HANDSHAKE
- U6 pad 2: ESP_DATA_READY -> /Controlboard Link/ESP_DATA_READY
- U6 pad 4: ESP_EN -> GND
- U6 pad 5: unconnected-(U6-D2--Pad5) -> /Controlboard Link/ESP_EN
- U6 pad 6: unconnected-(U6-NC-Pad6) -> /Controlboard Link/ESP_EN
- U6 pad 7: unconnected-(U6-NC-Pad7) -> GND
- U6 pad 9: unconnected-(U6-NC-Pad9) -> /Controlboard Link/ESP_DATA_READY
Routing:
- net /Controlboard Link/ESP_EN: track 0.00 -> 79.9 mm, vias 0 -> 2
- net ESP_HANDSHAKE: track 77.5 -> 0.00 mm, vias 3 -> 0
- net ESP_EN: track 75.6 -> 0.00 mm, vias 2 -> 0
- net /Controlboard Link/ESP_HANDSHAKE: track 0.00 -> 71.4 mm, vias 0 -> 2
- net /Controlboard Link/ESP_SPI_MISO: track 0.00 -> 63.3 mm, vias 0 -> 2
- net ESP_SPI_MISO: track 59.2 -> 0.00 mm, vias 2 -> 0
- net /Controlboard Link/ESP_SPI_SCK: track 0.00 -> 57.5 mm, vias 0 -> 2
- net /Controlboard Link/ESP_SPI_MOSI: track 0.00 -> 57.5 mm, vias 0 -> 2
- net /Controlboard Link/ESP_SPI_CS: track 0.00 -> 57.5 mm, vias 0 -> 2
- net ESP_SPI_SCK: track 50.2 -> 0.00 mm, vias 2 -> 0
- net ESP_SPI_MOSI: track 49.9 -> 0.00 mm, vias 2 -> 0
- net ESP_DATA_READY: track 49.8 -> 0.00 mm, vias 2 -> 0
- net ESP_SPI_CS: track 47.7 -> 0.00 mm, vias 2 -> 0
- net /Controlboard Link/ESP_DATA_READY: track 0.00 -> 43.5 mm, vias 0 -> 2
- net /ESP32-C5/USB_DN: track 30.8 -> 4.59 mm
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- added copper zone on In2.Cu, net GND
Other:
- board text added: "BOOT"
- board text added: "PWR"
- board text added: "RESET"
- board text added: "RX"
- board text added: "RadioBoard2027 rev A"
- board text added: "STAT"
- board text added: "TX"

Commit message: radioboard parts goes brrr
Parts:
- C1, C8: value 22uF 25V -> 22uF
- C5: value 4.7uF 25V -> 4.7uF
- SW1, SW2: value TS-1187A -> SKQGABE010; footprint Button_Switch_SMD:SW_Push_1P1T_XKB_TS-1187A -> Button_Switch_SMD:SW_SPST_SKQG_WithStem
- moved SW1 0.50 mm to (131.5, 127.8)
- moved SW2 0.50 mm to (131.5, 134.5)
Routing:
- net Net-(U1-GPIO28): track 27.8 -> 28.9 mm
