File: boards/develop-2027/controlboard/RadioBoard2027/RadioBoard2027.kicad_pcb (KiCad board)
At the start: 4 copper layers, 36 x 54 mm, 45 parts, among them J1 USB_C, J2 RADIO_LINK, SW1 SKQGABE010, SW2 SKQGABE010, U1 ESP32-C5-WROOM-1U-N8R8, U2 USBLC6-2SC6, U3 TPS2116DRL, U4 AP7361C-33E, U5 TPD4E05U06DQA, U6 TPD4E05U06DQA

Commit message: Radio link: Samtec LSHM mezzanine on both boards
ControlBoard2027 J9 and RadioBoard2027 J2 move from the JST GH cable header
to the same hermaphroditic Samtec LSHM-110-02.5 (5mm stack); the radio sits
right side up, overhanging the controlboard's east edge on J2 alone.

- Pinout and physical mating checked by script over both boards (rigid
  placement, all 20 pads land on partner pads with matching nets).
- ControlBoard: radio SPI re-routed with 45-degree trapezoid length bumps,
  CS crossing in a 4.4mm B.Cu hop over an In2 GND patch (priority above the
  +3V3 plane), pull resistors on their lines, straight J9 power/GND buses,
  R32 10k (100k read high against the C5 GPIO4 reset pull-up).
- RadioBoard: J2 on B.Cu near the board centre, U5/U6 flow-through on F.Cu
  above it, D4 on B.Cu inline on +3V3_HOST, SPI re-matched end to end
  (SCK/MOSI/CS within 0.17mm), inner-layer via clearance rule closes the
  antipad slot under the row-gap vias.
- BOMs, DESIGN_NOTES, TODOs, sources, sheet notes and schematic PDF updated.
  DRC 0 errors / 0 unconnected / parity clean on both; ERC clean apart from
  the documented ControlBoard VCAP exception.

Co-Authored-By: Claude Opus 5.5 <noreply@anthropic.com>
Parts:
- D4: moved to B.Cu
- J2: value RADIO_LINK -> RADIO_MEZZ; footprint Connector_JST:JST_GH_BM15B-GHS-TBT_1x15-1MP_P1.25mm_Vertical -> Connector_Samtec:Samtec_LSHM-110-xx.x-x-DV-S_2x10-1SH_P0.50mm_Vertical; moved to B.Cu
- moved U6 10.6 mm to (117.0, 145.7), turned to 90 degrees
- moved U5 4.03 mm to (119.5, 148.5)
- moved D4 3.15 mm to (110.5, 147.9)
- moved J2 0.80 mm to (118.8, 150.2)
Connections:
- J2 pad 1: +3V3_HOST -> /Controlboard Link/ESP_EN
- J2 pad 10: /Controlboard Link/ESP_SPI_CS -> GND
- J2 pad 11: GND -> /Controlboard Link/ESP_SPI_SCK
- J2 pad 12: /Controlboard Link/ESP_HANDSHAKE -> GND
- J2 pad 13: /Controlboard Link/ESP_DATA_READY -> GND
- J2 pad 14: /Controlboard Link/ESP_EN -> GND
- J2 pad 15: GND -> /Controlboard Link/ESP_SPI_MOSI
- J2 pad 3: GND -> /Controlboard Link/ESP_DATA_READY
- J2 pad 4: /Controlboard Link/ESP_SPI_SCK -> +3V3_HOST
- J2 pad 5: GND -> /Controlboard Link/ESP_HANDSHAKE
- J2 pad 6: /Controlboard Link/ESP_SPI_MOSI -> +3V3_HOST
- J2 pad 7: GND -> /Controlboard Link/ESP_SPI_MISO
- J2 pad 8: /Controlboard Link/ESP_SPI_MISO -> GND
- U5 pad 1: /Controlboard Link/ESP_SPI_SCK -> /Controlboard Link/ESP_SPI_MISO
- U5 pad 10: /Controlboard Link/ESP_SPI_SCK -> /Controlboard Link/ESP_SPI_MISO
- U5 pad 2: /Controlboard Link/ESP_SPI_MOSI -> /Controlboard Link/ESP_SPI_SCK
- U5 pad 4: /Controlboard Link/ESP_SPI_MISO -> /Controlboard Link/ESP_SPI_MOSI
- U5 pad 7: /Controlboard Link/ESP_SPI_MISO -> /Controlboard Link/ESP_SPI_MOSI
- U5 pad 9: /Controlboard Link/ESP_SPI_MOSI -> /Controlboard Link/ESP_SPI_SCK
- U6 pad 1: /Controlboard Link/ESP_HANDSHAKE -> /Controlboard Link/ESP_EN
- U6 pad 10: /Controlboard Link/ESP_HANDSHAKE -> /Controlboard Link/ESP_EN
- U6 pad 4: GND -> /Controlboard Link/ESP_HANDSHAKE
- U6 pad 5: /Controlboard Link/ESP_EN -> unconnected-(U6-D2--Pad5)
- U6 pad 6: /Controlboard Link/ESP_EN -> unconnected-(U6-D2-_FT-Pad6)
- U6 pad 7: GND -> /Controlboard Link/ESP_HANDSHAKE
Routing:
- net /Controlboard Link/ESP_EN: track 79.9 -> 89.7 mm, vias 2 -> 3
- net /Controlboard Link/ESP_DATA_READY: track 43.5 -> 51.6 mm, vias 2 -> 3
- net GND: track 44.9 -> 37.7 mm, vias 47 -> 45
- net /Controlboard Link/ESP_HANDSHAKE: track 71.4 -> 77.5 mm, vias 2 -> 3
- net +3V3_HOST: track 35.0 -> 36.5 mm, vias 2 -> 3
- net /Controlboard Link/ESP_SPI_CS: track 57.5 -> 58.8 mm, vias 2 -> 3
- net /Controlboard Link/ESP_SPI_SCK: track 57.5 -> 58.7 mm, vias 2 -> 3
- net /Controlboard Link/ESP_SPI_MOSI: track 57.5 -> 58.4 mm, vias 2 -> 3
- net /Controlboard Link/ESP_SPI_MISO: track 63.3 -> 62.4 mm, vias 2 -> 3

Commit message: RadioBoard2027: final audit fixes on the link
- CS J2-side meander bump moved clear of the CC2 via's In2 opening.
- D4 aligned so +3V3_HOST runs as one straight 0.5mm F.Cu segment from its via.
- U3_PR1 B.Cu track now ends on its via centre (kept at 45 degrees).
- MOSI trapezoids exactly 4W apart.
- Link-via inner clearance rule: hole clearance 0.22mm (margin over JLC 0.2mm).
- DESIGN_NOTES: rule precedence and fab-limit notes corrected.

Co-Authored-By: Claude Opus 5.5 <noreply@anthropic.com>
Routing:
- net GND: vias 45 -> 44
