File: boards/develop-2027/dribbler-motorboard/dribbler-board-v0.2/motor_controller.kicad_sch (KiCad schematic)
At the start: 27 parts, among them SW1 RESET, U4 STSPIN32G0B2

Commit message: updated SWD header and labels
updated SWD header and labels
Other:
- title: STSPIN32G0A2 Motor Controller -> STSPIN32G0B2 Motor Controller
Changed lines of the file:
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@@
 	(paper "A4")
 	(title_block
-		(title "STSPIN32G0A2 Motor Controller")
+		(title "STSPIN32G0B2 Motor Controller")
 		(date "2026-09-07")
 		(rev "v1.0")

Commit message: Edited P/N
Updated digikey P/Ns to correct components for current sensing and overcurrent protection. Changes reflected in digikey list for dribbler-board-v0.2
Parts:
- C10: Manufacturer P/N GRM155R71H102KA01D -> CC0402KRX7R9BB333; Vendor P/N 490-1303-1-ND -> 13-CC0402KRX7R9BB333CT-ND
- R9: Manufacturer P/N RT0402BRD071K13L -> CPF0402B33RE; Vendor P/N YAG1412CT-ND -> A119938CT-ND
Changed lines of the file:
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@@
 			)
 		)
-		(property "Datasheet" "https://search.murata.co.jp/Ceramy/image/img/A01X/G101/ENG/GRM155R71H272KA01-01.pdf"
+		(property "Datasheet" "https://yageogroup.com/content/datasheet/asset/file/UPY-GPHC_X7R_6_3V-TO-250V"
 			(at 222.25 127 0)
 			(hide yes)
@@
 			)
 		)
-		(property "Manufacturer P/N" "GRM155R71H102KA01D"
+		(property "Manufacturer P/N" "CC0402KRX7R9BB333"
 			(at 222.25 127 0)
 			(hide yes)
@@
 			)
 		)
-		(property "Vendor P/N" "490-1303-1-ND"
+		(property "Vendor P/N" "13-CC0402KRX7R9BB333CT-ND"
 			(at 222.25 127 0)
 			(hide yes)
@@
 			)
 		)
-		(property "Datasheet" "https://yageogroup.com/content/datasheet/asset/file/PYU-RT_1-TO-0-01_ROHS_L"
+		(property "Datasheet" "https://www.te.com/commerce/DocumentDelivery/DDEController?Action=srchrtrv&DocNm=1773200&DocType=Data%20Sheet&DocLang=English&DocFormat=pdf&PartCntxt=1879061-3"
 			(at 209.55 120.65 0)
 			(hide yes)
@@
 			)
 		)
-		(property "Manufacturer P/N" "RT0402BRD071K13L"
+		(property "Manufacturer P/N" "CPF0402B33RE"
 			(at 209.55 120.65 0)
 			(hide yes)
@@
 			)
 		)
-		(property "Vendor P/N" "YAG1412CT-ND"
+		(property "Vendor P/N" "A119938CT-ND"
 			(at 209.55 120.65 0)
 			(hide yes)
