File: boards/develop-2027/power-board/power-board-proto/mcu_conn.kicad_sch (KiCad schematic)
At the start: 0 parts

Commit message: Add MCU & MCU connectors
Parts:
- added J3: 12402012E212A, symbol Connector:USB_C_Receptacle_USB2.0_16P
- added J4: SWD, Package_SON:USON-10_2.5x1.0mm_P0.5mm, symbol Connector:Conn_01x04_Pin
- added R52, R53: 5.1k, symbol Device:R
- added U8: TPD4E02B04DQA, Package_SON:USON-10_2.5x1.0mm_P0.5mm, symbol Power_Protection:TPD4E02B04DQA
Connections:
- new net +3.3V: J4.1 (Pin_1)
- new net CC1: J3.A5 (CC1), R52.1
- new net CC2: J3.B5 (CC2), R53.1
- new net GND: J3.A1 (GND), J3.A12 (GND), J3.B1 (GND), J3.B12 (GND), J4.4 (Pin_4), R52.2, R53.2, U8.3 (G), U8.8 (G)
- new net SWDCLK: J4.3 (Pin_3)
- new net SWDIO: J4.2 (Pin_2)
- new net USP.DM: J3.A7 (D-), J3.B7 (D-), U8.1 (IO1)
- new net USP.DP: J3.A6 (D+), J3.B6 (D+), U8.2 (IO2)
- new net VBUS: J3.A4 (VBUS), J3.A9 (VBUS), J3.B4 (VBUS), J3.B9 (VBUS), U8.5 (IO4)
- no-connect marks 0 -> 4
Other:
- note added: "SWD Connector"
- note added: "USB-C Port"

Commit message: tweak footprints assignments
Parts:
- R52, R53: footprint (none) -> Resistor_SMD:R_0402_1005Metric_Pad0.72x0.64mm_HandSolder
Changed lines of the file:
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@@
 			)
 		)
-		(property "Footprint" ""
+		(property "Footprint" "Resistor_SMD:R_0402_1005Metric_Pad0.72x0.64mm_HandSolder"
 			(at 116.332 40.64 90)
 			(hide yes)
@@
 			)
 		)
-		(property "Footprint" ""
+		(property "Footprint" "Resistor_SMD:R_0402_1005Metric_Pad0.72x0.64mm_HandSolder"
 			(at 129.032 40.64 90)
 			(hide yes)

Commit message: fix ERC warnings
Connections:
- net USP.DM renamed USB.DM
- net USP.DP renamed USB.DP
Changed lines of the file:
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@@
 		)
 	)
-	(label "USP.DP"
-		(at 110.49 66.04 0)
+	(label "USB.DP"
+		(at 118.11 66.04 180)
 		(effects
 			(font
 				(size 1.27 1.27)
 			)
-			(justify left bottom)
+			(justify right bottom)
+		)
+	)
+	(label "USB.DM"
+		(at 118.11 63.5 180)
+		(effects
+			(font
+				(size 1.27 1.27)
+			)
+			(justify right bottom)
 		)
 	)
@@
 		)
 	)
-	(label "USP.DM"
-		(at 110.49 63.5 0)
-		(effects
-			(font
-				(size 1.27 1.27)
-			)
-			(justify left bottom)
-		)
-	)

Commit message: mostly finalize footprints
Parts:
- J3: footprint (none) -> RJ-Connectors:USB_C_Receptable_Amphenol_12402012E212A
Changed lines of the file:
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@@
 			)
 		)
-		(property "Footprint" ""
+		(property "Footprint" "RJ-Connectors:USB_C_Receptable_Amphenol_12402012E212A"
 			(at 60.96 63.5 0)
 			(hide yes)

Commit message: WIP layout & routing
Parts:
- removed J3: 12402012E212A, RJ-Connectors:USB_C_Receptable_Amphenol_12402012E212A, symbol Connector:USB_C_Receptacle_USB2.0_16P
- added J19: 12402012E212A, RJ-Connectors:USB_C_Receptable_Amphenol_12402012E212A, symbol RJ-Connectors:12402012E212A
- J17: renamed from J4; footprint Package_SON:USON-10_2.5x1.0mm_P0.5mm -> Connector_PinHeader_2.54mm:PinHeader_1x04_P2.54mm_Vertical
- renumbered R52 to R58, R53 to R59, U8 to U7
Connections:
- net CC1: now also J19.B5 (CC1_B)
- net CC2: now also J19.A5 (CC1_A)
- net GND: now also J19.A1_B12 (GND), J19.B1_A12 (GND), J19.SH1 (SHIELD), J19.SH2 (SHIELD), J19.SH3 (SHIELD), J19.SH4 (SHIELD)
- net USB.DM: now also J19.A7 (D-_A), J19.B7 (D-_B)
- net USB.DP: now also J19.A6 (D+_A), J19.B6 (D+_B)
- net VBUS: now also J19.A4_B9 (VBUS), J19.B4_A9 (VBUS)
- no-connect marks 4 -> 3
Other:
- moved on the sheet: R58, R59, U7

Commit message: add fixes for problems caught by AI design review
Connections:
- net VBUS: no longer U7.5 (IO4)
- no-connect marks 3 -> 4
Changed lines of the file:
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@@
-	)
-	(junction
-		(at 125.73 55.88)
-		(diameter 0)
-		(color 0 0 0 0)
 	)
 	(junction
@@
 		(at 57.15 68.58)
 	)
+	(no_connect
+		(at 125.73 69.85)
+	)
 	(bus_entry
 		(at 153.67 66.04)
@@
 	(wire
 		(pts
-			(xy 125.73 55.88) (xy 125.73 69.85)
-		)
-		(stroke
-			(width 0)
-			(type default)
-		)
-	)
-	(wire
-		(pts
 			(xy 138.43 66.04) (xy 138.43 69.85)
 		)
@@
 	(wire
 		(pts
-			(xy 92.71 55.88) (xy 125.73 55.88)
-		)
-		(stroke
-			(width 0)
-			(type default)
-		)
-	)
-	(wire
-		(pts
-			(xy 125.73 55.88) (xy 128.27 55.88)
+			(xy 92.71 55.88) (xy 95.25 55.88)
 		)
 		(stroke
@@
 	(hierarchical_label "VBUS"
 		(shape output)
-		(at 128.27 55.88 0)
-		(effects
-			(font
+		(at 95.25 55.88 0)
+		(effects
+			(font

Commit message: finalize DigiKey part numbers
Parts:
- R58, R59: Manufacturer P/N (none) -> RC0402FR-075K1L; Vendor (none) -> DigiKey; Vendor P/N (none) -> 311-5.10KLRCT-ND
Changed lines of the file:
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@@
 			)
 		)
-		(property "Datasheet" ""
-			(at 152.4 40.64 0)
-			(hide yes)
-			(show_name no)
-			(do_not_autoplace no)
-			(effects
-				(font
-					(size 1.27 1.27)
-				)
-			)
-		)
-		(property "Description" "Resistor"
+		(property "Datasheet" "https://yageogroup.com/content/datasheet/asset/file/PYU-RC_GROUP_51_ROHS_L"
+			(at 152.4 40.64 0)
+			(hide yes)
+			(show_name no)
+			(do_not_autoplace no)
+			(effects
+				(font
+					(size 1.27 1.27)
+				)
+			)
+		)
+		(property "Description" "5.1 kOhms ±1% 0.063W, 1/16W Chip Resistor 0402 (1005 Metric) Moisture Resistant Thick Film"
+			(at 152.4 40.64 0)
+			(hide yes)
+			(show_name no)
+			(do_not_autoplace no)
+			(effects
+				(font
+					(size 1.27 1.27)
+				)
+			)
+		)
+		(property "Manufacturer P/N" "RC0402FR-075K1L"
+			(at 152.4 40.64 0)
+			(hide yes)
+			(show_name no)
+			(do_not_autoplace no)
+			(effects
+				(font
+					(size 1.27 1.27)
+				)
+			)
+		)
+		(property "Vendor" "DigiKey"
+			(at 152.4 40.64 0)
+			(hide yes)
+			(show_name no)
+			(do_not_autoplace no)
+			(effects
+				(font
+					(size 1.27 1.27)
+				)
+			)
+		)
+		(property "Vendor P/N" "311-5.10KLRCT-ND"
 			(at 152.4 40.64 0)
 			(hide yes)
@@
 			)
 		)
-		(property "Datasheet" ""
-			(at 165.1 40.64 0)
-			(hide yes)
-			(show_name no)
-			(do_not_autoplace no)
-			(effects
-				(font
-					(size 1.27 1.27)
-				)
-			)
-		)
-		(property "Description" "Resistor"
-			(at 165.1 40.64 0)
-			(hide yes)
+		(property "Datasheet" "https://yageogroup.com/content/datasheet/asset/file/PYU-RC_GROUP_51_ROHS_L"
+			(at 165.1 40.64 0)
+			(hide yes)
+			(show_name no)
+			(do_not_autoplace no)
+			(effects
+				(font
+					(size 1.27 1.27)
+				)
+			)
+		)
+		(property "Description" "5.1 kOhms ±1% 0.063W, 1/16W Chip Resistor 0402 (1005 Metric) Moisture Resistant Thick Film"
+			(at 165.1 40.64 0)
+			(hide yes)
+			(show_name no)
+			(do_not_autoplace no)
+			(effects
+				(font
+					(size 1.27 1.27)
+				)
+			)
+		)
+		(property "Manufacturer P/N" "RC0402FR-075K1L"
+			(at 165.1 40.64 0)
+			(hide yes)
+			(show_name no)
+			(do_not_autoplace no)
+			(effects
+				(font
+					(size 1.27 1.27)
+				)
+			)
+		)
+		(property "Vendor" "DigiKey"
+			(at 165.1 40.64 0)
+			(hide yes)
+			(show_name no)
+			(do_not_autoplace no)
+			(effects
+				(font
+					(size 1.27 1.27)
+				)
+			)
+		)
+		(property "Vendor P/N" "311-5.10KLRCT-ND"
+			(at 165.1 40.64 0)
+			(hide yes)
