File: boards/develop-2027/power-board/power-board-proto/power-board-proto.kicad_pcb (KiCad board)
At the start: 4 copper layers, 100 x 100 mm, 220 parts, among them J1 Batt Balance, J11 Dribbler Motor, J12 Control, J14 Dribbler Board, J15 Kicker Board, J16 Fan, J17 SWD, J19 12402012E212A, J2 Batt Power, J3 Drive Motor 1, J4 Drive Motor 2, J7 Drive Motor 1, J8 Drive Motor 2, Q1 T2N7002BK,LM, Q11 AOD4185, Q13 T2N7002BK,LM, Q16 T2N7002BK,LM, Q17 T2N7002BK,LM, Q18 T2N7002BK,LM, Q2 T2N7002BK,LM, Q3 AOD4185, Q5 AOD4185, Q8 AOD4185, Q9 AOD4185, SW1 Main Power, SW2 BOOTSEL, SW3 RESET, U1 RP2354B, U10 LM75ADP, U2 TLV75533PDBVR, U3 INA4180A3IPWR, U4 LMR51430X, U5 LMR51430X, U6 SIC437A, U7 TPD4E02B04DQA, U8 LM66100DCK, U9 LM66100DCK, Y1 ABM8-272-T3

Commit message: WIP fixes from AI layout review
Parts:
- removed Q1: T2N7002BK,LM, Package_TO_SOT_SMD:SOT-23-3
- added Q19: T2N7002BK,LM, Package_TO_SOT_SMD:SOT-23-3, F.Cu at (107.0, 138.0)
- moved C50 4.25 mm to (123.5, 90.5), turned to 0 degrees
- moved R38 1.58 mm to (106.5, 140.5)
- moved D1 1.25 mm to (93.8, 62.0)
Routing:
- net Net-(Q19-G): track 3.80 -> 5.84 mm
- net Net-(D9-A): track 10.6 -> 12.2 mm
- net +3.3V: track 82.6 -> 81.3 mm
- net /Output Connectors/3.3V_EXT: track 37.9 -> 36.8 mm
- net /MCU/VBATT_Sense: track 70.9 -> 70.1 mm
- net /Output Connectors/5.0V_EXT: track 14.8 -> 14.1 mm
- net /MCU/VBATT_EN: track 107.5 -> 107.0 mm
- net GND: track 2.71 -> 2.61 mm, vias 177 -> 170
- net Net-(J2-Pin_2): vias 0 -> 59
- net /Output Power Stage/Output Load Switch (VBATT)/Output: vias 1 -> 44
- net /Battery Connectors/Output Load Switch (VBATT Master)/Input: vias 0 -> 79
- added copper zone on B.Cu, net /Battery Connectors/Output Load Switch (VBATT Master)/Input
- added copper zone on In2.Cu, net /Battery Connectors/Output Load Switch (VBATT Master)/Input
- added copper zone on B.Cu, net /Output Power Stage/Output Load Switch (VBATT)/Output
- added copper zone on F.Cu, net Net-(J2-Pin_2)
- added copper zone on In2.Cu, net Net-(J2-Pin_2)

Commit message: WIP current derating
Parts:
- removed C1, C2: 15p, Capacitor_SMD:C_0402_1005Metric_Pad0.74x0.62mm_HandSolder
- removed C10, C11, C13, C14, C15, C18, C19, C20, C21, C22, C23, C24, C25, C26, C27, C28, C3, C30, C34, C37, C39, C4, C41, C48, C6, C8, C9: 100n, Capacitor_SMD:C_0402_1005Metric_Pad0.74x0.62mm_HandSolder
- removed C12, C46, C47, C5: 4.7u, Capacitor_SMD:C_0402_1005Metric_Pad0.74x0.62mm_HandSolder
- removed C16, C17, C38: 1u, Capacitor_SMD:C_0402_1005Metric_Pad0.74x0.62mm_HandSolder
- removed C29, C33, C60, C61: 2.2u, Capacitor_SMD:C_0603_1608Metric_Pad1.08x0.95mm_HandSolder
- removed C31, C32, C35, C36: 47u, RJ-Passives:C_Elec_KEMET_A768
- removed C40, C42, C43, C44, C45, C54, C56, C57, C58, C59: 22u, RJ-Passives:C_Elec_KEMET_A768
- removed C50, C51, C52, C53, C55: 10u, Capacitor_SMD:C_1210_3225Metric_Pad1.33x2.70mm_HandSolder
- removed C7: 4.7u, Capacitor_SMD:C_0402_1005Metric
- removed D1: SMAJ22CA, Diode_SMD:D_SMA
- removed D13: OVERTEMP, LED_SMD:LED_0603_1608Metric
- removed D14, D16, D18, D2, D3, D4, D5, D7: LED, LED_SMD:LED_0603_1608Metric_Pad1.05x0.95mm_HandSolder
- removed D15, D17, D19, D6, D8: BZT52C12-13-F, Diode_SMD:D_SOD-123
- removed D9: SMD110PL-TP, Diode_SMD:D_SOD-123F
- removed F1: Fuse, RJ-Passives:Fuseholder_Keystone_3557-2
- removed G***: LOGO, RJ-Graphics:GRAPHIC_SERIAL_NUMBER
- removed G***: LOGO, RJ-Graphics:GRAPHIC_ROBOJACKET_LOGO
- removed G***: LOGO, RJ-Graphics:GRAPHIC_PIMAN_LINK_LOGO
- removed H1, H2, H3, H4: M3 Mount, MountingHole:MountingHole_3.2mm_M3_Pad
- removed J1: Batt Balance, Connector_JST:JST_XH_S6B-XH-A_1x06_P2.50mm_Horizontal
- removed J11: Dribbler Motor, Connector_JST:JST_VH_B2P-VH_1x02_P3.96mm_Vertical
- removed J12: Control, Connector_JST:JST_XH_B8B-XH-A_1x08_P2.50mm_Vertical
- removed J14: Dribbler Board, Connector_JST:JST_PH_B6B-PH-K_1x06_P2.00mm_Vertical
- removed J15: Kicker Board, Connector_JST:JST_VH_B2P-VH_1x02_P3.96mm_Vertical
- removed J16: Fan, Connector_JST:JST_XH_B2B-XH-A_1x02_P2.50mm_Vertical
- removed J17: SWD, Connector_PinHeader_2.54mm:PinHeader_1x04_P2.54mm_Vertical
- removed J19: 12402012E212A, RJ-Connectors:USB_C_Receptable_Amphenol_12402012E212A
- removed J2: Batt Power, Connector_AMASS:AMASS_XT60PW-M_1x02_P7.20mm_Horizontal
- removed J3: Drive Motor 1, Connector_JST:JST_VH_B2P-VH_1x02_P3.96mm_Vertical
- removed J4: Drive Motor 2, Connector_JST:JST_VH_B2P-VH_1x02_P3.96mm_Vertical
- removed J7: Drive Motor 1, Connector_JST:JST_PH_B8B-PH-K_1x08_P2.00mm_Vertical
- removed J8: Drive Motor 2, Connector_JST:JST_PH_B8B-PH-K_1x08_P2.00mm_Vertical
- removed JP1: SolderJumper_2_Bridged, Jumper:SolderJumper-2_P1.3mm_Bridged_Pad1.0x1.5mm
- removed JP2: SolderJumper_2_Open, Jumper:SolderJumper-2_P1.3mm_Open_Pad1.0x1.5mm
- removed L1: 3.3u 2.3A, RJ-Passives:L_Abracon_AOTA-B201610S
- removed L2: 5.6u 5.5A, RJ-Passives:L_Bourns_SRP6540
- removed L3: 6.8u 5A, RJ-Passives:L_Bourns_SRP6540
- removed L4: 3.3u 18A, RJ-Passives:L_Bourns_SRP1265A
- removed Q11, Q3, Q5, Q8, Q9: AOD4185, Package_TO_SOT_SMD:TO-252-2
- removed Q13, Q16, Q17, Q18, Q19, Q2: T2N7002BK,LM, Package_TO_SOT_SMD:SOT-23-3
- removed R1, R10, R11, R2, R38, R48, R50, R53, R54: 100k, Resistor_SMD:R_0402_1005Metric_Pad0.72x0.64mm_HandSolder
- removed R12, R6, R61, R62, R63, R7: 4.7k, Resistor_SMD:R_0402_1005Metric
- removed R13: 1m ± 1%, Resistor_SMD:R_2512_6332Metric_Pad1.40x3.35mm_HandSolder
- removed R14: 2m ± 1%, Resistor_SMD:R_2512_6332Metric_Pad1.40x3.35mm_HandSolder
- removed R15, R16: 10m ± 1%, Resistor_SMD:R_2512_6332Metric_Pad1.40x3.35mm_HandSolder
- removed R17, R30, R35, R66, R71, R76: 100, Resistor_SMD:R_0603_1608Metric_Pad0.98x0.95mm_HandSolder
- removed R18: 180k ± 1%, Resistor_SMD:R_0603_1608Metric_Pad0.98x0.95mm_HandSolder
- removed R19, R21, R23, R25, R27: 330k ± 1%, Resistor_SMD:R_0603_1608Metric_Pad0.98x0.95mm_HandSolder
- removed R20: 1.8M ± 1%, Resistor_SMD:R_0603_1608Metric_Pad0.98x0.95mm_HandSolder
- removed R22: 680k ± 1%, Resistor_SMD:R_0603_1608Metric_Pad0.98x0.95mm_HandSolder
- removed R24: 2.2M ± 1%, Resistor_SMD:R_0603_1608Metric_Pad0.98x0.95mm_HandSolder
- removed R26: 1.2M ± 1%, Resistor_SMD:R_0603_1608Metric_Pad0.98x0.95mm_HandSolder
- removed R28, R31, R32, R33, R36, R37, R64, R67, R68, R72, R73, R77, R78: 100k, Resistor_SMD:R_0603_1608Metric_Pad0.98x0.95mm_HandSolder
- removed R29, R34, R65, R70, R75: 10k, Resistor_SMD:R_0603_1608Metric_Pad0.98x0.95mm_HandSolder
- removed R3, R4: 27.4, Resistor_SMD:R_0402_1005Metric_Pad0.72x0.64mm_HandSolder
- removed R39, R60, R8, R9: 1k, Resistor_SMD:R_0402_1005Metric_Pad0.72x0.64mm_HandSolder
- removed R49: 22.1k, Resistor_SMD:R_0402_1005Metric_Pad0.72x0.64mm_HandSolder
- removed R5: 33, Resistor_SMD:R_0402_1005Metric_Pad0.72x0.64mm_HandSolder
- removed R51: 13.7k, Resistor_SMD:R_0402_1005Metric_Pad0.72x0.64mm_HandSolder
- removed R52: 499k, Resistor_SMD:R_0402_1005Metric_Pad0.72x0.64mm_HandSolder
- removed R55: 2.2R, Resistor_SMD:R_0402_1005Metric_Pad0.72x0.64mm_HandSolder
- removed R56: 191k, Resistor_SMD:R_0402_1005Metric_Pad0.72x0.64mm_HandSolder
- removed R57: 10k, Resistor_SMD:R_0402_1005Metric_Pad0.72x0.64mm_HandSolder
- removed R58, R59: 5.1k, Resistor_SMD:R_0402_1005Metric_Pad0.72x0.64mm_HandSolder
- removed R69, R74: 1k, Resistor_SMD:R_0603_1608Metric_Pad0.98x0.95mm_HandSolder
- removed SW1: Main Power, RJ-Connectors:SW_SPST_ESwitch_100SP1T2B4M6QE
- removed SW2: BOOTSEL, Button_Switch_SMD:SW_Push_1P1T_NO_CK_KMR2
- removed SW3: RESET, Button_Switch_SMD:SW_Push_1P1T_NO_CK_KMR2
- removed TP1: 3.3V, TestPoint:TestPoint_Loop_D1.80mm_Drill1.0mm_Beaded
- removed TP10: VBATT Sense, TestPoint:TestPoint_Pad_1.5x1.5mm
- removed TP11: 12.0V Sense, TestPoint:TestPoint_Pad_1.5x1.5mm
- removed TP12: 5.0V Sense, TestPoint:TestPoint_Pad_1.5x1.5mm
- removed TP13: 3.3V Sense, TestPoint:TestPoint_Pad_1.5x1.5mm
- removed TP14: UART RX, TestPoint:TestPoint_Loop_D1.80mm_Drill1.0mm_Beaded
- removed TP15: UART TX, TestPoint:TestPoint_Loop_D1.80mm_Drill1.0mm_Beaded
- removed TP16: Cell0 Scaled, TestPoint:TestPoint_Pad_1.5x1.5mm
- removed TP17: Cell3 Scaled, TestPoint:TestPoint_Pad_1.5x1.5mm
- removed TP18: Cell1 Scaled, TestPoint:TestPoint_Pad_1.5x1.5mm
- removed TP19: Cell4 Scaled, TestPoint:TestPoint_Pad_1.5x1.5mm
- removed TP2: VBATT, TestPoint:TestPoint_Loop_D1.80mm_Drill1.0mm_Beaded
- removed TP20: Cell2 Scaled, TestPoint:TestPoint_Pad_1.5x1.5mm
- removed TP21: SDA, TestPoint:TestPoint_Loop_D1.80mm_Drill1.0mm_Beaded
- removed TP22: SCL, TestPoint:TestPoint_Loop_D1.80mm_Drill1.0mm_Beaded
- removed TP23, TP24, TP25, TP26: GND, TestPoint:TestPoint_Loop_D1.80mm_Drill1.0mm_Beaded
- removed TP4: 12.0V, TestPoint:TestPoint_Loop_D1.80mm_Drill1.0mm_Beaded
- removed TP6: 5.0V, TestPoint:TestPoint_Loop_D1.80mm_Drill1.0mm_Beaded
- removed TP8: 3.3V EXT, TestPoint:TestPoint_Loop_D1.80mm_Drill1.0mm_Beaded
- removed U1: RP2354B, Package_DFN_QFN:QFN-80-1EP_10x10mm_P0.4mm_EP3.4x3.4mm
- removed U10: LM75ADP, Package_SO:TSSOP-8_3x3mm_P0.65mm
- removed U2: TLV75533PDBVR, Package_TO_SOT_SMD:SOT-23-5
- removed U3: INA4180A3IPWR, Package_SO:TSSOP-14_4.4x5mm_P0.65mm
- removed U4, U5: LMR51430X, Package_TO_SOT_SMD:SOT-23-6
- removed U6: SIC437A, Package_DFN_QFN:Vishay_PowerPAK_MLP44-24L_ThermalVias
- removed U7: TPD4E02B04DQA, Package_SON:USON-10_2.5x1.0mm_P0.5mm
- removed U8, U9: LM66100DCK, Package_TO_SOT_SMD:SOT-363_SC-70-6
- removed Y1: ABM8-272-T3, Crystal:Crystal_SMD_Abracon_ABM8G-4Pin_3.2x2.5mm
Routing:
- net /MCU/VBATT_EN: track 107.0 -> 0.00 mm, vias 2 -> 0
- net /Output Power Stage/3.3V_REG: track 91.7 -> 0.00 mm, vias 26 -> 0
- net +3.3V: track 81.3 -> 0.00 mm, vias 25 -> 0
- net /MCU/5.0V_EN: track 79.9 -> 0.00 mm, vias 2 -> 0
- net /MCU/5.0V_Sense: track 73.7 -> 0.00 mm, vias 3 -> 0
- net /MCU/3.3V_EN: track 72.6 -> 0.00 mm, vias 2 -> 0
- net /MCU/3.3V_Sense: track 70.9 -> 0.00 mm, vias 3 -> 0
- net /MCU/VBATT_Sense: track 70.1 -> 0.00 mm, vias 3 -> 0
- net /MCU/12.0V_Sense: track 67.2 -> 0.00 mm, vias 3 -> 0
- net /MCU/12.0V_EN: track 65.6 -> 0.00 mm, vias 2 -> 0
- net /MCU/12.0V_REG_EN: track 49.2 -> 0.00 mm, vias 2 -> 0
- net /Battery Connectors/Batt_Balance.Cell0: track 45.9 -> 0.00 mm
- net /Battery Connectors/Batt_Balance.Cell1: track 41.3 -> 0.00 mm
- net /MCU/UART0.TX: track 40.5 -> 0.00 mm
- net +1.1V: track 40.4 -> 0.00 mm, vias 5 -> 0
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- removed copper zone on In2.Cu, net +1.1V
- removed copper zone on F.Cu, net +3.3V
- removed copper zone on In2.Cu, net +3.3V
- removed copper zone on B.Cu, net /Battery Connectors/Output Load Switch (VBATT Master)/Input
- removed copper zone on F.Cu, net /Battery Connectors/Output Load Switch (VBATT Master)/Input
- removed copper zone on In2.Cu, net /Battery Connectors/Output Load Switch (VBATT Master)/Input
- removed copper zone on F.Cu, net /Output Connectors/+12.0V_EXT
- removed copper zone on B.Cu, net /Output Connectors/3.3V_EXT
- removed copper zone on F.Cu, net /Output Connectors/3.3V_EXT
- removed copper zone on F.Cu, net /Output Connectors/5.0V_EXT
- removed copper zone on In2.Cu, net /Output Connectors/5.0V_EXT
- removed copper zone on F.Cu, net /Output Connectors/VBATT_EXT
- removed copper zone on F.Cu, net /Output Power Stage/12.0V_REG
- removed copper zone on B.Cu, net /Output Power Stage/3.3V_REG
- removed copper zone on F.Cu, net /Output Power Stage/3.3V_REG
- removed copper zone on In2.Cu, net /Output Power Stage/3.3V_REG
- removed copper zone on B.Cu, net /Output Power Stage/5.0V_REG
- removed copper zone on F.Cu, net /Output Power Stage/5.0V_REG
- removed copper zone on F.Cu, net /Output Power Stage/Output Load Switch (12V)/Output
- removed copper zone on F.Cu, net /Output Power Stage/Output Load Switch (3.3V)/Output
- removed copper zone on F.Cu, net /Output Power Stage/Output Load Switch (5.0V)/Output
- removed copper zone on B.Cu, net /Output Power Stage/Output Load Switch (VBATT)/Output
- removed copper zone on F.Cu, net /Output Power Stage/Output Load Switch (VBATT)/Output
- removed copper zone on F.Cu, net /Output Power Stage/VBATT to 12.0V Regulator/VBATT_DECOUP
- removed copper zone on B.Cu, net GND
- removed copper zone on F.Cu, net GND
- removed copper zone on In1.Cu, net GND
- removed copper zone on In2.Cu, net GND
- removed copper zone on B.Cu, net Net-(J2-Pin_2)
- removed copper zone on F.Cu, net Net-(J2-Pin_2)
- removed copper zone on In2.Cu, net Net-(J2-Pin_2)
- removed copper zone on F.Cu, net Net-(L4-Pad1)
- removed copper zone on F.Cu, net Net-(U4-SW)
- removed copper zone on F.Cu, net Net-(U5-SW)
Other:
- board outline removed
- board text removed: "CONTROL"
- board text removed: "DRIBBLER"
- board text removed: "DRIBBLER RAW"
- board text removed: "DRIVE"
- board text removed: "Designed By: Aiden Lee Many Thanks: Sean Seguin"
- board text removed: "FAN"
- board text removed: "KICKER"
- board text removed: "Power Integration Test Board Revision v1.0"
- board text removed: "Robot Rev. 2027"
