File: boards/develop-2027/drive-motorboard/drive-motorboard/drive-motorboard.kicad_pcb (KiCad board)
At the start: 6 copper layers, 50 x 50 mm, 14 parts, among them J1 MOTOR HALL, J2 MOTOR UVW, J4 COMM SPI, J6 PWR_IN, U2 AS5047P

Commit message: change motor connector pin ordering
Parts:
- added C1: 100u 35V, Capacitor_SMD:C_Elec_6.3x5.8, F.Cu at (4.47, 3.58)
- added C10: 100n 10V, Capacitor_SMD:C_0402_1005Metric, F.Cu at (10.9, 17.5)
- added C11: 1n, Capacitor_SMD:C_0402_1005Metric, F.Cu at (10.9, 19.5)
- added C12: 1u 63V, Capacitor_SMD:C_0603_1608Metric, F.Cu at (9.86, 47.0)
- added C13: 1u 63V, Capacitor_SMD:C_0603_1608Metric, F.Cu at (9.86, 49.5)
- added C14: 1u 63V, Capacitor_SMD:C_0603_1608Metric, F.Cu at (41.8, 32.6)
- added C15: 1u 63V, Capacitor_SMD:C_0603_1608Metric, F.Cu at (41.8, 35.1)
- added C16: 1u 63V, Capacitor_SMD:C_0603_1608Metric, F.Cu at (25.9, 32.6)
- added C17: 1u 63V, Capacitor_SMD:C_0603_1608Metric, F.Cu at (25.9, 35.1)
- added C18: 100n, Capacitor_SMD:C_0402_1005Metric, F.Cu at (45.4, 3.98)
- added C2: 1u 10V, Capacitor_SMD:C_0603_1608Metric, F.Cu at (11.5, 0.76)
- added C20: 1u 63V, Capacitor_SMD:C_0603_1608Metric, F.Cu at (1.50, 29.2)
- added C21: 10u 25V, Capacitor_SMD:C_0603_1608Metric, F.Cu at (1.50, 31.7)
- added C22: 10u 25V, Capacitor_SMD:C_0603_1608Metric, F.Cu at (1.50, 34.2)
- added C23: 100n 10V, Capacitor_SMD:C_0402_1005Metric, F.Cu at (19.9, 44.7)
- added C3: 1u 63V, Capacitor_SMD:C_0603_1608Metric, F.Cu at (11.5, 3.27)
- added C4: 1u 63V, Capacitor_SMD:C_0603_1608Metric, F.Cu at (11.5, 5.78)
- added C5: 1u 63V, Capacitor_SMD:C_0603_1608Metric, F.Cu at (11.5, 8.29)
- added C6: 100u 35V, Capacitor_SMD:C_Elec_6.3x5.8, F.Cu at (4.47, 11.7)
- added C7: 100n 10V, Capacitor_SMD:C_0402_1005Metric, F.Cu at (10.9, 15.5)
- added C8: 1u 63V, Capacitor_SMD:C_0603_1608Metric, F.Cu at (11.5, 10.8)
- added C9: 10u 25V, Capacitor_SMD:C_0603_1608Metric, F.Cu at (11.5, 13.3)
- added D1: FAULT, LED_SMD:LED_0603_1608Metric, F.Cu at (15.5, 20.1)
- added D10: PUSB3FR4Z, Package_DFN_QFN:Diodes_UDFN-10_1x2.5mm_P0.5mm, F.Cu at (36.1, 17.2)
- added D11: SMAJ22A, Diode_SMD:D_SMA, F.Cu at (3.57, 25.6)
- added D12: VBATT PWR, LED_SMD:LED_0603_1608Metric, F.Cu at (11.5, 29.2)
- added D2: 1N4148WL2-TP, Diode_SMD:D_SOD-882, F.Cu at (12.1, 38.9)
- added D3: 1N4148WL2-TP, Diode_SMD:D_SOD-882, F.Cu at (12.1, 41.3)
- added D4: 1N4148WL2-TP, Diode_SMD:D_SOD-882, F.Cu at (44.1, 24.5)
- added D5: 1N4148WL2-TP, Diode_SMD:D_SOD-882, F.Cu at (44.1, 26.9)
- added D6: 1N4148WL2-TP, Diode_SMD:D_SOD-882, F.Cu at (28.1, 24.5)
- added D7: 1N4148WL2-TP, Diode_SMD:D_SOD-882, F.Cu at (28.1, 26.9)
- added D8: PUSB3FR4Z, Package_DFN_QFN:Diodes_UDFN-10_1x2.5mm_P0.5mm, F.Cu at (45.5, 11.6)
- added F1: 10A 63V, Fuse:Fuse_1206_3216Metric_Pad1.42x1.75mm_HandSolder, F.Cu at (6.49, 29.6)
- added J3: PROG SPI, Connector_JST:JST_GH_SM06B-GHS-TB_1x06-1MP_P1.25mm_Horizontal, F.Cu at (38.0, 42.8)
- added J5: Conn_ST_STDC14, Connector:Tag-Connect_TC2070-IDC-FP_2x07_P1.27mm_Vertical, F.Cu at (32.3, 4.28)
- added J7: Conn_ST_STDC14, Connector_PinHeader_1.27mm:PinHeader_2x07_P1.27mm_Vertical_SMD, F.Cu at (29.8, 14.5)
- added L1: 10u 540mA, Inductor_SMD:L_1210_3225Metric, F.Cu at (6.32, 33.3)
- added Q1: STL90N10F7, Package_DFN_QFN:PQFN-8-EP_6x5mm_P1.27mm_Generic, F.Cu at (3.58, 41.2)
- added Q2: STL90N10F7, Package_DFN_QFN:PQFN-8-EP_6x5mm_P1.27mm_Generic, F.Cu at (3.58, 48.0)
- added Q3: STL90N10F7, Package_DFN_QFN:PQFN-8-EP_6x5mm_P1.27mm_Generic, F.Cu at (35.5, 26.8)
- added Q4: STL90N10F7, Package_DFN_QFN:PQFN-8-EP_6x5mm_P1.27mm_Generic, F.Cu at (35.5, 33.6)
- added Q5: STL90N10F7, Package_DFN_QFN:PQFN-8-EP_6x5mm_P1.27mm_Generic, F.Cu at (19.6, 26.8)
- added Q6: STL90N10F7, Package_DFN_QFN:PQFN-8-EP_6x5mm_P1.27mm_Generic, F.Cu at (19.6, 33.6)
- added R1: 15m ±1% 3W, RJ-Passives:R_Shunt_Analog_2512_6332_HighAccuracy, F.Cu at (4.47, 18.6)
- added R10: 0R, Resistor_SMD:R_0402_1005Metric, F.Cu at (9.30, 44.7)
- added R11: 68R, Resistor_SMD:R_0402_1005Metric, F.Cu at (41.3, 24.3)
- added R12: 68R, Resistor_SMD:R_0402_1005Metric, F.Cu at (41.3, 26.3)
- added R13: 0R, Resistor_SMD:R_0402_1005Metric, F.Cu at (41.3, 28.3)
- added R14: 0R, Resistor_SMD:R_0402_1005Metric, F.Cu at (41.3, 30.3)
- added R15: 68R, Resistor_SMD:R_0402_1005Metric, F.Cu at (25.3, 24.3)
- added R16: 68R, Resistor_SMD:R_0402_1005Metric, F.Cu at (25.3, 26.3)
- added R17: 0R, Resistor_SMD:R_0402_1005Metric, F.Cu at (25.3, 28.3)
- added R18: 0R, Resistor_SMD:R_0402_1005Metric, F.Cu at (25.3, 30.3)
- added R19: 1.13k ±0.1%, Resistor_SMD:R_0402_1005Metric, F.Cu at (42.5, 0.49)
- added R2: 10k, Resistor_SMD:R_0402_1005Metric, F.Cu at (14.9, 0.49)
- added R20: 16.5k ±0.1%, Resistor_SMD:R_0402_1005Metric, F.Cu at (42.5, 2.48)
- added R21: 16.5k ±0.1%, Resistor_SMD:R_0402_1005Metric, F.Cu at (42.5, 4.47)
- added R22: 1.13k ±0.1%, Resistor_SMD:R_0402_1005Metric, F.Cu at (42.5, 6.46)
- added R23: 8.25k ±0.5%, Resistor_SMD:R_0201_0603Metric, F.Cu at (45.2, 0.38)
- added R24: 300R ±1%, Resistor_SMD:R_0201_0603Metric, F.Cu at (45.2, 2.12)
- added R25: 10k, Resistor_SMD:R_0402_1005Metric, F.Cu at (42.5, 10.5)
- added R26: 10k, Resistor_SMD:R_0402_1005Metric, F.Cu at (42.5, 12.4)
- added R27: 10k, Resistor_SMD:R_0402_1005Metric, F.Cu at (42.5, 14.4)
- added R3: 10k, Resistor_SMD:R_0402_1005Metric, F.Cu at (14.9, 2.48)
- added R31: 4.7k, Resistor_SMD:R_0402_1005Metric, F.Cu at (17.0, 44.7)
- added R32: 4.7k, Resistor_SMD:R_0402_1005Metric, F.Cu at (17.0, 46.7)
- added R33: 10k, Resistor_SMD:R_0402_1005Metric, F.Cu at (36.1, 10.0)
- added R34: 100, Resistor_SMD:R_0402_1005Metric, F.Cu at (36.1, 12.0)
- added R35: 100k, Resistor_SMD:R_0402_1005Metric, F.Cu at (9.04, 24.3)
- added R36: 10k, Resistor_SMD:R_0402_1005Metric, F.Cu at (9.04, 26.3)
- added R37: 100, Resistor_SMD:R_0402_1005Metric, F.Cu at (36.1, 14.0)
- added R4: 1.13k ±0.1%, Resistor_SMD:R_0402_1005Metric, F.Cu at (14.9, 4.47)
- added R5: 33k ±0.1%, Resistor_SMD:R_0402_1005Metric, F.Cu at (14.9, 6.46)
- added R6: 10k, Resistor_SMD:R_0402_1005Metric, F.Cu at (14.9, 8.46)
- added R7: 68R, Resistor_SMD:R_0402_1005Metric, F.Cu at (9.30, 38.8)
- added R8: 68R, Resistor_SMD:R_0402_1005Metric, F.Cu at (9.30, 40.7)
- added R9: 0R, Resistor_SMD:R_0402_1005Metric, F.Cu at (9.30, 42.7)
- added SW1: RESET, Button_Switch_SMD:SW_Push_1P1T_NO_CK_KMR2, F.Cu at (19.7, 1.82)
- added U1: STSPIN32G0B2, Package_DFN_QFN:VQFN-48-1EP_7x7mm_P0.5mm_EP2.6x2.6mm, F.Cu at (18.1, 14.1)
- added U3: LM75ADP, Package_SO:TSSOP-8_3x3mm_P0.65mm, F.Cu at (19.0, 41.4)
- added U4: TPS62177DQC, Package_SON:WSON-10-1EP_2x3mm_P0.5mm_EP0.84x2.4mm_ThermalVias, F.Cu at (11.3, 33.5)
Connections:
- J1 pad 1: GND -> /Motor Connections/HALL.B
- J1 pad 3: /Motor Connections/HALL.B -> /Motor Connections/HALL.C
- J1 pad 4: /Motor Connections/HALL.C -> +3.3V
- J1 pad 5: +3.3V -> GND
- J2 pad 1: /Motor Connections/MOTORW -> /Motor Connections/MOTORV
- J2 pad 2: /Motor Connections/MOTORV -> /Motor Connections/MOTORU
- J2 pad 3: /Motor Connections/MOTORU -> /Motor Connections/MOTORW
Other:
- board text added: "GND"
- board text added: "H1"
- board text added: "H2"
- board text added: "H3"
- board text added: "PHU"
- board text added: "PHV"
- board text added: "PHW"
- board text added: "V_{CC}"
