File: boards/develop-2027/drive-motorboard/drive-motorboard/motor_controller.kicad_sch (KiCad schematic)
At the start: 19 parts, among them SW1 RESET, U1 STSPIN32G0B2

Commit message: final schematic draft
Parts:
- added R3: 10k, Resistor_SMD:R_0402_1005Metric, symbol Device:R
- renumbered R24 to R4, R4 to R5, R5 to R6
Connections:
- net GND: now also R3.1; no longer U1.2 (PC14/OSC32_IN), U1.3 (PC15/OSC32_OUT)
- new net: R3.2, U1.2 (PC14/OSC32_IN), U1.3 (PC15/OSC32_OUT)
Other:
- moved on the sheet: C11, R4, R5, U1E

Commit message: fix mess caused by multiple variants
Parts:
- C11: Manufacturer P/N GRM155R71H102KA01D -> CL05B102KB5NNNC; Vendor DigiKey -> LCSC; Vendor P/N 490-1303-1-ND -> C14442
- R1: Vendor DigiKey -> LCSC; Vendor P/N CRA2512-FZ-R015ELFCT-ND -> C2073490
- R4: Vendor DigiKey -> LCSC; Vendor P/N YAG1370CT-ND -> C852599
- R5: Manufacturer P/N RT0402BRD0733KL -> AT0402BRD0733KL; Vendor DigiKey -> LCSC; Vendor P/N YAG1412CT-ND -> C5455470
- U1: Vendor DigiKey -> LCSC; Vendor P/N 497-STSPIN32G0B2-ND -> C23064814; now left out of the parts list

Commit message: final layout draft
Parts:
- removed C6: 100u 35V, Capacitor_SMD:C_Elec_6.3x5.8, symbol Device:C_Polarized
Changed lines of the file:
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@@
 	)
 	(junction
-		(at 43.18 27.94)
-		(diameter 0)
-		(color 0 0 0 0)
-	)
-	(junction
 		(at 101.6 144.78)
 		(diameter 0)
@@
 	(wire
 		(pts
-			(xy 43.18 27.94) (xy 43.18 30.48)
-		)
-		(stroke
-			(width 0)
-			(type default)
-		)
-	)
-	(wire
-		(pts
 			(xy 101.6 115.57) (xy 82.55 115.57)
 		)
@@
 	(wire
 		(pts
-			(xy 43.18 27.94) (xy 57.15 27.94)
-		)
-		(stroke
-			(width 0)
-			(type default)
-		)
-	)
-	(wire
-		(pts
 			(xy 101.6 173.99) (xy 101.6 144.78)
 		)
@@
 	(wire
 		(pts
-			(xy 26.67 27.94) (xy 43.18 27.94)
+			(xy 26.67 27.94) (xy 57.15 27.94)
 		)
 		(stroke
@@
 	(wire
 		(pts
-			(xy 43.18 38.1) (xy 43.18 40.64)
-		)
-		(stroke
-			(width 0)
-			(type default)
-		)
-	)
-	(wire
-		(pts
 			(xy 90.17 78.74) (xy 90.17 80.01)
 		)
@@
 	)
 	(symbol
-		(lib_id "power:GND")
-		(at 43.18 40.64 0)
-		(unit 1)
-		(body_style 1)
-		(exclude_from_sim no)
-		(in_bom yes)
-		(on_board yes)
-		(in_pos_files yes)
-		(dnp no)
-		(fields_autoplaced yes)
-		(property "Reference" "#PWR05"
-			(at 43.18 46.99 0)
-			(hide yes)
-			(show_name no)
-			(do_not_autoplace no)
-			(effects
-				(font
-					(size 1.27 1.27)
-				)
-			)
-		)
-		(property "Value" "GND"
-			(at 43.18 45.72 0)
-			(show_name no)
-			(do_not_autoplace no)
-			(effects
-				(font
-					(size 1.27 1.27)
-				)
-			)
-		)
-		(property "Footprint" ""
-			(at 43.18 40.64 0)
-			(hide yes)
-			(show_name no)
-			(do_not_autoplace no)
-			(effects
-				(font
-					(size 1.27 1.27)
-				)
-			)
-		)
-		(property "Datasheet" ""
-			(at 43.18 40.64 0)
-			(hide yes)
-			(show_name no)
-			(do_not_autoplace no)
-			(effects
-				(font
-					(size 1.27 1.27)
-				)
-			)
-		)
-		(property "Description" "Power symbol creates a global label with name \"GND\" , ground"
-			(at 43.18 40.64 0)
-			(hide yes)
-			(show_name no)
-			(do_not_autoplace no)
-			(effects
-				(font
-					(size 1.27 1.27)
-				)
-			)
-		)
-		(pin "1"
-		)
-		(instances
-			(project "drive-motorboard"
-				(path "/9e9815bc-cf1c-424b-a03b-224c05c2b627/73cb52ef-7536-45c8-9d54-fc54b3c8b275"
-					(reference "#PWR05")
-					(unit 1)
-				)
-			)
-		)
-	)
-	(symbol
 		(lib_id "power:+3.3V")
 		(at 172.72 38.1 0)
@@
 					(unit 1)
 				)
-			)
-		)
-	)
-	(symbol
-		(lib_id "Device:C_Polarized")
-		(at 43.18 34.29 0)
-		(mirror y)
-		(unit 1)
-		(body_style 1)
-		(exclude_from_sim no)
-		(in_bom yes)
-		(on_board yes)
-		(in_pos_files yes)
-		(dnp no)
-		(property "Reference" "C6"
-			(at 39.37 32.1309 0)
-			(show_name no)
-			(do_not_autoplace no)
-			(effects
-				(font
-					(size 1.27 1.27)
-				)
-				(justify left)
-			)
-		)
-		(property "Value" "100u 35V"
-			(at 39.37 34.6709 0)
-			(show_name no)
-			(do_not_autoplace no)
-			(effects
-				(font
-					(size 1.27 1.27)
-				)
-				(justify left)
-			)
-		)
-		(property "Footprint" "Capacitor_SMD:C_Elec_6.3x5.8"
-			(at 42.2148 38.1 0)
-			(hide yes)
-			(show_name no)
-			(do_not_autoplace no)
-			(effects
-				(font
-					(size 1.27 1.27)
-				)
-			)
-		)
-		(property "Datasheet" "https://industrial.panasonic.com/cdbs/www-data/pdf/RDE0000/ABA0000C1240.pdf"
-			(at 43.18 34.29 0)
-			(hide yes)
-			(show_name no)
-			(do_not_autoplace no)
-			(effects
-				(font
-					(size 1.27 1.27)
-				)
-			)
-		)
-		(property "Description" "CAP ALUM 100uF ±20% 35V SMD"
-			(at 43.18 34.29 0)
-			(hide yes)
-			(show_name no)
-			(do_not_autoplace no)
-			(effects
-				(font
-					(size 1.27 1.27)
-				)
-			)
-		)
-		(property "Manufacturer P/N" "EEE-FT1V101AP"
-			(at 43.18 34.29 0)
-			(hide yes)
-			(show_name no)
-			(do_not_autoplace no)
-			(effects
-				(font
-					(size 1.27 1.27)
-				)
-			)
-		)
-		(property "Vendor" "LCSC"
-			(at 43.18 34.29 0)
-			(hide yes)
-			(show_name no)
-			(do_not_autoplace no)
-			(effects
-				(font
-					(size 1.27 1.27)
-				)
-			)
-		)
-		(property "Vendor P/N" "C128464"
-			(at 43.18 34.29 0)
-			(hide yes)
-			(show_name no)
-			(do_not_autoplace no)
-			(effects
-				(font
-					(size 1.27 1.27)
-				)
-			)
-		)
-		(pin "1"
-		)
-		(pin "2"
-		)
-		(instances
-			(project "drive-motorboard"
-				(path "/9e9815bc-cf1c-424b-a03b-224c05c2b627/73cb52ef-7536-45c8-9d54-fc54b3c8b275"
-					(reference "C6")
-					(unit 1)
-				)
